Commit message: update model

File: open_manipulator_description/urdf/open_manipulator_chain.urdf.xacro (robot description, xacro)
@@ -18,5 +18,5 @@
   <link name="link1">
     <visual>
-      <origin xyz="0.0 0.0 0.0" rpy="0 0 0"/>
+      <origin xyz="0 0 0" rpy="0 0 0"/>
       <geometry>
         <mesh filename="package://open_manipulator_description/meshes/chain_link1.stl" scale="0.001 0.001 0.001"/>
@@ -42,5 +42,5 @@
     <parent link="link1"/>
     <child link="link2"/>
-    <origin xyz="0.012 0.0 0.036" rpy="0 0 0"/>
+    <origin xyz="0.012 0.0 0.017" rpy="0 0 0"/>
     <axis xyz="0 0 1"/>
     <limit velocity="6.5" effort="1000" lower="${-pi*0.9}" upper="${pi*0.9}" />
@@ -60,5 +60,5 @@
   <link name="link2">
     <visual>
-      <origin xyz="0.0 0.0 0.040" rpy="0 0 0"/>
+      <origin xyz="0 0 0.018" rpy="0 0 0"/>
       <geometry>
         <mesh filename="package://open_manipulator_description/meshes/chain_link2.stl" scale="0.001 0.001 0.001"/>
@@ -67,5 +67,5 @@
     </visual>
     <collision>
-      <origin xyz="0.0 0.0 0.030" rpy="0 0 0"/>
+      <origin xyz="0.0 0.0 0.048" rpy="0 0 0"/>
       <geometry>
         <box size="0.0355 0.0550 0.0515"/>
@@ -84,5 +84,5 @@
     <parent link="link2"/>
     <child link="link3"/>
-    <origin xyz="0.0 0.0 0.040" rpy="0 0 0"/>
+    <origin xyz="0.0 0.0 0.058" rpy="0 0 0"/>
     <axis xyz="0 1 0"/>
     <limit velocity="6.5" effort="1000" lower="${-pi*0.5}" upper="${pi*0.5}" />
@@ -102,5 +102,5 @@
   <link name="link3">
     <visual>
-      <origin xyz="0.022 0 0.122" rpy="0 0 0"/>
+      <origin xyz="0 0 0" rpy="0 0 0"/>
       <geometry>
         <mesh filename="package://open_manipulator_description/meshes/chain_link3.stl" scale="0.001 0.001 0.001"/>
@@ -126,7 +126,7 @@
     <parent link="link3"/>
     <child link="link4"/>
-    <origin xyz="0.022 0 0.122" rpy="0 0 0"/>
-    <axis xyz="0 1 0"/>
-    <limit velocity="6.5" effort="1000" lower="${-pi*0.5}" upper="${pi*0.4}" />
+    <origin xyz="0.024 0 0.128" rpy="0 0 0"/>
+    <axis xyz="0 1 0"/>
+    <limit velocity="6.5" effort="1000" lower="${-pi*0.3}" upper="${pi*0.3}" />
   </joint>
   <!-- Transmission 3 -->
@@ -144,5 +144,5 @@
   <link name="link4">
     <visual>
-      <origin xyz="0.124 0 0.0" rpy="0 0 0"/>
+      <origin xyz="0 0 0" rpy="0 0 0"/>
       <geometry>
         <mesh filename="package://open_manipulator_description/meshes/chain_link4.stl" scale="0.001 0.001 0.001"/>
@@ -151,7 +151,7 @@
     </visual>
     <collision>
-      <origin xyz="0.080 0 0.0" rpy="0 0 0"/>
-      <geometry>
-        <box size="0.110 0.055 0.035"/>
+      <origin xyz="0.065 0 0.0" rpy="0 0 0"/>
+      <geometry>
+        <box size="0.115 0.055 0.035"/>
       </geometry>
     </collision>
@@ -186,5 +186,5 @@
   <link name="link5">
     <visual>
-      <origin xyz="0.046 0 0" rpy="0 0 0"/>
+      <origin xyz="0 0 0" rpy="0 0 0"/>
       <geometry>
         <mesh filename="package://open_manipulator_description/meshes/chain_link5.stl" scale="0.001 0.001 0.001"/>
@@ -193,7 +193,7 @@
     </visual>
     <collision>
-      <origin xyz="0.050 0 0.005" rpy="0 0 0"/>
-      <geometry>
-        <box size="0.040 0.120 0.0650"/>
+      <origin xyz="0.043 0 0.005" rpy="0 0 0"/>
+      <geometry>
+        <box size="0.048 0.120 0.0650"/>
       </geometry>
     </collision>
@@ -209,5 +209,5 @@
   <link name="grip_link">
     <visual>
-      <origin xyz="0.0 0.047 0" rpy="0 0 0"/>
+      <origin xyz="0.028 0.0246 0" rpy="0 0 0"/>
       <geometry>
         <mesh filename="package://open_manipulator_description/meshes/chain_link_grip_l.stl" scale="0.001 0.001 0.001"/>
@@ -216,7 +216,7 @@
     </visual>
     <collision>
-      <origin xyz="0.040 0.047 0" rpy="0 0 0"/>
-      <geometry>
-        <box size="0.060 0.025 0.050"/>
+      <origin xyz="0.060 0.030 0" rpy="0 0 0"/>
+      <geometry>
+        <box size="0.065 0.035 0.050"/>
       </geometry>
     </collision>
@@ -233,7 +233,7 @@
     <parent link="link5"/>
     <child link="grip_link"/>
-    <origin xyz="0.071 0.0 0.0" rpy="0 0 0"/>
+    <origin xyz="0.0536 0.0 0.0" rpy="0 0 0"/>
     <axis xyz="0 -1 0"/>
-    <limit velocity="6.5" effort="1000" lower="-0.01" upper="0.035" />
+    <limit velocity="3.5" effort="100" lower="-0.015" upper="0.0105" />
   </joint>
   <!-- Transmission 5 -->
@@ -251,5 +251,5 @@
   <link name="grip_link_sub">
     <visual>
-      <origin xyz="0 -0.047 0" rpy="0 0 0"/>
+      <origin xyz="0.028 -0.0246 0" rpy="0 0 0"/>
       <geometry>
         <mesh filename="package://open_manipulator_description/meshes/chain_link_grip_r.stl" scale="0.001 0.001 0.001"/>
@@ -258,7 +258,7 @@
     </visual>
     <collision>
-      <origin xyz="0.040 -0.047 0" rpy="0 0 0"/>
-      <geometry>
-        <box size="0.060 0.025 0.050"/>
+      <origin xyz="0.060 -0.030 0" rpy="0 0 0"/>
+      <geometry>
+        <box size="0.065 0.035 0.050"/>
       </geometry>
     </collision>
@@ -275,7 +275,7 @@
     <parent link="link5"/>
     <child link="grip_link_sub"/>
-    <origin xyz="0.071 0.0 0" rpy="0 0 0"/>
-    <axis xyz="0 1 0"/>
-    <limit velocity="6.5" effort="1000" lower="-0.01" upper="0.035" />
+    <origin xyz="0.0536 0 0" rpy="0 0 0"/>
+    <axis xyz="0 1 0"/>
+    <limit velocity="3.5" effort="100" lower="-0.015" upper="0.0105" />
   </joint>
   <!-- Transmission 6 -->

Commit message: update joint limit

File: open_manipulator_description/urdf/open_manipulator_chain.urdf.xacro (robot description, xacro)
@@ -128,5 +128,5 @@
     <origin xyz="0.024 0 0.128" rpy="0 0 0"/>
     <axis xyz="0 1 0"/>
-    <limit velocity="6.5" effort="1000" lower="${-pi*0.3}" upper="${pi*0.3}" />
+    <limit velocity="6.5" effort="1000" lower="${-pi*0.3}" upper="${pi*0.44}" />
   </joint>
   <!-- Transmission 3 -->

Commit message: edit collision param

File: open_manipulator_description/urdf/open_manipulator_chain.urdf.xacro (robot description, xacro)
@@ -216,7 +216,7 @@
     </visual>
     <collision>
-      <origin xyz="0.060 0.030 0" rpy="0 0 0"/>
-      <geometry>
-        <box size="0.065 0.035 0.050"/>
+      <origin xyz="0.060 0.033 0" rpy="0 0 0"/>
+      <geometry>
+        <box size="0.065 0.025 0.050"/>
       </geometry>
     </collision>
@@ -258,7 +258,7 @@
     </visual>
     <collision>
-      <origin xyz="0.060 -0.030 0" rpy="0 0 0"/>
-      <geometry>
-        <box size="0.065 0.035 0.050"/>
+      <origin xyz="0.060 -0.033 0" rpy="0 0 0"/>
+      <geometry>
+        <box size="0.065 0.025 0.050"/>
       </geometry>
     </collision>

File: open_manipulator_with_tb3/urdf/open_manipulator_chain_with_tb3_waffle.urdf.xacro (robot description, xacro)
@@ -213,7 +213,7 @@
     </visual>
     <collision>
-      <origin xyz="0.060 0.030 0" rpy="0 0 0"/>
-      <geometry>
-        <box size="0.065 0.035 0.050"/>
+      <origin xyz="0.060 0.033 0" rpy="0 0 0"/>
+      <geometry>
+        <box size="0.065 0.025 0.050"/>
       </geometry>
     </collision>
@@ -255,7 +255,7 @@
     </visual>
     <collision>
-      <origin xyz="0.060 -0.030 0" rpy="0 0 0"/>
-      <geometry>
-        <box size="0.065 0.035 0.050"/>
+      <origin xyz="0.060 -0.033 0" rpy="0 0 0"/>
+      <geometry>
+        <box size="0.065 0.025 0.050"/>
       </geometry>
     </collision>

File: open_manipulator_with_tb3/urdf/open_manipulator_chain_with_tb3_waffle_pi.urdf.xacro (robot description, xacro)
@@ -213,7 +213,7 @@
     </visual>
     <collision>
-      <origin xyz="0.060 0.030 0" rpy="0 0 0"/>
-      <geometry>
-        <box size="0.065 0.035 0.050"/>
+      <origin xyz="0.060 0.033 0" rpy="0 0 0"/>
+      <geometry>
+        <box size="0.065 0.025 0.050"/>
       </geometry>
     </collision>
@@ -255,7 +255,7 @@
     </visual>
     <collision>
-      <origin xyz="0.060 -0.030 0" rpy="0 0 0"/>
-      <geometry>
-        <box size="0.065 0.035 0.050"/>
+      <origin xyz="0.060 -0.033 0" rpy="0 0 0"/>
+      <geometry>
+        <box size="0.065 0.025 0.050"/>
       </geometry>
     </collision>

Commit message: change collision range

File: open_manipulator_description/urdf/open_manipulator_chain.urdf.xacro (robot description, xacro)
@@ -25,7 +25,7 @@
     </visual>
     <collision>
-      <origin xyz="0.0 0.0 0.017" rpy="0 0 0"/>
-      <geometry>
-        <box size="0.0475 0.0295 0.0340"/>
+      <origin xyz="0 0 0" rpy="0 0 0"/>
+      <geometry>
+        <mesh filename="package://open_manipulator_description/meshes/chain_link1.stl" scale="0.001 0.001 0.001"/>
       </geometry>
     </collision>
@@ -67,7 +67,7 @@
     </visual>
     <collision>
-      <origin xyz="0.0 0.0 0.048" rpy="0 0 0"/>
-      <geometry>
-        <box size="0.0355 0.0550 0.0515"/>
+      <origin xyz="0 0 0.018" rpy="0 0 0"/>
+      <geometry>
+        <mesh filename="package://open_manipulator_description/meshes/chain_link2.stl" scale="0.001 0.001 0.001"/>
       </geometry>
     </collision>
@@ -109,7 +109,7 @@
     </visual>
     <collision>
-      <origin xyz="0.0 0 0.085" rpy="0 0 0"/>
-      <geometry>
-        <box size="0.030 0.055 0.120"/>
+      <origin xyz="0 0 0" rpy="0 0 0"/>
+      <geometry>
+        <mesh filename="package://open_manipulator_description/meshes/chain_link3.stl" scale="0.001 0.001 0.001"/>
       </geometry>
     </collision>
@@ -151,7 +151,7 @@
     </visual>
     <collision>
-      <origin xyz="0.065 0 0.0" rpy="0 0 0"/>
-      <geometry>
-        <box size="0.115 0.055 0.035"/>
+      <origin xyz="0 0 0" rpy="0 0 0"/>
+      <geometry>
+        <mesh filename="package://open_manipulator_description/meshes/chain_link4.stl" scale="0.001 0.001 0.001"/>
       </geometry>
     </collision>
@@ -193,7 +193,7 @@
     </visual>
     <collision>
-      <origin xyz="0.043 0 0.005" rpy="0 0 0"/>
-      <geometry>
-        <box size="0.048 0.120 0.0650"/>
+      <origin xyz="0 0 0" rpy="0 0 0"/>
+      <geometry>
+        <mesh filename="package://open_manipulator_description/meshes/chain_link5.stl" scale="0.001 0.001 0.001"/>
       </geometry>
     </collision>
@@ -216,7 +216,7 @@
     </visual>
     <collision>
-      <origin xyz="0.060 0.033 0" rpy="0 0 0"/>
-      <geometry>
-        <box size="0.065 0.025 0.050"/>
+      <origin xyz="0.028 0.0246 0" rpy="0 0 0"/>
+      <geometry>
+        <mesh filename="package://open_manipulator_description/meshes/chain_link_grip_l.stl" scale="0.001 0.001 0.001"/>
       </geometry>
     </collision>
@@ -258,7 +258,7 @@
     </visual>
     <collision>
-      <origin xyz="0.060 -0.033 0" rpy="0 0 0"/>
-      <geometry>
-        <box size="0.065 0.025 0.050"/>
+      <origin xyz="0.028 -0.0246 0" rpy="0 0 0"/>
+      <geometry>
+        <mesh filename="package://open_manipulator_description/meshes/chain_link_grip_r.stl" scale="0.001 0.001 0.001"/>
       </geometry>
     </collision>
