Commit message: first commit

File: open_manipulator_description/urdf/open_manipulator_chain.xacro (robot description, xacro)
@@ -1,4 +1,4 @@
 <?xml version="1.0"?>
-<!-- ROBOTIS Manipulator-X4 -->
+<!-- Open_Manipulator Chain -->
 <robot name="gazebo_open_manipulator_chain" xmlns:xacro="http://www.ros.org/wiki/xacro">
   <!-- some parameters -->
@@ -112,5 +112,5 @@
     <origin xyz="0.0 0.0 0.04235" rpy="0 0 0"/>
     <axis xyz="0 -1 0"/>
-    <limit velocity="6.5" effort="1000" lower="${-pi*0.5}" upper="${pi*0.5}" />
+    <limit velocity="6.5" effort="1000" lower="${-pi*0.9}" upper="${pi*0.9}" />
     <dynamics damping="0.1"/>
   </joint>
@@ -153,5 +153,5 @@
     <origin xyz="0.024 0.0 0.12165" rpy="0 0 0"/>
     <axis xyz="0 -1 0"/>
-    <limit velocity="6.5" effort="1000" lower="${-pi*0.5}" upper="${pi*0.5}" />
+    <limit velocity="6.5" effort="1000" lower="${-pi*0.9}" upper="${pi*0.9}" />
     <dynamics damping="0.1"/>
   </joint>
@@ -194,5 +194,5 @@
     <origin xyz="0.1235 0.0 0.0" rpy="0 0 0"/>
     <axis xyz="0 -1 0"/>
-    <limit velocity="6.5" effort="1000" lower="${-pi*0.5}" upper="${pi*0.5}" />
+    <limit velocity="6.5" effort="1000" lower="${-pi*0.9}" upper="${pi*0.9}" />
     <dynamics damping="0.1"/>
   </joint>

Commit message: update description

File: open_manipulator_description/urdf/open_manipulator_chain.xacro (robot description, xacro)
@@ -1,4 +1,4 @@
 <?xml version="1.0"?>
-<!-- ROBOTIS Manipulator-X4 -->
+<!-- Open_Manipulator Chain -->
 <robot name="gazebo_open_manipulator_chain" xmlns:xacro="http://www.ros.org/wiki/xacro">
   <!-- some parameters -->
@@ -15,30 +15,4 @@
     <origin xyz="0 0 0" rpy="0 0 0"/>
     <parent link="world"/>
-    <child link="base"/>
-  </joint>
-  <!-- Base Plate -->
-  <link name="base">
-    <collision>
-      <origin xyz="0 0 0" rpy="0 0 0"/>
-      <geometry>
-        <mesh filename="package://open_manipulator_description/meshes/turtlebot3_premium.stl" scale="0.001 0.001 0.001"/>
-      </geometry>
-    </collision>
-    <visual>
-      <origin xyz="0 0 0" rpy="0 0 0"/>
-      <geometry>
-        <mesh filename="package://open_manipulator_description/meshes/turtlebot3_premium.stl" scale="0.001 0.001 0.001"/>
-      </geometry>
-      <material name="grey"/>
-    </visual>
-    <inertial>
-      <origin xyz="0 0 0" rpy="0 0 0"/>
-      <mass value="1.0"/>
-      <inertia ixx="1.0" ixy="0.0" ixz="0" iyy="1.0" iyz="0.0" izz="1.0" />
-    </inertial>
-  </link>
-  <!-- Base fixed joint -->
-  <joint name="base_fixed" type="fixed">
-    <parent link="base"/>
     <child link="link1"/>
   </joint>
@@ -46,5 +20,5 @@
   <link name="link1">
     <collision>
-      <origin xyz="0.036 0 0.103" rpy="0 0 0"/>
+      <origin xyz="0.0 0.0 0.0" rpy="0 0 0"/>
       <geometry>
         <mesh filename="package://open_manipulator_description/meshes/chain_link1.stl" scale="0.001 0.001 0.001"/>
@@ -52,5 +26,5 @@
     </collision>
     <visual>
-      <origin xyz="0.036 0 0.103" rpy="0 0 0"/>
+      <origin xyz="0.0 0.0 0.0" rpy="0 0 0"/>
       <geometry>
         <mesh filename="package://open_manipulator_description/meshes/chain_link1.stl" scale="0.001 0.001 0.001"/>
@@ -69,5 +43,5 @@
     <parent link="link1"/>
     <child link="link2"/>
-    <origin xyz="0.048 0.0 0.137" rpy="0 0 0"/>
+    <origin xyz="0.012 0.0 0.036" rpy="0 0 0"/>
     <axis xyz="0 0 1"/>
     <limit velocity="6.5" effort="1000" lower="${-pi*0.9}" upper="${pi*0.9}" />
@@ -84,8 +58,8 @@
     </actuator>
   </transmission>
-  <!-- Link 2 -->
+  <!--  Link 2 -->
   <link name="link2">
     <collision>
-      <origin xyz="0 0 0" rpy="0 0 0"/>
+      <origin xyz="0.0 0.0 0.0" rpy="0 0 0"/>
       <geometry>
         <mesh filename="package://open_manipulator_description/meshes/chain_link2.stl" scale="0.001 0.001 0.001"/>
@@ -93,5 +67,5 @@
     </collision>
     <visual>
-      <origin xyz="0 0 0" rpy="0 0 0"/>
+      <origin xyz="0.0 0.0 0.040" rpy="0 0 0"/>
       <geometry>
         <mesh filename="package://open_manipulator_description/meshes/chain_link2.stl" scale="0.001 0.001 0.001"/>
@@ -106,11 +80,11 @@
     </inertial>
   </link>
-  <!-- Joint 2 -->
+  <!--  Joint 2 -->
   <joint name="joint2" type="revolute">
     <parent link="link2"/>
     <child link="link3"/>
-    <origin xyz="0.0 0.0 0.04235" rpy="0 0 0"/>
-    <axis xyz="0 -1 0"/>
-    <limit velocity="6.5" effort="1000" lower="${-pi*0.5}" upper="${pi*0.5}" />
+    <origin xyz="0.0 0.0 0.040" rpy="0 0 0"/>
+    <axis xyz="0 -1 0"/>
+    <limit velocity="6.5" effort="1000" lower="${-pi*0.9}" upper="${pi*0.9}" />
     <dynamics damping="0.1"/>
   </joint>
@@ -125,8 +99,8 @@
     </actuator>
   </transmission>
-  <!-- Link 3 -->
+  <!--  Link 3 -->
   <link name="link3">
     <collision>
-      <origin xyz="0 -0.020 0" rpy="0 0 0"/>
+      <origin xyz="0 0 0" rpy="0 0 0"/>
       <geometry>
         <mesh filename="package://open_manipulator_description/meshes/chain_link3.stl" scale="0.001 0.001 0.001"/>
@@ -134,5 +108,5 @@
     </collision>
     <visual>
-      <origin xyz="0 -0.020 0" rpy="0 0 0"/>
+      <origin xyz="0.022 0 0.122" rpy="0 0 0"/>
       <geometry>
         <mesh filename="package://open_manipulator_description/meshes/chain_link3.stl" scale="0.001 0.001 0.001"/>
@@ -147,11 +121,11 @@
     </inertial>
   </link>
-  <!-- Joint 3 -->
+  <!--  Joint 3 -->
   <joint name="joint3" type="revolute">
     <parent link="link3"/>
     <child link="link4"/>
-    <origin xyz="0.024 0.0 0.12165" rpy="0 0 0"/>
-    <axis xyz="0 -1 0"/>
-    <limit velocity="6.5" effort="1000" lower="${-pi*0.5}" upper="${pi*0.5}" />
+    <origin xyz="0.022 0 0.122" rpy="0 0 0"/>
+    <axis xyz="0 -1 0"/>
+    <limit velocity="6.5" effort="1000" lower="${-pi*0.9}" upper="${pi*0.9}" />
     <dynamics damping="0.1"/>
   </joint>
@@ -166,8 +140,8 @@
     </actuator>
   </transmission>
-  <!-- Link 4 -->
+  <!--  Link 4 -->
   <link name="link4">
     <collision>
-      <origin xyz="0 -0.020 0.0" rpy="0 0 0"/>
+      <origin xyz="0 0 0.0" rpy="0 0 0"/>
       <geometry>
         <mesh filename="package://open_manipulator_description/meshes/chain_link4.stl" scale="0.001 0.001 0.001"/>
@@ -175,5 +149,5 @@
     </collision>
     <visual>
-      <origin xyz="0 -0.020 0.0" rpy="0 0 0"/>
+      <origin xyz="0.124 0 0.0" rpy="0 0 0"/>
       <geometry>
         <mesh filename="package://open_manipulator_description/meshes/chain_link4.stl" scale="0.001 0.001 0.001"/>
@@ -188,11 +162,11 @@
     </inertial>
   </link>
-  <!-- Joint 4 -->
+  <!--  Joint 4 -->
   <joint name="joint4" type="revolute">
     <parent link="link4"/>
     <child link="link5"/>
-    <origin xyz="0.1235 0.0 0.0" rpy="0 0 0"/>
-    <axis xyz="0 -1 0"/>
-    <limit velocity="6.5" effort="1000" lower="${-pi*0.5}" upper="${pi*0.5}" />
+    <origin xyz="0.124 0.0 0.0" rpy="0 0 0"/>
+    <axis xyz="0 -1 0"/>
+    <limit velocity="6.5" effort="1000" lower="${-pi*0.9}" upper="${pi*0.9}" />
     <dynamics damping="0.1"/>
   </joint>
@@ -207,8 +181,8 @@
     </actuator>
   </transmission>
-  <!-- Link 5 -->
+  <!--  Link 5 -->
   <link name="link5">
     <collision>
-      <origin xyz="0 -0.020 0" rpy="0 0 0"/>
+      <origin xyz="0 0 0" rpy="0 0 0"/>
       <geometry>
         <mesh filename="package://open_manipulator_description/meshes/chain_link5.stl" scale="0.001 0.001 0.001"/>
@@ -216,5 +190,5 @@
     </collision>
     <visual>
-      <origin xyz="0 -0.020 0" rpy="0 0 0"/>
+      <origin xyz="0.065 0 0" rpy="0 0 0"/>
       <geometry>
         <mesh filename="package://open_manipulator_description/meshes/chain_link5.stl" scale="0.001 0.001 0.001"/>
@@ -229,11 +203,11 @@
     </inertial>
   </link>
-  <!-- Grip Joint -->
+  <!--  Grip joint -->
   <joint name="grip_joint" type="prismatic">
     <parent link="link5"/>
     <child link="grip_link"/>
-    <origin xyz="0.064 0.0 0.0" rpy="0 0 0"/>
+    <origin xyz="0.090 0.0 0.0" rpy="0 0 0"/>
     <axis xyz="0 1 0"/>
-    <limit velocity="6.5" effort="1000" lower="-0.01" upper="0.035" />
+    <limit velocity="6.5" effort="1000" lower="-0.035" upper="0.01" />
     <dynamics damping="0.1"/>
   </joint>
@@ -248,16 +222,16 @@
     </actuator>
   </transmission>
-  <!-- Grip Link -->
+  <!--  Grip link -->
   <link name="grip_link">
     <collision>
-      <origin xyz="-0.064 -0.020 0" rpy="0 0 0"/>
-      <geometry>
-        <mesh filename="package://open_manipulator_description/meshes/chain_link_grip1.stl" scale="0.001 0.001 0.001"/>
-      </geometry>
-    </collision>
-    <visual>
-      <origin xyz="-0.064 -0.020 0" rpy="0 0 0"/>
-      <geometry>
-        <mesh filename="package://open_manipulator_description/meshes/chain_link_grip1.stl" scale="0.001 0.001 0.001"/>
+      <origin xyz="0.0 0.0 0" rpy="0 0 0"/>
+      <geometry>
+        <mesh filename="package://open_manipulator_description/meshes/chain_link_grip_l.stl" scale="0.001 0.001 0.001"/>
+      </geometry>
+    </collision>
+    <visual>
+      <origin xyz="0.0 0.047 0" rpy="0 0 0"/>
+      <geometry>
+        <mesh filename="package://open_manipulator_description/meshes/chain_link_grip_l.stl" scale="0.001 0.001 0.001"/>
       </geometry>
       <material name="grey"/>
@@ -270,11 +244,11 @@
     </inertial>
   </link>
-  <!-- Grip Joint Sub -->
+  <!--  Grip joint sub -->
   <joint name="grip_joint_sub" type="prismatic">
     <parent link="link5"/>
     <child link="grip_link_sub"/>
-    <origin xyz="0.064 0.0 0" rpy="0 0 0"/>
-    <axis xyz="0 -1 0"/>
-    <limit velocity="6.5" effort="1000" lower="-0.01" upper="0.035" />
+    <origin xyz="0.090 0.0 0" rpy="0 0 0"/>
+    <axis xyz="0 -1 0"/>
+    <limit velocity="6.5" effort="1000" lower="-0.035" upper="0.01" />
     <dynamics damping="0.1"/>
   </joint>
@@ -289,16 +263,16 @@
     </actuator>
   </transmission>
-  <!-- Grip Link Sub -->
+  <!--  Grip link sub -->
   <link name="grip_link_sub">
     <collision>
-      <origin xyz="-0.064 -0.020 0" rpy="0 0 0"/>
-      <geometry>
-        <mesh filename="package://open_manipulator_description/meshes/chain_link_grip2.stl" scale="0.001 0.001 0.001"/>
-      </geometry>
-    </collision>
-    <visual>
-      <origin xyz="-0.064 -0.020 0" rpy="0 0 0"/>
-      <geometry>
-        <mesh filename="package://open_manipulator_description/meshes/chain_link_grip2.stl" scale="0.001 0.001 0.001"/>
+      <origin xyz="0 0 0" rpy="0 0 0"/>
+      <geometry>
+        <mesh filename="package://open_manipulator_description/meshes/chain_link_grip_r.stl" scale="0.001 0.001 0.001"/>
+      </geometry>
+    </collision>
+    <visual>
+      <origin xyz="0 -0.047 0" rpy="0 0 0"/>
+      <geometry>
+        <mesh filename="package://open_manipulator_description/meshes/chain_link_grip_r.stl" scale="0.001 0.001 0.001"/>
       </geometry>
       <material name="grey"/>

Commit message: update moveit

File: open_manipulator_description/urdf/open_manipulator_chain.xacro (robot description, xacro)
@@ -5,5 +5,5 @@
   <xacro:property name="pi" value="3.141592654" />
   <!-- Import all Gazebo-customization elements, including Gazebo colors -->
-  <xacro:include filename="$(find open_manipulator_description)/urdf/open_manipulator_chain.gazebo" />
+  <xacro:include filename="$(find open_manipulator_description)/urdf/open_manipulator_chain.gazebo.xacro" />
   <!-- Import Rviz colors -->
   <xacro:include filename="$(find open_manipulator_description)/urdf/materials.xacro" />
@@ -33,8 +33,9 @@
     </visual>
     <inertial>
-      <origin xyz="0.00025 0.00000 0.01780" rpy="0 0 0"/>
-      <mass value="0.087"/>
-      <inertia ixx="1.0" ixy="0.0" ixz="0.0" iyy="1.0" iyz="0.0" izz="1.0" />
-      <inertia ixx="0.00001378" ixy="0.0" ixz="-0.00000025" iyy="0.00002381" iyz="0.0" izz="0.00002107" />
+      <origin xyz="0 0 0" />
+      <mass value="0.01" />
+      <inertia ixx="0.001" ixy="0.0" ixz="0.0"
+               iyy="0.001" iyz="0.0"
+               izz="0.001" />
     </inertial>
   </link>
@@ -61,5 +62,5 @@
   <link name="link2">
     <collision>
-      <origin xyz="0.0 0.0 0.0" rpy="0 0 0"/>
+      <origin xyz="0.0 0.0 0.040" rpy="0 0 0"/>
       <geometry>
         <mesh filename="package://open_manipulator_description/meshes/chain_link2.stl" scale="0.001 0.001 0.001"/>
@@ -74,8 +75,9 @@
     </visual>
     <inertial>
-      <origin xyz="0.00002 -0.00045 0.03293" rpy="0 0 0"/>
-      <mass value="0.117"/>
-      <inertia ixx="1.0" ixy="0.0" ixz="0.0" iyy="1.0" iyz="0.0" izz="1.0" />
-      <inertia ixx="0.00004110" ixy="0.0" ixz="-0.00000025" iyy="0.00002381" iyz="0.0" izz="0.00002107" />
+      <origin xyz="0 0 0" />
+      <mass value="0.01" />
+      <inertia ixx="0.001" ixy="0.0" ixz="0.0"
+               iyy="0.001" iyz="0.0"
+               izz="0.001" />
     </inertial>
   </link>
@@ -102,5 +104,5 @@
   <link name="link3">
     <collision>
-      <origin xyz="0 0 0" rpy="0 0 0"/>
+      <origin xyz="0.022 0 0.122" rpy="0 0 0"/>
       <geometry>
         <mesh filename="package://open_manipulator_description/meshes/chain_link3.stl" scale="0.001 0.001 0.001"/>
@@ -115,8 +117,9 @@
     </visual>
     <inertial>
-      <origin xyz="0.00966 -0.00034 0.11795" rpy="0 0 0"/>
-      <mass value="0.156"/>
-      <inertia ixx="1.0" ixy="0.0" ixz="0.0" iyy="1.0" iyz="0.0" izz="1.0" />
-      <inertia ixx="0.00041624" ixy="0.00000017" ixz="-0.00004492" iyy="0.00042758" iyz="0.00000159" izz="0.00005317" />
+      <origin xyz="0 0 0" />
+      <mass value="0.01" />
+      <inertia ixx="0.001" ixy="0.0" ixz="0.0"
+               iyy="0.001" iyz="0.0"
+               izz="0.001" />
     </inertial>
   </link>
@@ -143,5 +146,5 @@
   <link name="link4">
     <collision>
-      <origin xyz="0 0 0.0" rpy="0 0 0"/>
+      <origin xyz="0.124 0 0.0" rpy="0 0 0"/>
       <geometry>
         <mesh filename="package://open_manipulator_description/meshes/chain_link4.stl" scale="0.001 0.001 0.001"/>
@@ -156,8 +159,9 @@
     </visual>
     <inertial>
-      <origin xyz="0.11076 -0.00035 0.00050" rpy="0 0 0"/>
-      <mass value="0.149"/>
-      <inertia ixx="1.0" ixy="0.0" ixz="0.0" iyy="1.0" iyz="0.0" izz="1.0" />
-      <inertia ixx="0.00003083" ixy="0.00000147" ixz="-0.00000222" iyy="0.00036703" iyz="-0.00000003" izz="0.00037667" />
+      <origin xyz="0 0 0" />
+      <mass value="0.01" />
+      <inertia ixx="0.001" ixy="0.0" ixz="0.0"
+               iyy="0.001" iyz="0.0"
+               izz="0.001" />
     </inertial>
   </link>
@@ -184,5 +188,5 @@
   <link name="link5">
     <collision>
-      <origin xyz="0 0 0" rpy="0 0 0"/>
+      <origin xyz="0.046 0 0" rpy="0 0 0"/>
       <geometry>
         <mesh filename="package://open_manipulator_description/meshes/chain_link5.stl" scale="0.001 0.001 0.001"/>
@@ -190,5 +194,5 @@
     </collision>
     <visual>
-      <origin xyz="0.065 0 0" rpy="0 0 0"/>
+      <origin xyz="0.046 0 0" rpy="0 0 0"/>
       <geometry>
         <mesh filename="package://open_manipulator_description/meshes/chain_link5.stl" scale="0.001 0.001 0.001"/>
@@ -197,8 +201,32 @@
     </visual>
     <inertial>
-      <origin xyz="0.03767 0.00262 -0.00043" rpy="0 0 0"/>
-      <mass value="0.124"/>
-      <inertia ixx="1.0" ixy="0.0" ixz="0.0" iyy="1.0" iyz="0.0" izz="1.0" />
-      <inertia ixx="0.00004822" ixy="-0.00000148" ixz="0.00000024" iyy="0.00004342" iyz="0.00000014" izz="0.00005784" />
+      <origin xyz="0 0 0" />
+      <mass value="0.01" />
+      <inertia ixx="0.001" ixy="0.0" ixz="0.0"
+               iyy="0.001" iyz="0.0"
+               izz="0.001" />
+    </inertial>
+  </link>
+  <!--  Grip link -->
+  <link name="grip_link">
+    <collision>
+      <origin xyz="0.0 0.047 0" rpy="0 0 0"/>
+      <geometry>
+        <mesh filename="package://open_manipulator_description/meshes/chain_link_grip_l.stl" scale="0.001 0.001 0.001"/>
+      </geometry>
+    </collision>
+    <visual>
+      <origin xyz="0.0 0.047 0" rpy="0 0 0"/>
+      <geometry>
+        <mesh filename="package://open_manipulator_description/meshes/chain_link_grip_l.stl" scale="0.001 0.001 0.001"/>
+      </geometry>
+      <material name="grey"/>
+    </visual>
+    <inertial>
+      <origin xyz="0 0 0" />
+      <mass value="0.01" />
+      <inertia ixx="0.001" ixy="0.0" ixz="0.0"
+               iyy="0.001" iyz="0.0"
+               izz="0.001" />
     </inertial>
   </link>
@@ -207,5 +235,5 @@
     <parent link="link5"/>
     <child link="grip_link"/>
-    <origin xyz="0.090 0.0 0.0" rpy="0 0 0"/>
+    <origin xyz="0.071 0.0 0.0" rpy="0 0 0"/>
     <axis xyz="0 1 0"/>
     <limit velocity="6.5" effort="1000" lower="-0.035" upper="0.01" />
@@ -222,24 +250,25 @@
     </actuator>
   </transmission>
-  <!--  Grip link -->
-  <link name="grip_link">
-    <collision>
-      <origin xyz="0.0 0.0 0" rpy="0 0 0"/>
-      <geometry>
-        <mesh filename="package://open_manipulator_description/meshes/chain_link_grip_l.stl" scale="0.001 0.001 0.001"/>
-      </geometry>
-    </collision>
-    <visual>
-      <origin xyz="0.0 0.047 0" rpy="0 0 0"/>
-      <geometry>
-        <mesh filename="package://open_manipulator_description/meshes/chain_link_grip_l.stl" scale="0.001 0.001 0.001"/>
-      </geometry>
-      <material name="grey"/>
-    </visual>
-    <inertial>
-      <origin xyz="0.02666 -0.00910 -0.02300" rpy="0 0 0"/>
-      <mass value="0.06721"/>
-      <inertia ixx="1.0" ixy="0.0" ixz="0.0" iyy="1.0" iyz="0.0" izz="1.0" />
-      <inertia ixx="0.00002875" ixy="-0.00000593" ixz="-0.00000006" iyy="0.00006646" iyz="-0.00000009" izz="0.00005474" />
+  <!--  Grip link sub -->
+  <link name="grip_link_sub">
+    <collision>
+      <origin xyz="0 -0.047 0" rpy="0 0 0"/>
+      <geometry>
+        <mesh filename="package://open_manipulator_description/meshes/chain_link_grip_r.stl" scale="0.001 0.001 0.001"/>
+      </geometry>
+    </collision>
+    <visual>
+      <origin xyz="0 -0.047 0" rpy="0 0 0"/>
+      <geometry>
+        <mesh filename="package://open_manipulator_description/meshes/chain_link_grip_r.stl" scale="0.001 0.001 0.001"/>
+      </geometry>
+      <material name="grey"/>
+    </visual>
+    <inertial>
+      <origin xyz="0 0 0" />
+      <mass value="0.01" />
+      <inertia ixx="0.001" ixy="0.0" ixz="0.0"
+               iyy="0.001" iyz="0.0"
+               izz="0.001" />
     </inertial>
   </link>
@@ -248,5 +277,5 @@
     <parent link="link5"/>
     <child link="grip_link_sub"/>
-    <origin xyz="0.090 0.0 0" rpy="0 0 0"/>
+    <origin xyz="0.071 0.0 0" rpy="0 0 0"/>
     <axis xyz="0 -1 0"/>
     <limit velocity="6.5" effort="1000" lower="-0.035" upper="0.01" />
@@ -263,25 +292,3 @@
     </actuator>
   </transmission>
-  <!--  Grip link sub -->
-  <link name="grip_link_sub">
-    <collision>
-      <origin xyz="0 0 0" rpy="0 0 0"/>
-      <geometry>
-        <mesh filename="package://open_manipulator_description/meshes/chain_link_grip_r.stl" scale="0.001 0.001 0.001"/>
-      </geometry>
-    </collision>
-    <visual>
-      <origin xyz="0 -0.047 0" rpy="0 0 0"/>
-      <geometry>
-        <mesh filename="package://open_manipulator_description/meshes/chain_link_grip_r.stl" scale="0.001 0.001 0.001"/>
-      </geometry>
-      <material name="grey"/>
-    </visual>
-    <inertial>
-      <origin xyz="0.02666 0.00910 -0.02300" rpy="0 0 0"/>
-      <mass value="0.06721"/>
-      <inertia ixx="1.0" ixy="0.0" ixz="0.0" iyy="1.0" iyz="0.0" izz="1.0" />
-      <inertia ixx="0.00002875" ixy="0.00000593" ixz="0.00000006" iyy="0.00006646" iyz="-0.00000009" izz="0.00005474" />
-    </inertial>
-  </link>
 </robot>

Commit message: modify line

File: open_manipulator_description/urdf/open_manipulator_chain.xacro (robot description, xacro)
@@ -47,5 +47,4 @@
     <axis xyz="0 0 1"/>
     <limit velocity="6.5" effort="1000" lower="${-pi*0.9}" upper="${pi*0.9}" />
-    <dynamics damping="0.1"/>
   </joint>
   <!--  Link 2 -->
@@ -79,5 +78,4 @@
     <axis xyz="0 -1 0"/>
     <limit velocity="6.5" effort="1000" lower="${-pi*0.9}" upper="${pi*0.9}" />
-    <dynamics damping="0.1"/>
   </joint>
   <!--  Link 3 -->
@@ -111,5 +109,4 @@
     <axis xyz="0 -1 0"/>
     <limit velocity="6.5" effort="1000" lower="${-pi*0.9}" upper="${pi*0.9}" />
-    <dynamics damping="0.1"/>
   </joint>
   <!--  Link 4 -->
@@ -143,5 +140,4 @@
     <axis xyz="0 -1 0"/>
     <limit velocity="6.5" effort="1000" lower="${-pi*0.9}" upper="${pi*0.9}" />
-    <dynamics damping="0.1"/>
   </joint>
   <!--  Link 5 -->
@@ -198,5 +194,4 @@
     <axis xyz="0 1 0"/>
     <limit velocity="6.5" effort="1000" lower="-0.035" upper="0.01" />
-    <dynamics damping="0.1"/>
   </joint>
   <!--  Grip link sub -->
@@ -230,5 +225,4 @@
     <axis xyz="0 -1 0"/>
     <limit velocity="6.5" effort="1000" lower="-0.035" upper="0.01" />
-    <dynamics damping="0.1"/>
   </joint>
 </robot>

Commit message: modified gripper topic

File: open_manipulator_description/urdf/open_manipulator_chain.xacro (robot description, xacro)
@@ -236,6 +236,6 @@
     <child link="grip_link"/>
     <origin xyz="0.071 0.0 0.0" rpy="0 0 0"/>
-    <axis xyz="0 1 0"/>
-    <limit velocity="6.5" effort="1000" lower="-0.035" upper="0.01" />
+    <axis xyz="0 -1 0"/>
+    <limit velocity="6.5" effort="1000" lower="-0.01" upper="0.035" />
   </joint>
   <!-- Transmisstion 5 -->
@@ -278,6 +278,6 @@
     <child link="grip_link_sub"/>
     <origin xyz="0.071 0.0 0" rpy="0 0 0"/>
-    <axis xyz="0 -1 0"/>
-    <limit velocity="6.5" effort="1000" lower="-0.035" upper="0.01" />
+    <axis xyz="0 1 0"/>
+    <limit velocity="6.5" effort="1000" lower="-0.01" upper="0.035" />
   </joint>
   <!-- Transmisstion 6 -->
