Commit message: modified collision geometry

File: open_manipulator_description/urdf/open_manipulator_chain.xacro (robot description, xacro)
@@ -19,17 +19,17 @@
   <!-- Link 1 -->
   <link name="link1">
-    <collision>
+    <visual>
       <origin xyz="0.0 0.0 0.0" rpy="0 0 0"/>
       <geometry>
         <mesh filename="package://open_manipulator_description/meshes/chain_link1.stl" scale="0.001 0.001 0.001"/>
       </geometry>
-    </collision>
-    <visual>
-      <origin xyz="0.0 0.0 0.0" rpy="0 0 0"/>
-      <geometry>
-        <mesh filename="package://open_manipulator_description/meshes/chain_link1.stl" scale="0.001 0.001 0.001"/>
-      </geometry>
-      <material name="grey"/>
-    </visual>
+      <material name="grey"/>
+    </visual>
+    <collision>
+      <origin xyz="0.0 0.0 0.017" rpy="0 0 0"/>
+      <geometry>
+        <box size="0.0475 0.0295 0.0340"/>
+      </geometry>
+    </collision>
     <inertial>
       <origin xyz="0 0 0" />
@@ -61,17 +61,17 @@
   <!--  Link 2 -->
   <link name="link2">
-    <collision>
+    <visual>
       <origin xyz="0.0 0.0 0.040" rpy="0 0 0"/>
       <geometry>
         <mesh filename="package://open_manipulator_description/meshes/chain_link2.stl" scale="0.001 0.001 0.001"/>
       </geometry>
-    </collision>
-    <visual>
-      <origin xyz="0.0 0.0 0.040" rpy="0 0 0"/>
-      <geometry>
-        <mesh filename="package://open_manipulator_description/meshes/chain_link2.stl" scale="0.001 0.001 0.001"/>
-      </geometry>
-      <material name="grey"/>
-    </visual>
+      <material name="grey"/>
+    </visual>
+    <collision>
+      <origin xyz="0.0 0.0 0.030" rpy="0 0 0"/>
+      <geometry>
+        <box size="0.0355 0.0550 0.0515"/>
+      </geometry>
+    </collision>
     <inertial>
       <origin xyz="0 0 0" />
@@ -87,6 +87,6 @@
     <child link="link3"/>
     <origin xyz="0.0 0.0 0.040" rpy="0 0 0"/>
-    <axis xyz="0 -1 0"/>
-    <limit velocity="6.5" effort="1000" lower="${-pi*0.9}" upper="${pi*0.9}" />
+    <axis xyz="0 1 0"/>
+    <limit velocity="6.5" effort="1000" lower="${-pi*0.5}" upper="${pi*0.5}" />
   </joint>
   <!-- Transmission 2 -->
@@ -103,17 +103,17 @@
   <!--  Link 3 -->
   <link name="link3">
-    <collision>
+    <visual>
       <origin xyz="0.022 0 0.122" rpy="0 0 0"/>
       <geometry>
         <mesh filename="package://open_manipulator_description/meshes/chain_link3.stl" scale="0.001 0.001 0.001"/>
       </geometry>
-    </collision>
-    <visual>
-      <origin xyz="0.022 0 0.122" rpy="0 0 0"/>
-      <geometry>
-        <mesh filename="package://open_manipulator_description/meshes/chain_link3.stl" scale="0.001 0.001 0.001"/>
-      </geometry>
-      <material name="grey"/>
-    </visual>
+      <material name="grey"/>
+    </visual>
+    <collision>
+      <origin xyz="0.0 0 0.085" rpy="0 0 0"/>
+      <geometry>
+        <box size="0.030 0.055 0.120"/>
+      </geometry>
+    </collision>
     <inertial>
       <origin xyz="0 0 0" />
@@ -129,6 +129,6 @@
     <child link="link4"/>
     <origin xyz="0.022 0 0.122" rpy="0 0 0"/>
-    <axis xyz="0 -1 0"/>
-    <limit velocity="6.5" effort="1000" lower="${-pi*0.9}" upper="${pi*0.9}" />
+    <axis xyz="0 1 0"/>
+    <limit velocity="6.5" effort="1000" lower="${-pi*0.5}" upper="${pi*0.4}" />
   </joint>
   <!-- Transmission 3 -->
@@ -145,17 +145,17 @@
   <!--  Link 4 -->
   <link name="link4">
-    <collision>
+    <visual>
       <origin xyz="0.124 0 0.0" rpy="0 0 0"/>
       <geometry>
         <mesh filename="package://open_manipulator_description/meshes/chain_link4.stl" scale="0.001 0.001 0.001"/>
       </geometry>
-    </collision>
-    <visual>
-      <origin xyz="0.124 0 0.0" rpy="0 0 0"/>
-      <geometry>
-        <mesh filename="package://open_manipulator_description/meshes/chain_link4.stl" scale="0.001 0.001 0.001"/>
-      </geometry>
-      <material name="grey"/>
-    </visual>
+      <material name="grey"/>
+    </visual>
+    <collision>
+      <origin xyz="0.080 0 0.0" rpy="0 0 0"/>
+      <geometry>
+        <box size="0.110 0.055 0.035"/>
+      </geometry>
+    </collision>
     <inertial>
       <origin xyz="0 0 0" />
@@ -171,6 +171,6 @@
     <child link="link5"/>
     <origin xyz="0.124 0.0 0.0" rpy="0 0 0"/>
-    <axis xyz="0 -1 0"/>
-    <limit velocity="6.5" effort="1000" lower="${-pi*0.9}" upper="${pi*0.9}" />
+    <axis xyz="0 1 0"/>
+    <limit velocity="6.5" effort="1000" lower="${-pi*0.4}" upper="${pi*0.5}" />
   </joint>
   <!-- Transmission 4 -->
@@ -187,17 +187,17 @@
   <!--  Link 5 -->
   <link name="link5">
-    <collision>
+    <visual>
       <origin xyz="0.046 0 0" rpy="0 0 0"/>
       <geometry>
         <mesh filename="package://open_manipulator_description/meshes/chain_link5.stl" scale="0.001 0.001 0.001"/>
       </geometry>
-    </collision>
-    <visual>
-      <origin xyz="0.046 0 0" rpy="0 0 0"/>
-      <geometry>
-        <mesh filename="package://open_manipulator_description/meshes/chain_link5.stl" scale="0.001 0.001 0.001"/>
-      </geometry>
-      <material name="grey"/>
-    </visual>
+      <material name="grey"/>
+    </visual>
+    <collision>
+      <origin xyz="0.050 0 0.005" rpy="0 0 0"/>
+      <geometry>
+        <box size="0.040 0.120 0.0650"/>
+      </geometry>
+    </collision>
     <inertial>
       <origin xyz="0 0 0" />
@@ -210,17 +210,17 @@
   <!--  Grip link -->
   <link name="grip_link">
-    <collision>
+    <visual>
       <origin xyz="0.0 0.047 0" rpy="0 0 0"/>
       <geometry>
         <mesh filename="package://open_manipulator_description/meshes/chain_link_grip_l.stl" scale="0.001 0.001 0.001"/>
       </geometry>
-    </collision>
-    <visual>
-      <origin xyz="0.0 0.047 0" rpy="0 0 0"/>
-      <geometry>
-        <mesh filename="package://open_manipulator_description/meshes/chain_link_grip_l.stl" scale="0.001 0.001 0.001"/>
-      </geometry>
-      <material name="grey"/>
-    </visual>
+      <material name="grey"/>
+    </visual>
+    <collision>
+      <origin xyz="0.040 0.047 0" rpy="0 0 0"/>
+      <geometry>
+        <box size="0.060 0.025 0.070"/>
+      </geometry>
+    </collision>
     <inertial>
       <origin xyz="0 0 0" />
@@ -252,17 +252,17 @@
   <!--  Grip link sub -->
   <link name="grip_link_sub">
-    <collision>
+    <visual>
       <origin xyz="0 -0.047 0" rpy="0 0 0"/>
       <geometry>
         <mesh filename="package://open_manipulator_description/meshes/chain_link_grip_r.stl" scale="0.001 0.001 0.001"/>
       </geometry>
-    </collision>
-    <visual>
-      <origin xyz="0 -0.047 0" rpy="0 0 0"/>
-      <geometry>
-        <mesh filename="package://open_manipulator_description/meshes/chain_link_grip_r.stl" scale="0.001 0.001 0.001"/>
-      </geometry>
-      <material name="grey"/>
-    </visual>
+      <material name="grey"/>
+    </visual>
+    <collision>
+      <origin xyz="0.040 -0.047 0" rpy="0 0 0"/>
+      <geometry>
+        <box size="0.060 0.025 0.070"/>
+      </geometry>
+    </collision>
     <inertial>
       <origin xyz="0 0 0" />

File: open_manipulator_with_tb3/urdf/open_manipulator_chain_with_tb3.xacro (robot description, xacro)
@@ -14,17 +14,17 @@
   <!-- Link 1 -->
   <link name="link1">
-    <collision>
-      <origin xyz="0.0 0 0.0" rpy="0 0 0"/>
-      <geometry>
-        <mesh filename="package://open_manipulator_with_tb3/meshes/chain_link1.stl" scale="0.001 0.001 0.001"/>
-      </geometry>
-    </collision>
-    <visual>
-      <origin xyz="0.0 0 0.0" rpy="0 0 0"/>
-      <geometry>
-        <mesh filename="package://open_manipulator_with_tb3/meshes/chain_link1.stl" scale="0.001 0.001 0.001"/>
-      </geometry>
-      <material name="grey"/>
-    </visual>
+    <visual>
+      <origin xyz="0.0 0.0 0.0" rpy="0 0 0"/>
+      <geometry>
+        <mesh filename="package://open_manipulator_description/meshes/chain_link1.stl" scale="0.001 0.001 0.001"/>
+      </geometry>
+      <material name="grey"/>
+    </visual>
+    <collision>
+      <origin xyz="0.0 0.0 0.017" rpy="0 0 0"/>
+      <geometry>
+        <box size="0.0475 0.0295 0.0340"/>
+      </geometry>
+    </collision>
     <inertial>
       <origin xyz="0 0 0" />
@@ -43,5 +43,5 @@
     <limit velocity="6.5" effort="1000" lower="${-pi*0.9}" upper="${pi*0.9}" />
   </joint>
-  <!-- Transmisstion 1 -->
+  <!-- Transmission 1 -->
   <transmission name="tran1">
     <type>transmission_interface/SimpleTransmission</type>
@@ -56,17 +56,17 @@
   <!--  Link 2 -->
   <link name="link2">
-    <collision>
+    <visual>
       <origin xyz="0.0 0.0 0.040" rpy="0 0 0"/>
       <geometry>
-        <mesh filename="package://open_manipulator_with_tb3/meshes/chain_link2.stl" scale="0.001 0.001 0.001"/>
-      </geometry>
-    </collision>
-    <visual>
-      <origin xyz="0.0 0.0 0.040" rpy="0 0 0"/>
-      <geometry>
-        <mesh filename="package://open_manipulator_with_tb3/meshes/chain_link2.stl" scale="0.001 0.001 0.001"/>
-      </geometry>
-      <material name="grey"/>
-    </visual>
+        <mesh filename="package://open_manipulator_description/meshes/chain_link2.stl" scale="0.001 0.001 0.001"/>
+      </geometry>
+      <material name="grey"/>
+    </visual>
+    <collision>
+      <origin xyz="0.0 0.0 0.030" rpy="0 0 0"/>
+      <geometry>
+        <box size="0.0355 0.0550 0.0515"/>
+      </geometry>
+    </collision>
     <inertial>
       <origin xyz="0 0 0" />
@@ -82,8 +82,8 @@
     <child link="link3"/>
     <origin xyz="0.0 0.0 0.040" rpy="0 0 0"/>
-    <axis xyz="0 -1 0"/>
-    <limit velocity="6.5" effort="1000" lower="${-pi*0.9}" upper="${pi*0.9}" />
-  </joint>
-  <!-- Transmisstion 2 -->
+    <axis xyz="0 1 0"/>
+    <limit velocity="6.5" effort="1000" lower="${-pi*0.5}" upper="${pi*0.5}" />
+  </joint>
+  <!-- Transmission 2 -->
   <transmission name="tran2">
     <type>transmission_interface/SimpleTransmission</type>
@@ -98,17 +98,17 @@
   <!--  Link 3 -->
   <link name="link3">
-    <collision>
+    <visual>
       <origin xyz="0.022 0 0.122" rpy="0 0 0"/>
       <geometry>
-        <mesh filename="package://open_manipulator_with_tb3/meshes/chain_link3.stl" scale="0.001 0.001 0.001"/>
-      </geometry>
-    </collision>
-    <visual>
-      <origin xyz="0.022 0 0.122" rpy="0 0 0"/>
-      <geometry>
-        <mesh filename="package://open_manipulator_with_tb3/meshes/chain_link3.stl" scale="0.001 0.001 0.001"/>
-      </geometry>
-      <material name="grey"/>
-    </visual>
+        <mesh filename="package://open_manipulator_description/meshes/chain_link3.stl" scale="0.001 0.001 0.001"/>
+      </geometry>
+      <material name="grey"/>
+    </visual>
+    <collision>
+      <origin xyz="0.0 0 0.085" rpy="0 0 0"/>
+      <geometry>
+        <box size="0.030 0.055 0.120"/>
+      </geometry>
+    </collision>
     <inertial>
       <origin xyz="0 0 0" />
@@ -124,8 +124,8 @@
     <child link="link4"/>
     <origin xyz="0.022 0 0.122" rpy="0 0 0"/>
-    <axis xyz="0 -1 0"/>
-    <limit velocity="6.5" effort="1000" lower="${-pi*0.9}" upper="${pi*0.9}" />
-  </joint>
-  <!-- Transmisstion 3 -->
+    <axis xyz="0 1 0"/>
+    <limit velocity="6.5" effort="1000" lower="${-pi*0.5}" upper="${pi*0.4}" />
+  </joint>
+  <!-- Transmission 3 -->
   <transmission name="tran3">
     <type>transmission_interface/SimpleTransmission</type>
@@ -140,17 +140,17 @@
   <!--  Link 4 -->
   <link name="link4">
-    <collision>
+    <visual>
       <origin xyz="0.124 0 0.0" rpy="0 0 0"/>
       <geometry>
-        <mesh filename="package://open_manipulator_with_tb3/meshes/chain_link4.stl" scale="0.001 0.001 0.001"/>
-      </geometry>
-    </collision>
-    <visual>
-      <origin xyz="0.124 0 0.0" rpy="0 0 0"/>
-      <geometry>
-        <mesh filename="package://open_manipulator_with_tb3/meshes/chain_link4.stl" scale="0.001 0.001 0.001"/>
-      </geometry>
-      <material name="grey"/>
-    </visual>
+        <mesh filename="package://open_manipulator_description/meshes/chain_link4.stl" scale="0.001 0.001 0.001"/>
+      </geometry>
+      <material name="grey"/>
+    </visual>
+    <collision>
+      <origin xyz="0.080 0 0.0" rpy="0 0 0"/>
+      <geometry>
+        <box size="0.110 0.055 0.035"/>
+      </geometry>
+    </collision>
     <inertial>
       <origin xyz="0 0 0" />
@@ -166,8 +166,8 @@
     <child link="link5"/>
     <origin xyz="0.124 0.0 0.0" rpy="0 0 0"/>
-    <axis xyz="0 -1 0"/>
-    <limit velocity="6.5" effort="1000" lower="${-pi*0.9}" upper="${pi*0.9}" />
-  </joint>
-  <!-- Transmisstion 4 -->
+    <axis xyz="0 1 0"/>
+    <limit velocity="6.5" effort="1000" lower="${-pi*0.4}" upper="${pi*0.5}" />
+  </joint>
+  <!-- Transmission 4 -->
   <transmission name="tran4">
     <type>transmission_interface/SimpleTransmission</type>
@@ -182,17 +182,17 @@
   <!--  Link 5 -->
   <link name="link5">
-    <collision>
+    <visual>
       <origin xyz="0.046 0 0" rpy="0 0 0"/>
       <geometry>
-        <mesh filename="package://open_manipulator_with_tb3/meshes/chain_link5.stl" scale="0.001 0.001 0.001"/>
-      </geometry>
-    </collision>
-    <visual>
-      <origin xyz="0.046 0 0" rpy="0 0 0"/>
-      <geometry>
-        <mesh filename="package://open_manipulator_with_tb3/meshes/chain_link5.stl" scale="0.001 0.001 0.001"/>
-      </geometry>
-      <material name="grey"/>
-    </visual>
+        <mesh filename="package://open_manipulator_description/meshes/chain_link5.stl" scale="0.001 0.001 0.001"/>
+      </geometry>
+      <material name="grey"/>
+    </visual>
+    <collision>
+      <origin xyz="0.050 0 0.005" rpy="0 0 0"/>
+      <geometry>
+        <box size="0.040 0.120 0.0650"/>
+      </geometry>
+    </collision>
     <inertial>
       <origin xyz="0 0 0" />
@@ -205,17 +205,17 @@
   <!--  Grip link -->
   <link name="grip_link">
-    <collision>
+    <visual>
       <origin xyz="0.0 0.047 0" rpy="0 0 0"/>
       <geometry>
-        <mesh filename="package://open_manipulator_with_tb3/meshes/chain_link_grip_l.stl" scale="0.001 0.001 0.001"/>
-      </geometry>
-    </collision>
-    <visual>
-      <origin xyz="0.0 0.047 0" rpy="0 0 0"/>
-      <geometry>
-        <mesh filename="package://open_manipulator_with_tb3/meshes/chain_link_grip_l.stl" scale="0.001 0.001 0.001"/>
-      </geometry>
-      <material name="grey"/>
-    </visual>
+        <mesh filename="package://open_manipulator_description/meshes/chain_link_grip_l.stl" scale="0.001 0.001 0.001"/>
+      </geometry>
+      <material name="grey"/>
+    </visual>
+    <collision>
+      <origin xyz="0.040 0.047 0" rpy="0 0 0"/>
+      <geometry>
+        <box size="0.060 0.025 0.070"/>
+      </geometry>
+    </collision>
     <inertial>
       <origin xyz="0 0 0" />
@@ -234,5 +234,5 @@
     <limit velocity="6.5" effort="1000" lower="-0.01" upper="0.035" />
   </joint>
-  <!-- Transmisstion 5 -->
+  <!-- Transmission 5 -->
   <transmission name="tran5">
     <type>transmission_interface/SimpleTransmission</type>
@@ -247,17 +247,17 @@
   <!--  Grip link sub -->
   <link name="grip_link_sub">
-    <collision>
+    <visual>
       <origin xyz="0 -0.047 0" rpy="0 0 0"/>
       <geometry>
-        <mesh filename="package://open_manipulator_with_tb3/meshes/chain_link_grip_r.stl" scale="0.001 0.001 0.001"/>
-      </geometry>
-    </collision>
-    <visual>
-      <origin xyz="0 -0.047 0" rpy="0 0 0"/>
-      <geometry>
-        <mesh filename="package://open_manipulator_with_tb3/meshes/chain_link_grip_r.stl" scale="0.001 0.001 0.001"/>
-      </geometry>
-      <material name="grey"/>
-    </visual>
+        <mesh filename="package://open_manipulator_description/meshes/chain_link_grip_r.stl" scale="0.001 0.001 0.001"/>
+      </geometry>
+      <material name="grey"/>
+    </visual>
+    <collision>
+      <origin xyz="0.040 -0.047 0" rpy="0 0 0"/>
+      <geometry>
+        <box size="0.060 0.025 0.070"/>
+      </geometry>
+    </collision>
     <inertial>
       <origin xyz="0 0 0" />
@@ -276,5 +276,5 @@
     <limit velocity="6.5" effort="1000" lower="-0.01" upper="0.035" />
   </joint>
-  <!-- Transmisstion 6 -->
+  <!-- Transmission 6 -->
   <transmission name="tran6">
     <type>transmission_interface/SimpleTransmission</type>

Commit message: update transmission tag

File: open_manipulator_description/urdf/open_manipulator_chain.xacro (robot description, xacro)
@@ -52,5 +52,5 @@
     <type>transmission_interface/SimpleTransmission</type>
     <joint name="joint1">
-      <hardwareInterface>PositionJointInterface</hardwareInterface>
+      <hardwareInterface>hardware_interface/PositionJointInterface</hardwareInterface>
     </joint>
     <actuator name="motor1">
@@ -94,5 +94,5 @@
     <type>transmission_interface/SimpleTransmission</type>
     <joint name="joint2">
-      <hardwareInterface>PositionJointInterface</hardwareInterface>
+      <hardwareInterface>hardware_interface/PositionJointInterface</hardwareInterface>
     </joint>
     <actuator name="motor2">
@@ -136,5 +136,5 @@
     <type>transmission_interface/SimpleTransmission</type>
     <joint name="joint3">
-      <hardwareInterface>PositionJointInterface</hardwareInterface>
+      <hardwareInterface>hardware_interface/PositionJointInterface</hardwareInterface>
     </joint>
     <actuator name="motor3">
@@ -178,5 +178,5 @@
     <type>transmission_interface/SimpleTransmission</type>
     <joint name="joint4">
-      <hardwareInterface>PositionJointInterface</hardwareInterface>
+      <hardwareInterface>hardware_interface/PositionJointInterface</hardwareInterface>
     </joint>
     <actuator name="motor4">
@@ -243,5 +243,5 @@
     <type>transmission_interface/SimpleTransmission</type>
     <joint name="grip_joint">
-      <hardwareInterface>PositionJointInterface</hardwareInterface>
+      <hardwareInterface>hardware_interface/PositionJointInterface</hardwareInterface>
     </joint>
     <actuator name="motor7">
@@ -285,5 +285,5 @@
     <type>transmission_interface/SimpleTransmission</type>
     <joint name="grip_joint_sub">
-      <hardwareInterface>PositionJointInterface</hardwareInterface>
+      <hardwareInterface>hardware_interface/PositionJointInterface</hardwareInterface>
     </joint>
     <actuator name="motor8">

File: open_manipulator_with_tb3/urdf/open_manipulator_chain_with_tb3.xacro (robot description, xacro)
@@ -2,6 +2,4 @@
 <!-- Open_Manipulator Chain -->
 <robot name="open_manipulator_chain_with_tb3" xmlns:xacro="http://www.ros.org/wiki/xacro">
-  <!-- some parameters -->
-  <xacro:property name="pi" value="3.141592654" />
   <!-- Include TurtleBot3 Waffle URDF -->
   <xacro:include filename="$(find turtlebot3_description)/urdf/turtlebot3_waffle_naked.urdf.xacro" />
@@ -47,5 +45,5 @@
     <type>transmission_interface/SimpleTransmission</type>
     <joint name="joint1">
-      <hardwareInterface>PositionJointInterface</hardwareInterface>
+      <hardwareInterface>hardware_interface/PositionJointInterface</hardwareInterface>
     </joint>
     <actuator name="motor1">
@@ -89,5 +87,5 @@
     <type>transmission_interface/SimpleTransmission</type>
     <joint name="joint2">
-      <hardwareInterface>PositionJointInterface</hardwareInterface>
+      <hardwareInterface>hardware_interface/PositionJointInterface</hardwareInterface>
     </joint>
     <actuator name="motor2">
@@ -131,5 +129,5 @@
     <type>transmission_interface/SimpleTransmission</type>
     <joint name="joint3">
-      <hardwareInterface>PositionJointInterface</hardwareInterface>
+      <hardwareInterface>hardware_interface/PositionJointInterface</hardwareInterface>
     </joint>
     <actuator name="motor3">
@@ -173,5 +171,5 @@
     <type>transmission_interface/SimpleTransmission</type>
     <joint name="joint4">
-      <hardwareInterface>PositionJointInterface</hardwareInterface>
+      <hardwareInterface>hardware_interface/PositionJointInterface</hardwareInterface>
     </joint>
     <actuator name="motor4">
@@ -238,5 +236,5 @@
     <type>transmission_interface/SimpleTransmission</type>
     <joint name="grip_joint">
-      <hardwareInterface>PositionJointInterface</hardwareInterface>
+      <hardwareInterface>hardware_interface/PositionJointInterface</hardwareInterface>
     </joint>
     <actuator name="motor7">
@@ -280,5 +278,5 @@
     <type>transmission_interface/SimpleTransmission</type>
     <joint name="grip_joint_sub">
-      <hardwareInterface>PositionJointInterface</hardwareInterface>
+      <hardwareInterface>hardware_interface/PositionJointInterface</hardwareInterface>
     </joint>
     <actuator name="motor8">

Commit message: delete pi

File: open_manipulator_description/urdf/open_manipulator_chain.xacro (robot description, xacro)
@@ -2,6 +2,4 @@
 <!-- Open_Manipulator Chain -->
 <robot name="open_manipulator_chain" xmlns:xacro="http://www.ros.org/wiki/xacro">
-  <!-- some parameters -->
-  <xacro:property name="pi" value="3.141592654" />
   <!-- Import all Gazebo-customization elements, including Gazebo colors -->
   <xacro:include filename="$(find open_manipulator_description)/urdf/open_manipulator_chain.gazebo.xacro" />

Commit message: add kinect setting

File: open_manipulator_description/urdf/open_manipulator_chain.xacro (robot description, xacro)
@@ -4,4 +4,22 @@
   <!-- some parameters -->
   <xacro:property name="pi" value="3.141592654" />
+  <xacro:property name="M_PI" value="3.141592654" />
+  <!-- for kinect -->
+	<xacro:property name="cam_px" value="-0.3150" />
+	<xacro:property name="cam_py" value="0.11" />
+	<xacro:property name="cam_pz" value="0.63" />
+	<xacro:property name="cam_or" value="0" />
+	<xacro:property name="cam_op" value="${pi * 30 / 180}" /> <!-- 25 deg  -->
+	<xacro:property name="cam_oy" value="${-pi * 0 / 180}" />
+    <xacro:include filename="$(find realsense_ros_camera)/urdf/_r430.urdf.xacro"/>
+	<xacro:include filename="$(find cube_description)/urdf/sensors/kinect.urdf.xacro"/>
+	<xacro:include filename="$(find cube_description)/urdf/common_properties.urdf.xacro"/>
+  <!-- realsense-->
+    <!-- <xacro:sensor_r430 parent="world">                                                 -->
+		  <!-- <origin xyz="${cam_px} ${cam_py} ${cam_pz}" rpy="${cam_or} ${cam_op} ${cam_oy}" /> -->
+    <!-- </xacro:sensor_r430>                                                               -->
+  <!-- kinect -->
+    <xacro:sensor_kinect parent="world">
+    </xacro:sensor_kinect>
   <!-- Import all Gazebo-customization elements, including Gazebo colors -->
   <xacro:include filename="$(find open_manipulator_description)/urdf/open_manipulator_chain.gazebo.xacro" />
