Commit message: add mimic param and end effector point

File: open_manipulator_description/urdf/open_manipulator.gazebo.xacro (robot description, xacro)
@@ -30,8 +30,12 @@
   <!-- grip_link_sub -->
   <RefLink ref="grip_link_sub"/>
+  <!-- end effector link -->
+  <gazebo reference="end_effector_link">
+    <material>Gazebo/Red</material>
+  </gazebo>
   <!-- ros_control plugin -->
   <gazebo>
     <plugin name="gazebo_ros_control" filename="libgazebo_ros_control.so">
-      <robotNamespace>/open_manipulator</robotNamespace>
+      <robotNamespace>open_manipulator</robotNamespace>
       <controlPeriod>0.001</controlPeriod>
       <robotSimType>gazebo_ros_control/DefaultRobotHWSim</robotSimType>

File: open_manipulator_description/urdf/open_manipulator.urdf.xacro (robot description, xacro)
@@ -11,5 +11,5 @@
       <type>transmission_interface/SimpleTransmission</type>
       <joint name="${joint}">
-	      <hardwareInterface>hardware_interface/PositionJointInterface</hardwareInterface>
+        <hardwareInterface>hardware_interface/PositionJointInterface</hardwareInterface>
       </joint>
       <actuator name="motor${n}">
@@ -64,5 +64,5 @@
     <origin xyz="0.012 0.0 0.017" rpy="0 0 0"/>
     <axis xyz="0 0 1"/>
-    <limit velocity="6.5" effort="1000" lower="${-pi*0.9}" upper="${pi*0.9}" />
+    <limit velocity="4.8" effort="1" lower="${-pi*0.9}" upper="${pi*0.9}" />
   </joint>
   <!-- Transmission 1 -->
@@ -104,5 +104,5 @@
     <origin xyz="0.0 0.0 0.058" rpy="0 0 0"/>
     <axis xyz="0 1 0"/>
-    <limit velocity="6.5" effort="1000" lower="${-pi*0.57}" upper="${pi*0.5}" />
+    <limit velocity="4.8" effort="1" lower="${-pi*0.57}" upper="${pi*0.5}" />
   </joint>
   <!-- Transmission 2 -->
@@ -144,5 +144,5 @@
     <origin xyz="0.024 0 0.128" rpy="0 0 0"/>
     <axis xyz="0 1 0"/>
-    <limit velocity="6.5" effort="1000" lower="${-pi*0.3}" upper="${pi*0.44}" />
+    <limit velocity="4.8" effort="1" lower="${-pi*0.3}" upper="${pi*0.44}" />
   </joint>
   <!-- Transmission 3 -->
@@ -184,5 +184,5 @@
     <origin xyz="0.124 0.0 0.0" rpy="0 0 0"/>
     <axis xyz="0 1 0"/>
-    <limit velocity="6.5" effort="1000" lower="${-pi*0.57}" upper="${pi*0.65}" />
+    <limit velocity="4.8" effort="1" lower="${-pi*0.57}" upper="${pi*0.65}" />
   </joint>
   <!-- Transmission 4 -->
@@ -221,5 +221,5 @@
   <link name="grip_link">
     <visual>
-      <origin xyz="0.028 0.0246 0" rpy="0 0 0"/>
+      <origin xyz="0.0 0.0 0" rpy="0 0 0"/>
       <geometry>
         <mesh filename="package://open_manipulator_description/meshes/chain_link_grip_l.stl" scale="0.001 0.001 0.001"/>
@@ -228,5 +228,5 @@
     </visual>
     <collision>
-      <origin xyz="0.028 0.0246 0" rpy="0 0 0"/>
+      <origin xyz="0.0 0.0 0" rpy="0 0 0"/>
       <geometry>
         <mesh filename="package://open_manipulator_description/meshes/chain_link_grip_l.stl" scale="0.001 0.001 0.001"/>
@@ -252,7 +252,7 @@
     <parent link="link5"/>
     <child link="grip_link"/>
-    <origin xyz="0.0536 0.0 0.0" rpy="0 0 0"/>
+    <origin xyz="0.0817 0.019 0.0" rpy="0 0 0"/>
     <axis xyz="0 1 0"/>
-    <limit velocity="3.5" effort="100" lower="-0.015" upper="0.0105" />
+    <limit velocity="4.8" effort="1" lower="-0.010" upper="0.019" />
   </joint>
   <!-- Transmission 5 -->
@@ -261,5 +261,5 @@
   <link name="grip_link_sub">
     <visual>
-      <origin xyz="0.028 -0.0246 0" rpy="0 0 0"/>
+      <origin xyz="0.0 -0.0 0" rpy="0 0 0"/>
       <geometry>
         <mesh filename="package://open_manipulator_description/meshes/chain_link_grip_r.stl" scale="0.001 0.001 0.001"/>
@@ -268,5 +268,5 @@
     </visual>
     <collision>
-      <origin xyz="0.028 -0.0246 0" rpy="0 0 0"/>
+      <origin xyz="0.0 -0.0 0" rpy="0 0 0"/>
       <geometry>
         <mesh filename="package://open_manipulator_description/meshes/chain_link_grip_r.stl" scale="0.001 0.001 0.001"/>
@@ -292,9 +292,31 @@
     <parent link="link5"/>
     <child link="grip_link_sub"/>
-    <origin xyz="0.0536 0 0" rpy="0 0 0"/>
+    <origin xyz="0.0817 -0.019 0" rpy="0 0 0"/>
     <axis xyz="0 -1 0"/>
-    <limit velocity="3.5" effort="100" lower="-0.015" upper="0.0105" />
+    <limit velocity="4.8" effort="1" lower="-0.010" upper="0.019" />
+    <mimic joint="grip_joint" multiplier="1"/>
   </joint>
   <!-- Transmission 6 -->
   <xacro:SimpleTransmission n="6" joint="grip_joint_sub" />
+  <!-- end effector joint -->
+  <joint name="end_effector_joint" type="fixed">
+    <origin xyz="0.130 0.0 0.0" rpy="0 0 0"/>
+    <parent link="link5"/>
+    <child link="end_effector_link"/>
+  </joint>
+  <!-- end effector link -->
+  <link name="end_effector_link">
+    <visual>
+      <origin xyz="0 0 0" rpy="0 0 0"/>
+      <geometry>
+        <box size="0.01 0.01 0.01" />
+      </geometry>
+      <material name="red"/>
+     </visual>
+    <inertial>
+      <origin xyz="0.0 0.0 0.0" rpy="0 0 0"/>
+      <mass value="0.001"/>
+      <inertia ixx="1.0" ixy="0.0" ixz="0.0" iyy="1.0" iyz="0.0" izz="1.0" />
+    </inertial>
+  </link>
 </robot>

Commit message: change gripper link name

File: open_manipulator_description/urdf/open_manipulator.gazebo.xacro (robot description, xacro)
@@ -26,8 +26,8 @@
   <!-- Link5 -->
   <RefLink ref="link5"/>
-  <!-- grip_link -->
-  <RefLink ref="grip_link"/>
-  <!-- grip_link_sub -->
-  <RefLink ref="grip_link_sub"/>
+  <!-- gripper_link -->
+  <RefLink ref="gripper_link"/>
+  <!-- gripper_link_sub -->
+  <RefLink ref="gripper_link_sub"/>
   <!-- end effector link -->
   <gazebo reference="end_effector_link">

File: open_manipulator_description/urdf/open_manipulator.urdf.xacro (robot description, xacro)
@@ -218,6 +218,6 @@
     </inertial> -->
   </link>
-  <!--  Grip link -->
-  <link name="grip_link">
+  <!--  Gripper link -->
+  <link name="gripper_link">
     <visual>
       <origin xyz="0.0 0.0 0" rpy="0 0 0"/>
@@ -248,8 +248,8 @@
     </inertial> -->
   </link>
-  <!--  Grip joint -->
-  <joint name="grip_joint" type="prismatic">
+  <!--  Gripper joint -->
+  <joint name="gripper" type="prismatic">
     <parent link="link5"/>
-    <child link="grip_link"/>
+    <child link="gripper_link"/>
     <origin xyz="0.0817 0.019 0.0" rpy="0 0 0"/>
     <axis xyz="0 1 0"/>
@@ -257,7 +257,7 @@
   </joint>
   <!-- Transmission 5 -->
-  <xacro:SimpleTransmission n="5" joint="grip_joint" />
-  <!--  Grip link sub -->
-  <link name="grip_link_sub">
+  <xacro:SimpleTransmission n="5" joint="gripper" />
+  <!--  Gripper link sub -->
+  <link name="gripper_link_sub">
     <visual>
       <origin xyz="0.0 -0.0 0" rpy="0 0 0"/>
@@ -288,15 +288,15 @@
     </inertial> -->
   </link>
-  <!--  Grip joint sub -->
-  <joint name="grip_joint_sub" type="prismatic">
+  <!--  Gripper joint sub -->
+  <joint name="gripper_sub" type="prismatic">
     <parent link="link5"/>
-    <child link="grip_link_sub"/>
+    <child link="gripper_link_sub"/>
     <origin xyz="0.0817 -0.019 0" rpy="0 0 0"/>
     <axis xyz="0 -1 0"/>
     <limit velocity="4.8" effort="1" lower="-0.010" upper="0.019" />
-    <mimic joint="grip_joint" multiplier="1"/>
+    <mimic joint="gripper" multiplier="1"/>
   </joint>
   <!-- Transmission 6 -->
-  <xacro:SimpleTransmission n="6" joint="grip_joint_sub" />
+  <xacro:SimpleTransmission n="6" joint="gripper_sub" />
   <!-- end effector joint -->
   <joint name="end_effector_joint" type="fixed">

Commit message: updated gazebo.xacro file

File: open_manipulator_description/urdf/open_manipulator.gazebo.xacro (robot description, xacro)
@@ -42,3 +42,12 @@
     </plugin>
   </gazebo>
+  <gazebo>
+    <!-- loading plugin: mimic joints works in gazebo now -->
+    <plugin name="gazebo_gripper_ros_control" filename="libroboticsgroup_gazebo_mimic_joint_plugin.so">
+      <joint>gripper</joint>
+      <mimicJoint>gripper_sub</mimicJoint>
+      <multiplier>1.0</multiplier>
+      <offset>0.0</offset>
+    </plugin>
+  </gazebo>
 </robot>

Commit message: added camera to urdf files for om_perception

File: open_manipulator_description/urdf/open_manipulator.gazebo.xacro (robot description, xacro)
@@ -51,3 +51,43 @@
     </plugin>
   </gazebo>
+  <!-- camera -->
+  <gazebo reference="camera_link">
+    <sensor type="camera" name="intel_realsense_r200">
+      <update_rate>30.0</update_rate>
+      <camera name="head">
+        <horizontal_fov>1.02974</horizontal_fov>
+        <image>
+          <width>1920</width>
+          <height>1080</height>
+          <format>R8G8B8</format>
+        </image>
+        <clip>
+          <near>0.02</near>
+          <far>300</far>
+        </clip>
+        <noise>
+          <type>gaussian</type>
+          <!-- Noise is sampled independently per pixel on each frame.
+               That pixel's noise value is added to each of its color
+               channels, which at that point lie in the range [0,1]. -->
+          <mean>0.0</mean>
+          <stddev>0.007</stddev>
+        </noise>
+      </camera>
+      <plugin name="camera_controller" filename="libgazebo_ros_camera.so">
+        <alwaysOn>true</alwaysOn>
+        <updateRate>0.0</updateRate>
+        <cameraName>camera/color</cameraName>
+        <imageTopicName>image_raw</imageTopicName>
+        <cameraInfoTopicName>camera_info</cameraInfoTopicName>
+        <frameName>camera_link</frameName>
+        <hackBaseline>0.07</hackBaseline>
+        <distortionK1>0.0</distortionK1>
+        <distortionK2>0.0</distortionK2>
+        <distortionK3>0.0</distortionK3>
+        <distortionT1>0.0</distortionT1>
+        <distortionT2>0.0</distortionT2>
+      </plugin>
+    </sensor>
+  </gazebo>
 </robot>

File: open_manipulator_description/urdf/open_manipulator.urdf.xacro (robot description, xacro)
@@ -149,4 +149,12 @@
     </inertial>
   </link>
+  <!--  Gripper joint -->
+  <joint name="gripper" type="prismatic">
+    <parent link="link5"/>
+    <child link="gripper_link"/>
+    <origin xyz="0.0817 0.021 0.0" rpy="0 0 0"/>
+    <axis xyz="0 1 0"/>
+    <limit velocity="4.8" effort="1" lower="-0.010" upper="0.019" />
+  </joint>
   <!--  Gripper link -->
   <link name="gripper_link">
@@ -172,11 +180,12 @@
     </inertial>
   </link>
-  <!--  Gripper joint -->
-  <joint name="gripper" type="prismatic">
-    <parent link="link5"/>
-    <child link="gripper_link"/>
-    <origin xyz="0.0817 0.021 0.0" rpy="0 0 0"/>
-    <axis xyz="0 1 0"/>
+  <!--  Gripper joint sub -->
+  <joint name="gripper_sub" type="prismatic">
+    <parent link="link5"/>
+    <child link="gripper_link_sub"/>
+    <origin xyz="0.0817 -0.021 0" rpy="0 0 0"/>
+    <axis xyz="0 -1 0"/>
     <limit velocity="4.8" effort="1" lower="-0.010" upper="0.019" />
+    <mimic joint="gripper" multiplier="1"/>
   </joint>
   <!--  Gripper link sub -->
@@ -203,13 +212,4 @@
     </inertial>
   </link>
-  <!--  Gripper joint sub -->
-  <joint name="gripper_sub" type="prismatic">
-    <parent link="link5"/>
-    <child link="gripper_link_sub"/>
-    <origin xyz="0.0817 -0.021 0" rpy="0 0 0"/>
-    <axis xyz="0 -1 0"/>
-    <limit velocity="4.8" effort="1" lower="-0.010" upper="0.019" />
-    <mimic joint="gripper" multiplier="1"/>
-  </joint>
   <!-- end effector joint -->
   <joint name="end_effector_joint" type="fixed">
@@ -235,3 +235,11 @@
     </inertial>
   </link>
+  <!-- Realsense Camera Joint Position -->
+  <joint name="camera_joint" type="fixed">
+    <axis xyz="0 1 0" />
+    <origin xyz="0.070 0.040 0.052" rpy="0 0 0"/>
+    <parent link="link5"/>
+    <child link="camera_link"/>
+  </joint>
+  <link name="camera_link"/>
 </robot>
