Commit message: change calculated inertia param

File: open_manipulator_description/urdf/open_manipulator.urdf.xacro (robot description, xacro)
@@ -43,5 +43,5 @@
       </geometry>
     </collision>
-    <inertial>
+<!--    <inertial>
       <origin xyz="0 0 0" />
       <mass value="0.082" />
@@ -49,6 +49,6 @@
                iyy="0.1" iyz="0.0"
                izz="0.1" />
-    </inertial>
-    <!-- <inertial>
+    </inertial>-->
+     <inertial>
       <origin xyz="3.0876154e-04 0.0000000e+00 -1.2176461e-04" />
       <mass value="7.9119962e-02" />
@@ -56,5 +56,5 @@
                iyy="2.1898364e-05" iyz="0.0"
                izz="1.9267361e-05" />
-    </inertial> -->
+    </inertial>
   </link>
   <!-- Joint 1 -->
@@ -83,5 +83,5 @@
       </geometry>
     </collision>
-    <inertial>
+<!--    <inertial>
       <origin xyz="0 0 0" />
       <mass value="0.098" />
@@ -89,6 +89,6 @@
                iyy="0.1" iyz="0.0"
                izz="0.1" />
-    </inertial>
-    <!-- <inertial>
+    </inertial>-->
+     <inertial>
       <origin xyz="-3.0184870e-04 5.4043684e-04 ${0.018 + 2.9433464e-02}" />
       <mass value="9.8406837e-02" />
@@ -96,5 +96,5 @@
                iyy="3.2689329e-05" iyz="2.8511935e-08"
                izz="1.8850320e-05" />
-    </inertial> -->
+    </inertial>
   </link>
   <!--  Joint 2 -->
@@ -123,5 +123,5 @@
       </geometry>
     </collision>
-    <inertial>
+<!--    <inertial>
       <origin xyz="0 0 0" />
       <mass value="0.136" />
@@ -129,6 +129,6 @@
                iyy="0.1" iyz="0.0"
                izz="0.1" />
-    </inertial>
-    <!-- <inertial>
+    </inertial>-->
+     <inertial>
       <origin xyz="1.0308393e-02 3.7743363e-04 1.0170197e-01" />
       <mass value="1.3850917e-01" />
@@ -136,5 +136,5 @@
                iyy="3.4290447e-04" iyz="-1.5717516e-06"
                izz="6.0346498e-05" />
-    </inertial> -->
+    </inertial>
   </link>
   <!--  Joint 3 -->
@@ -163,5 +163,5 @@
       </geometry>
     </collision>
-    <inertial>
+<!--    <inertial>
       <origin xyz="0 0 0" />
       <mass value="0.131" />
@@ -169,6 +169,6 @@
                iyy="0.1" iyz="0.0"
                izz="0.1" />
-    </inertial>
-    <!-- <inertial>
+    </inertial>-->
+     <inertial>
       <origin xyz="9.0909590e-02 3.8929816e-04 2.2413279e-04" />
       <mass value="1.3274562e-01" />
@@ -176,5 +176,5 @@
                iyy="2.4230292e-04" iyz="1.1559550e-08"
                izz="2.5155057e-04" />
-    </inertial> -->
+    </inertial>
   </link>
   <!--  Joint 4 -->
@@ -203,5 +203,5 @@
       </geometry>
     </collision>
-    <inertial>
+<!--    <inertial>
       <origin xyz="0 0 0" />
       <mass value="0.141" />
@@ -209,6 +209,6 @@
                iyy="0.1" iyz="0.0"
                izz="0.1" />
-    </inertial>
-    <!-- <inertial>
+    </inertial>-->
+     <inertial>
       <origin xyz="4.4206755e-02 3.6839985e-07 8.9142216e-03" />
       <mass value="1.4327573e-01" />
@@ -216,5 +216,5 @@
                iyy="7.5980465e-05" iyz="0.0"
                izz="9.3127351e-05" />
-    </inertial> -->
+    </inertial>
   </link>
   <!--  Gripper link -->
@@ -236,9 +236,9 @@
       <origin xyz="0 0 0" />
       <mass value="0.017" />
-      <inertia ixx="0.1" ixy="0.0" ixz="0.0"
-               iyy="0.1" iyz="0.0"
-               izz="0.1" />
-    </inertial>
-    <!-- <inertial>
+      <inertia ixx="0.001" ixy="0.0" ixz="0.0"
+               iyy="0.001" iyz="0.0"
+               izz="0.001" />
+    </inertial>
+<!--     <inertial>
       <origin xyz="${0.028 + 8.3720668e-03} ${0.0246 + 9.9696160e-03} -4.2836895e-07" />
       <mass value="3.2218127e-02" />
@@ -246,5 +246,5 @@
                iyy="2.2552871e-05" iyz="-3.1463634e-10"
                izz="1.7605306e-05" />
-    </inertial> -->
+    </inertial>-->
   </link>
   <!--  Gripper joint -->
@@ -276,9 +276,9 @@
       <origin xyz="0 0 0" />
       <mass value="0.017" />
-      <inertia ixx="0.1" ixy="0.0" ixz="0.0"
-               iyy="0.1" iyz="0.0"
-               izz="0.1" />
-    </inertial>
-    <!-- <inertial>
+      <inertia ixx="0.001" ixy="0.0" ixz="0.0"
+               iyy="0.001" iyz="0.0"
+               izz="0.001" />
+    </inertial>
+<!--     <inertial>
       <origin xyz="${0.028 + 8.3720668e-03} ${-0.0246 - 9.9696160e-03} -4.2836895e-07" />
       <mass value="3.2218127e-02" />
@@ -286,5 +286,5 @@
                iyy="2.2552871e-05" iyz="-3.1463634e-10"
                izz="1.7605306e-05" />
-    </inertial> -->
+    </inertial>-->
   </link>
   <!--  Gripper joint sub -->
@@ -317,5 +317,5 @@
       <origin xyz="0.0 0.0 0.0" rpy="0 0 0"/>
       <mass value="0.001"/>
-      <inertia ixx="1.0" ixy="0.0" ixz="0.0" iyy="1.0" iyz="0.0" izz="1.0" />
+      <inertia ixx="0.001" ixy="0.0" ixz="0.0" iyy="0.001" iyz="0.0" izz="0.001" />
     </inertial>
   </link>

Commit message: update inertia

File: open_manipulator_description/urdf/open_manipulator.urdf.xacro (robot description, xacro)
@@ -236,7 +236,7 @@
       <origin xyz="0 0 0" />
       <mass value="0.017" />
-      <inertia ixx="0.001" ixy="0.0" ixz="0.0"
-               iyy="0.001" iyz="0.0"
-               izz="0.001" />
+      <inertia ixx="1.0e-03" ixy="0.0" ixz="0.0"
+               iyy="1.0e-03" iyz="0.0"
+               izz="1.0e-03" />
     </inertial>
 <!--     <inertial>
@@ -276,7 +276,7 @@
       <origin xyz="0 0 0" />
       <mass value="0.017" />
-      <inertia ixx="0.001" ixy="0.0" ixz="0.0"
-               iyy="0.001" iyz="0.0"
-               izz="0.001" />
+      <inertia ixx="1.0e-03" ixy="0.0" ixz="0.0"
+               iyy="1.0e-03" iyz="0.0"
+               izz="1.0e-03" />
     </inertial>
 <!--     <inertial>
@@ -317,5 +317,5 @@
       <origin xyz="0.0 0.0 0.0" rpy="0 0 0"/>
       <mass value="0.001"/>
-      <inertia ixx="0.001" ixy="0.0" ixz="0.0" iyy="0.001" iyz="0.0" izz="0.001" />
+      <inertia ixx="1.0e-06" ixy="0.0" ixz="0.0" iyy="1.0e-06" iyz="0.0" izz="1.0e-06" />
     </inertial>
   </link>

Commit message: modified link2 and joint2 position

File: open_manipulator_description/urdf/open_manipulator.urdf.xacro (robot description, xacro)
@@ -71,5 +71,5 @@
   <link name="link2">
     <visual>
-      <origin xyz="0 0 0.018" rpy="0 0 0"/>
+      <origin xyz="0 0 0.019" rpy="0 0 0"/>
       <geometry>
         <mesh filename="package://open_manipulator_description/meshes/chain_link2.stl" scale="0.001 0.001 0.001"/>
@@ -78,5 +78,5 @@
     </visual>
     <collision>
-      <origin xyz="0 0 0.018" rpy="0 0 0"/>
+      <origin xyz="0 0 0.019" rpy="0 0 0"/>
       <geometry>
         <mesh filename="package://open_manipulator_description/meshes/chain_link2.stl" scale="0.001 0.001 0.001"/>
@@ -102,5 +102,5 @@
     <parent link="link2"/>
     <child link="link3"/>
-    <origin xyz="0.0 0.0 0.058" rpy="0 0 0"/>
+    <origin xyz="0.0 0.0 0.0595" rpy="0 0 0"/>
     <axis xyz="0 1 0"/>
     <limit velocity="4.8" effort="1" lower="${-pi*0.57}" upper="${pi*0.5}" />

Commit message: modified end_effector origin

File: open_manipulator_description/urdf/open_manipulator.urdf.xacro (robot description, xacro)
@@ -301,5 +301,5 @@
   <!-- end effector joint -->
   <joint name="end_effector_joint" type="fixed">
-    <origin xyz="0.130 0.0 0.0" rpy="0 0 0"/>
+    <origin xyz="0.126 0.0 0.0" rpy="0 0 0"/>
     <parent link="link5"/>
     <child link="end_effector_link"/>

Commit message: modified gripper origin

File: open_manipulator_description/urdf/open_manipulator.urdf.xacro (robot description, xacro)
@@ -252,5 +252,5 @@
     <parent link="link5"/>
     <child link="gripper_link"/>
-    <origin xyz="0.0817 0.019 0.0" rpy="0 0 0"/>
+    <origin xyz="0.0817 0.021 0.0" rpy="0 0 0"/>
     <axis xyz="0 1 0"/>
     <limit velocity="4.8" effort="1" lower="-0.010" upper="0.019" />
@@ -292,5 +292,5 @@
     <parent link="link5"/>
     <child link="gripper_link_sub"/>
-    <origin xyz="0.0817 -0.019 0" rpy="0 0 0"/>
+    <origin xyz="0.0817 -0.021 0" rpy="0 0 0"/>
     <axis xyz="0 -1 0"/>
     <limit velocity="4.8" effort="1" lower="-0.010" upper="0.019" />

Commit message: updated urdf files

File: open_manipulator_description/urdf/open_manipulator.urdf.xacro (robot description, xacro)
@@ -6,17 +6,6 @@
   <!-- Import Rviz colors -->
   <xacro:include filename="$(find open_manipulator_description)/urdf/materials.xacro" />
-  <!-- Transmission macro -->
-  <xacro:macro name="SimpleTransmission" params="joint n">
-    <transmission name="tran${n}">
-      <type>transmission_interface/SimpleTransmission</type>
-      <joint name="${joint}">
-        <hardwareInterface>hardware_interface/EffortJointInterface</hardwareInterface>
-      </joint>
-      <actuator name="motor${n}">
-        <hardwareInterface>hardware_interface/EffortJointInterface</hardwareInterface>
-        <mechanicalReduction>1</mechanicalReduction>
-      </actuator>
-    </transmission>
-  </xacro:macro>
+  <!-- Import Transmission -->
+  <xacro:include filename="$(find open_manipulator_description)/urdf/transmission.xacro" />
   <!-- World -->
   <link name="world">
@@ -66,6 +55,4 @@
     <limit velocity="4.8" effort="1" lower="${-pi*0.9}" upper="${pi*0.9}" />
   </joint>
-  <!-- Transmission 1 -->
-  <xacro:SimpleTransmission n="1" joint="joint1" />
   <!--  Link 2 -->
   <link name="link2">
@@ -106,6 +93,4 @@
     <limit velocity="4.8" effort="1" lower="${-pi*0.57}" upper="${pi*0.5}" />
   </joint>
-  <!-- Transmission 2 -->
-  <xacro:SimpleTransmission n="2" joint="joint2" />
   <!--  Link 3 -->
   <link name="link3">
@@ -146,6 +131,4 @@
     <limit velocity="4.8" effort="1" lower="${-pi*0.3}" upper="${pi*0.44}" />
   </joint>
-  <!-- Transmission 3 -->
-  <xacro:SimpleTransmission n="3" joint="joint3" />
   <!--  Link 4 -->
   <link name="link4">
@@ -186,6 +169,4 @@
     <limit velocity="4.8" effort="1" lower="${-pi*0.57}" upper="${pi*0.65}" />
   </joint>
-  <!-- Transmission 4 -->
-  <xacro:SimpleTransmission n="4" joint="joint4" />
   <!--  Link 5 -->
   <link name="link5">
@@ -256,6 +237,4 @@
     <limit velocity="4.8" effort="1" lower="-0.010" upper="0.019" />
   </joint>
-  <!-- Transmission 5 -->
-  <xacro:SimpleTransmission n="5" joint="gripper" />
   <!--  Gripper link sub -->
   <link name="gripper_link_sub">
@@ -297,6 +276,4 @@
     <mimic joint="gripper" multiplier="1"/>
   </joint>
-  <!-- Transmission 6 -->
-  <xacro:SimpleTransmission n="6" joint="gripper_sub" />
   <!-- end effector joint -->
   <joint name="end_effector_joint" type="fixed">

Commit message: fixed uredf files

File: open_manipulator_description/urdf/open_manipulator.urdf.xacro (robot description, xacro)
@@ -2,10 +2,10 @@
 <!-- Open_Manipulator Chain -->
 <robot name="open_manipulator" xmlns:xacro="http://ros.org/wiki/xacro">
+  <!-- Import Rviz colors -->
+  <xacro:include filename="$(find open_manipulator_description)/urdf/materials.xacro" />
   <!-- Import all Gazebo-customization elements, including Gazebo colors -->
   <xacro:include filename="$(find open_manipulator_description)/urdf/open_manipulator.gazebo.xacro" />
-  <!-- Import Rviz colors -->
-  <xacro:include filename="$(find open_manipulator_description)/urdf/materials.xacro" />
   <!-- Import Transmission -->
-  <xacro:include filename="$(find open_manipulator_description)/urdf/transmission.xacro" />
+  <xacro:include filename="$(find open_manipulator_description)/urdf/open_manipulator.transmission.xacro" />
   <!-- World -->
   <link name="world">
@@ -32,11 +32,4 @@
       </geometry>
     </collision>
-<!--    <inertial>
-      <origin xyz="0 0 0" />
-      <mass value="0.082" />
-      <inertia ixx="0.1" ixy="0.0" ixz="0.0"
-               iyy="0.1" iyz="0.0"
-               izz="0.1" />
-    </inertial>-->
      <inertial>
       <origin xyz="3.0876154e-04 0.0000000e+00 -1.2176461e-04" />
@@ -70,11 +63,4 @@
       </geometry>
     </collision>
-<!--    <inertial>
-      <origin xyz="0 0 0" />
-      <mass value="0.098" />
-      <inertia ixx="0.1" ixy="0.0" ixz="0.0"
-               iyy="0.1" iyz="0.0"
-               izz="0.1" />
-    </inertial>-->
      <inertial>
       <origin xyz="-3.0184870e-04 5.4043684e-04 ${0.018 + 2.9433464e-02}" />
@@ -108,11 +94,4 @@
       </geometry>
     </collision>
-<!--    <inertial>
-      <origin xyz="0 0 0" />
-      <mass value="0.136" />
-      <inertia ixx="0.1" ixy="0.0" ixz="0.0"
-               iyy="0.1" iyz="0.0"
-               izz="0.1" />
-    </inertial>-->
      <inertial>
       <origin xyz="1.0308393e-02 3.7743363e-04 1.0170197e-01" />
@@ -146,11 +125,4 @@
       </geometry>
     </collision>
-<!--    <inertial>
-      <origin xyz="0 0 0" />
-      <mass value="0.131" />
-      <inertia ixx="0.1" ixy="0.0" ixz="0.0"
-               iyy="0.1" iyz="0.0"
-               izz="0.1" />
-    </inertial>-->
      <inertial>
       <origin xyz="9.0909590e-02 3.8929816e-04 2.2413279e-04" />
@@ -184,11 +156,4 @@
       </geometry>
     </collision>
-<!--    <inertial>
-      <origin xyz="0 0 0" />
-      <mass value="0.141" />
-      <inertia ixx="0.1" ixy="0.0" ixz="0.0"
-               iyy="0.1" iyz="0.0"
-               izz="0.1" />
-    </inertial>-->
      <inertial>
       <origin xyz="4.4206755e-02 3.6839985e-07 8.9142216e-03" />
@@ -216,16 +181,9 @@
     <inertial>
       <origin xyz="0 0 0" />
-      <mass value="0.017" />
+      <mass value="1.0e-03" />
       <inertia ixx="1.0e-03" ixy="0.0" ixz="0.0"
                iyy="1.0e-03" iyz="0.0"
                izz="1.0e-03" />
     </inertial>
-<!--     <inertial>
-      <origin xyz="${0.028 + 8.3720668e-03} ${0.0246 + 9.9696160e-03} -4.2836895e-07" />
-      <mass value="3.2218127e-02" />
-      <inertia ixx="9.5568826e-06" ixy="2.8424644e-06" ixz="-3.2829197e-10"
-               iyy="2.2552871e-05" iyz="-3.1463634e-10"
-               izz="1.7605306e-05" />
-    </inertial>-->
   </link>
   <!--  Gripper joint -->
@@ -254,16 +212,9 @@
     <inertial>
       <origin xyz="0 0 0" />
-      <mass value="0.017" />
+      <mass value="1.0e-03" />
       <inertia ixx="1.0e-03" ixy="0.0" ixz="0.0"
                iyy="1.0e-03" iyz="0.0"
                izz="1.0e-03" />
     </inertial>
-<!--     <inertial>
-      <origin xyz="${0.028 + 8.3720668e-03} ${-0.0246 - 9.9696160e-03} -4.2836895e-07" />
-      <mass value="3.2218127e-02" />
-      <inertia ixx="9.5568826e-06" ixy="2.8424644e-06" ixz="-3.2829197e-10"
-               iyy="2.2552871e-05" iyz="-3.1463634e-10"
-               izz="1.7605306e-05" />
-    </inertial>-->
   </link>
   <!--  Gripper joint sub -->
@@ -292,7 +243,9 @@
      </visual>
     <inertial>
-      <origin xyz="0.0 0.0 0.0" rpy="0 0 0"/>
-      <mass value="0.001"/>
-      <inertia ixx="1.0e-06" ixy="0.0" ixz="0.0" iyy="1.0e-06" iyz="0.0" izz="1.0e-06" />
+      <origin xyz="0 0 0" />
+      <mass value="1.0e-03" />
+      <inertia ixx="1.0e-03" ixy="0.0" ixz="0.0"
+               iyy="1.0e-03" iyz="0.0"
+               izz="1.0e-03" />
     </inertial>
   </link>

Commit message: modified urdf file

File: open_manipulator_description/urdf/open_manipulator.urdf.xacro (robot description, xacro)
@@ -1,20 +1,5 @@
 <?xml version="1.0"?>
 <!-- Open_Manipulator Chain -->
-<robot name="open_manipulator" xmlns:xacro="http://ros.org/wiki/xacro">
-  <!-- Import Rviz colors -->
-  <xacro:include filename="$(find open_manipulator_description)/urdf/materials.xacro" />
-  <!-- Import all Gazebo-customization elements, including Gazebo colors -->
-  <xacro:include filename="$(find open_manipulator_description)/urdf/open_manipulator.gazebo.xacro" />
-  <!-- Import Transmission -->
-  <xacro:include filename="$(find open_manipulator_description)/urdf/open_manipulator.transmission.xacro" />
-  <!-- World -->
-  <link name="world">
-  </link>
-  <!-- World fixed joint-->
-  <joint name="world_fixed" type="fixed">
-    <origin xyz="0 0 0" rpy="0 0 0"/>
-    <parent link="world"/>
-    <child link="link1"/>
-  </joint>
+<robot xmlns:xacro="http://ros.org/wiki/xacro">
   <!-- Link 1 -->
   <link name="link1">

Commit message: updated urdf file camera position

File: open_manipulator_description/urdf/open_manipulator.urdf.xacro (robot description, xacro)
@@ -238,5 +238,5 @@
   <joint name="camera_joint" type="fixed">
     <axis xyz="0 1 0" />
-    <origin xyz="0.070 0.040 0.052" rpy="0 0 0"/>
+    <origin xyz="0.070 0.032 0.052" rpy="0 0 0"/>
     <parent link="link5"/>
     <child link="camera_link"/>

Commit message: minor changes

File: open_manipulator_description/urdf/open_manipulator.urdf.xacro (robot description, xacro)
@@ -17,5 +17,5 @@
       </geometry>
     </collision>
-     <inertial>
+    <inertial>
       <origin xyz="3.0876154e-04 0.0000000e+00 -1.2176461e-04" />
       <mass value="7.9119962e-02" />
@@ -48,5 +48,5 @@
       </geometry>
     </collision>
-     <inertial>
+    <inertial>
       <origin xyz="-3.0184870e-04 5.4043684e-04 ${0.018 + 2.9433464e-02}" />
       <mass value="9.8406837e-02" />
@@ -79,5 +79,5 @@
       </geometry>
     </collision>
-     <inertial>
+    <inertial>
       <origin xyz="1.0308393e-02 3.7743363e-04 1.0170197e-01" />
       <mass value="1.3850917e-01" />
@@ -110,5 +110,5 @@
       </geometry>
     </collision>
-     <inertial>
+    <inertial>
       <origin xyz="9.0909590e-02 3.8929816e-04 2.2413279e-04" />
       <mass value="1.3274562e-01" />
@@ -141,5 +141,5 @@
       </geometry>
     </collision>
-     <inertial>
+    <inertial>
       <origin xyz="4.4206755e-02 3.6839985e-07 8.9142216e-03" />
       <mass value="1.4327573e-01" />

Commit message: muted camera_link in open_manipulator.urdf.xacro
The " camera_link " is not frequently used. Adding it by default may cause naming conflicts with actual camera sensor with that name. So I commented out it.

File: open_manipulator_description/urdf/open_manipulator.urdf.xacro (robot description, xacro)
@@ -236,5 +236,5 @@
   </link>
   <!-- Realsense Camera Joint Position -->
-  <joint name="camera_joint" type="fixed">
+<!--   <joint name="camera_joint" type="fixed">
     <axis xyz="0 1 0" />
     <origin xyz="0.070 0.032 0.052" rpy="0 0 0"/>
@@ -242,4 +242,4 @@
     <child link="camera_link"/>
   </joint>
-  <link name="camera_link"/>
+  <link name="camera_link"/> -->
 </robot>
