Commit message: update manipulator model

File: open_manipulator_with_tb3/urdf/open_manipulator_chain_with_tb3_waffle.urdf.xacro (robot description, xacro)
@@ -15,5 +15,5 @@
   <link name="link1">
     <visual>
-      <origin xyz="0.0 0.0 0.0" rpy="0 0 0"/>
+      <origin xyz="0 0 0" rpy="0 0 0"/>
       <geometry>
         <mesh filename="package://open_manipulator_description/meshes/chain_link1.stl" scale="0.001 0.001 0.001"/>
@@ -39,5 +39,5 @@
     <parent link="link1"/>
     <child link="link2"/>
-    <origin xyz="0.012 0.0 0.036" rpy="0 0 0"/>
+    <origin xyz="0.012 0.0 0.017" rpy="0 0 0"/>
     <axis xyz="0 0 1"/>
     <limit velocity="6.5" effort="1000" lower="${-pi*0.9}" upper="${pi*0.9}" />
@@ -57,5 +57,5 @@
   <link name="link2">
     <visual>
-      <origin xyz="0.0 0.0 0.040" rpy="0 0 0"/>
+      <origin xyz="0 0 0.018" rpy="0 0 0"/>
       <geometry>
         <mesh filename="package://open_manipulator_description/meshes/chain_link2.stl" scale="0.001 0.001 0.001"/>
@@ -64,5 +64,5 @@
     </visual>
     <collision>
-      <origin xyz="0.0 0.0 0.030" rpy="0 0 0"/>
+      <origin xyz="0.0 0.0 0.048" rpy="0 0 0"/>
       <geometry>
         <box size="0.0355 0.0550 0.0515"/>
@@ -81,5 +81,5 @@
     <parent link="link2"/>
     <child link="link3"/>
-    <origin xyz="0.0 0.0 0.040" rpy="0 0 0"/>
+    <origin xyz="0.0 0.0 0.058" rpy="0 0 0"/>
     <axis xyz="0 1 0"/>
     <limit velocity="6.5" effort="1000" lower="${-pi*0.5}" upper="${pi*0.5}" />
@@ -99,5 +99,5 @@
   <link name="link3">
     <visual>
-      <origin xyz="0.022 0 0.122" rpy="0 0 0"/>
+      <origin xyz="0 0 0" rpy="0 0 0"/>
       <geometry>
         <mesh filename="package://open_manipulator_description/meshes/chain_link3.stl" scale="0.001 0.001 0.001"/>
@@ -123,7 +123,7 @@
     <parent link="link3"/>
     <child link="link4"/>
-    <origin xyz="0.022 0 0.122" rpy="0 0 0"/>
-    <axis xyz="0 1 0"/>
-    <limit velocity="6.5" effort="1000" lower="${-pi*0.5}" upper="${pi*0.4}" />
+    <origin xyz="0.024 0 0.128" rpy="0 0 0"/>
+    <axis xyz="0 1 0"/>
+    <limit velocity="6.5" effort="1000" lower="${-pi*0.3}" upper="${pi*0.3}" />
   </joint>
   <!-- Transmission 3 -->
@@ -141,5 +141,5 @@
   <link name="link4">
     <visual>
-      <origin xyz="0.124 0 0.0" rpy="0 0 0"/>
+      <origin xyz="0 0 0" rpy="0 0 0"/>
       <geometry>
         <mesh filename="package://open_manipulator_description/meshes/chain_link4.stl" scale="0.001 0.001 0.001"/>
@@ -148,7 +148,7 @@
     </visual>
     <collision>
-      <origin xyz="0.080 0 0.0" rpy="0 0 0"/>
-      <geometry>
-        <box size="0.110 0.055 0.035"/>
+      <origin xyz="0.065 0 0.0" rpy="0 0 0"/>
+      <geometry>
+        <box size="0.115 0.055 0.035"/>
       </geometry>
     </collision>
@@ -183,5 +183,5 @@
   <link name="link5">
     <visual>
-      <origin xyz="0.046 0 0" rpy="0 0 0"/>
+      <origin xyz="0 0 0" rpy="0 0 0"/>
       <geometry>
         <mesh filename="package://open_manipulator_description/meshes/chain_link5.stl" scale="0.001 0.001 0.001"/>
@@ -190,7 +190,7 @@
     </visual>
     <collision>
-      <origin xyz="0.050 0 0.005" rpy="0 0 0"/>
-      <geometry>
-        <box size="0.040 0.120 0.0650"/>
+      <origin xyz="0.043 0 0.005" rpy="0 0 0"/>
+      <geometry>
+        <box size="0.048 0.120 0.0650"/>
       </geometry>
     </collision>
@@ -206,5 +206,5 @@
   <link name="grip_link">
     <visual>
-      <origin xyz="0.0 0.047 0" rpy="0 0 0"/>
+      <origin xyz="0.028 0.0246 0" rpy="0 0 0"/>
       <geometry>
         <mesh filename="package://open_manipulator_description/meshes/chain_link_grip_l.stl" scale="0.001 0.001 0.001"/>
@@ -213,7 +213,7 @@
     </visual>
     <collision>
-      <origin xyz="0.040 0.047 0" rpy="0 0 0"/>
-      <geometry>
-        <box size="0.060 0.025 0.050"/>
+      <origin xyz="0.060 0.030 0" rpy="0 0 0"/>
+      <geometry>
+        <box size="0.065 0.035 0.050"/>
       </geometry>
     </collision>
@@ -230,7 +230,7 @@
     <parent link="link5"/>
     <child link="grip_link"/>
-    <origin xyz="0.071 0.0 0.0" rpy="0 0 0"/>
+    <origin xyz="0.0536 0.0 0.0" rpy="0 0 0"/>
     <axis xyz="0 -1 0"/>
-    <limit velocity="6.5" effort="1000" lower="-0.01" upper="0.035" />
+    <limit velocity="3.5" effort="100" lower="-0.015" upper="0.0105" />
   </joint>
   <!-- Transmission 5 -->
@@ -248,5 +248,5 @@
   <link name="grip_link_sub">
     <visual>
-      <origin xyz="0 -0.047 0" rpy="0 0 0"/>
+      <origin xyz="0.028 -0.0246 0" rpy="0 0 0"/>
       <geometry>
         <mesh filename="package://open_manipulator_description/meshes/chain_link_grip_r.stl" scale="0.001 0.001 0.001"/>
@@ -255,7 +255,7 @@
     </visual>
     <collision>
-      <origin xyz="0.040 -0.047 0" rpy="0 0 0"/>
-      <geometry>
-        <box size="0.060 0.025 0.050"/>
+      <origin xyz="0.060 -0.030 0" rpy="0 0 0"/>
+      <geometry>
+        <box size="0.065 0.035 0.050"/>
       </geometry>
     </collision>
@@ -272,7 +272,7 @@
     <parent link="link5"/>
     <child link="grip_link_sub"/>
-    <origin xyz="0.071 0.0 0" rpy="0 0 0"/>
-    <axis xyz="0 1 0"/>
-    <limit velocity="6.5" effort="1000" lower="-0.01" upper="0.035" />
+    <origin xyz="0.0536 0 0" rpy="0 0 0"/>
+    <axis xyz="0 1 0"/>
+    <limit velocity="3.5" effort="100" lower="-0.015" upper="0.0105" />
   </joint>
   <!-- Transmission 6 -->

File: open_manipulator_with_tb3/urdf/open_manipulator_chain_with_tb3_waffle_pi.urdf.xacro (robot description, xacro)
@@ -15,5 +15,5 @@
   <link name="link1">
     <visual>
-      <origin xyz="0.0 0.0 0.0" rpy="0 0 0"/>
+      <origin xyz="0 0 0" rpy="0 0 0"/>
       <geometry>
         <mesh filename="package://open_manipulator_description/meshes/chain_link1.stl" scale="0.001 0.001 0.001"/>
@@ -39,15 +39,15 @@
     <parent link="link1"/>
     <child link="link2"/>
-    <origin xyz="0.012 0.0 0.036" rpy="0 0 0"/>
+    <origin xyz="0.012 0.0 0.017" rpy="0 0 0"/>
     <axis xyz="0 0 1"/>
     <limit velocity="6.5" effort="1000" lower="${-pi*0.9}" upper="${pi*0.9}" />
   </joint>
   <!-- Transmission 1 -->
-  <transmission name="joint1_trans">
+  <transmission name="tran1">
     <type>transmission_interface/SimpleTransmission</type>
     <joint name="joint1">
       <hardwareInterface>hardware_interface/EffortJointInterface</hardwareInterface>
     </joint>
-    <actuator name="joint1_actuator">
+    <actuator name="motor1">
       <hardwareInterface>hardware_interface/EffortJointInterface</hardwareInterface>
       <mechanicalReduction>1</mechanicalReduction>
@@ -57,5 +57,5 @@
   <link name="link2">
     <visual>
-      <origin xyz="0.0 0.0 0.040" rpy="0 0 0"/>
+      <origin xyz="0 0 0.018" rpy="0 0 0"/>
       <geometry>
         <mesh filename="package://open_manipulator_description/meshes/chain_link2.stl" scale="0.001 0.001 0.001"/>
@@ -64,5 +64,5 @@
     </visual>
     <collision>
-      <origin xyz="0.0 0.0 0.030" rpy="0 0 0"/>
+      <origin xyz="0.0 0.0 0.048" rpy="0 0 0"/>
       <geometry>
         <box size="0.0355 0.0550 0.0515"/>
@@ -81,15 +81,15 @@
     <parent link="link2"/>
     <child link="link3"/>
-    <origin xyz="0.0 0.0 0.040" rpy="0 0 0"/>
+    <origin xyz="0.0 0.0 0.058" rpy="0 0 0"/>
     <axis xyz="0 1 0"/>
     <limit velocity="6.5" effort="1000" lower="${-pi*0.5}" upper="${pi*0.5}" />
   </joint>
   <!-- Transmission 2 -->
-  <transmission name="joint2_trans">
+  <transmission name="tran2">
     <type>transmission_interface/SimpleTransmission</type>
     <joint name="joint2">
       <hardwareInterface>hardware_interface/EffortJointInterface</hardwareInterface>
     </joint>
-    <actuator name="joint2_actuator">
+    <actuator name="motor2">
       <hardwareInterface>hardware_interface/EffortJointInterface</hardwareInterface>
       <mechanicalReduction>1</mechanicalReduction>
@@ -99,5 +99,5 @@
   <link name="link3">
     <visual>
-      <origin xyz="0.022 0 0.122" rpy="0 0 0"/>
+      <origin xyz="0 0 0" rpy="0 0 0"/>
       <geometry>
         <mesh filename="package://open_manipulator_description/meshes/chain_link3.stl" scale="0.001 0.001 0.001"/>
@@ -123,15 +123,15 @@
     <parent link="link3"/>
     <child link="link4"/>
-    <origin xyz="0.022 0 0.122" rpy="0 0 0"/>
-    <axis xyz="0 1 0"/>
-    <limit velocity="6.5" effort="1000" lower="${-pi*0.5}" upper="${pi*0.4}" />
+    <origin xyz="0.024 0 0.128" rpy="0 0 0"/>
+    <axis xyz="0 1 0"/>
+    <limit velocity="6.5" effort="1000" lower="${-pi*0.3}" upper="${pi*0.3}" />
   </joint>
   <!-- Transmission 3 -->
-  <transmission name="joint3_trans">
+  <transmission name="tran3">
     <type>transmission_interface/SimpleTransmission</type>
     <joint name="joint3">
       <hardwareInterface>hardware_interface/EffortJointInterface</hardwareInterface>
     </joint>
-    <actuator name="joint3_actuator">
+    <actuator name="motor3">
       <hardwareInterface>hardware_interface/EffortJointInterface</hardwareInterface>
       <mechanicalReduction>1</mechanicalReduction>
@@ -141,5 +141,5 @@
   <link name="link4">
     <visual>
-      <origin xyz="0.124 0 0.0" rpy="0 0 0"/>
+      <origin xyz="0 0 0" rpy="0 0 0"/>
       <geometry>
         <mesh filename="package://open_manipulator_description/meshes/chain_link4.stl" scale="0.001 0.001 0.001"/>
@@ -148,7 +148,7 @@
     </visual>
     <collision>
-      <origin xyz="0.080 0 0.0" rpy="0 0 0"/>
-      <geometry>
-        <box size="0.110 0.055 0.035"/>
+      <origin xyz="0.065 0 0.0" rpy="0 0 0"/>
+      <geometry>
+        <box size="0.115 0.055 0.035"/>
       </geometry>
     </collision>
@@ -170,10 +170,10 @@
   </joint>
   <!-- Transmission 4 -->
-  <transmission name="joint4_trans">
+  <transmission name="tran4">
     <type>transmission_interface/SimpleTransmission</type>
     <joint name="joint4">
       <hardwareInterface>hardware_interface/EffortJointInterface</hardwareInterface>
     </joint>
-    <actuator name="joint4_actuator">
+    <actuator name="motor4">
       <hardwareInterface>hardware_interface/EffortJointInterface</hardwareInterface>
       <mechanicalReduction>1</mechanicalReduction>
@@ -183,5 +183,5 @@
   <link name="link5">
     <visual>
-      <origin xyz="0.046 0 0" rpy="0 0 0"/>
+      <origin xyz="0 0 0" rpy="0 0 0"/>
       <geometry>
         <mesh filename="package://open_manipulator_description/meshes/chain_link5.stl" scale="0.001 0.001 0.001"/>
@@ -190,7 +190,7 @@
     </visual>
     <collision>
-      <origin xyz="0.050 0 0.005" rpy="0 0 0"/>
-      <geometry>
-        <box size="0.040 0.120 0.0650"/>
+      <origin xyz="0.043 0 0.005" rpy="0 0 0"/>
+      <geometry>
+        <box size="0.048 0.120 0.0650"/>
       </geometry>
     </collision>
@@ -206,5 +206,5 @@
   <link name="grip_link">
     <visual>
-      <origin xyz="0.0 0.047 0" rpy="0 0 0"/>
+      <origin xyz="0.028 0.0246 0" rpy="0 0 0"/>
       <geometry>
         <mesh filename="package://open_manipulator_description/meshes/chain_link_grip_l.stl" scale="0.001 0.001 0.001"/>
@@ -213,7 +213,7 @@
     </visual>
     <collision>
-      <origin xyz="0.040 0.047 0" rpy="0 0 0"/>
-      <geometry>
-        <box size="0.060 0.025 0.050"/>
+      <origin xyz="0.060 0.030 0" rpy="0 0 0"/>
+      <geometry>
+        <box size="0.065 0.035 0.050"/>
       </geometry>
     </collision>
@@ -230,15 +230,15 @@
     <parent link="link5"/>
     <child link="grip_link"/>
-    <origin xyz="0.071 0.0 0.0" rpy="0 0 0"/>
+    <origin xyz="0.0536 0.0 0.0" rpy="0 0 0"/>
     <axis xyz="0 -1 0"/>
-    <limit velocity="6.5" effort="1000" lower="-0.01" upper="0.035" />
+    <limit velocity="3.5" effort="100" lower="-0.015" upper="0.0105" />
   </joint>
   <!-- Transmission 5 -->
-  <transmission name="grip_joint_trans">
+  <transmission name="tran5">
     <type>transmission_interface/SimpleTransmission</type>
     <joint name="grip_joint">
       <hardwareInterface>hardware_interface/EffortJointInterface</hardwareInterface>
     </joint>
-    <actuator name="grip_joint_actuator">
+    <actuator name="motor7">
       <hardwareInterface>hardware_interface/EffortJointInterface</hardwareInterface>
       <mechanicalReduction>1</mechanicalReduction>
@@ -248,5 +248,5 @@
   <link name="grip_link_sub">
     <visual>
-      <origin xyz="0 -0.047 0" rpy="0 0 0"/>
+      <origin xyz="0.028 -0.0246 0" rpy="0 0 0"/>
       <geometry>
         <mesh filename="package://open_manipulator_description/meshes/chain_link_grip_r.stl" scale="0.001 0.001 0.001"/>
@@ -255,7 +255,7 @@
     </visual>
     <collision>
-      <origin xyz="0.040 -0.047 0" rpy="0 0 0"/>
-      <geometry>
-        <box size="0.060 0.025 0.050"/>
+      <origin xyz="0.060 -0.030 0" rpy="0 0 0"/>
+      <geometry>
+        <box size="0.065 0.035 0.050"/>
       </geometry>
     </collision>
@@ -272,15 +272,15 @@
     <parent link="link5"/>
     <child link="grip_link_sub"/>
-    <origin xyz="0.071 0.0 0" rpy="0 0 0"/>
-    <axis xyz="0 1 0"/>
-    <limit velocity="6.5" effort="1000" lower="-0.01" upper="0.035" />
+    <origin xyz="0.0536 0 0" rpy="0 0 0"/>
+    <axis xyz="0 1 0"/>
+    <limit velocity="3.5" effort="100" lower="-0.015" upper="0.0105" />
   </joint>
   <!-- Transmission 6 -->
-  <transmission name="grip_joint_sub_trans">
+  <transmission name="tran6">
     <type>transmission_interface/SimpleTransmission</type>
     <joint name="grip_joint_sub">
       <hardwareInterface>hardware_interface/EffortJointInterface</hardwareInterface>
     </joint>
-    <actuator name="grip_joint_sub_actuator">
+    <actuator name="motor8">
       <hardwareInterface>hardware_interface/EffortJointInterface</hardwareInterface>
       <mechanicalReduction>1</mechanicalReduction>

Commit message: modified joint limit

File: open_manipulator_with_tb3/urdf/open_manipulator_chain_with_tb3_waffle.urdf.xacro (robot description, xacro)
@@ -125,5 +125,5 @@
     <origin xyz="0.024 0 0.128" rpy="0 0 0"/>
     <axis xyz="0 1 0"/>
-    <limit velocity="6.5" effort="1000" lower="${-pi*0.3}" upper="${pi*0.3}" />
+    <limit velocity="6.5" effort="1000" lower="${-pi*0.3}" upper="${pi*0.44}" />
   </joint>
   <!-- Transmission 3 -->

File: open_manipulator_with_tb3/urdf/open_manipulator_chain_with_tb3_waffle_pi.urdf.xacro (robot description, xacro)
@@ -125,5 +125,5 @@
     <origin xyz="0.024 0 0.128" rpy="0 0 0"/>
     <axis xyz="0 1 0"/>
-    <limit velocity="6.5" effort="1000" lower="${-pi*0.3}" upper="${pi*0.3}" />
+    <limit velocity="6.5" effort="1000" lower="${-pi*0.3}" upper="${pi*0.44}" />
   </joint>
   <!-- Transmission 3 -->

Commit message: modified collision models

File: open_manipulator_with_tb3/urdf/open_manipulator_chain_with_tb3_waffle.urdf.xacro (robot description, xacro)
@@ -22,7 +22,7 @@
     </visual>
     <collision>
-      <origin xyz="0.0 0.0 0.017" rpy="0 0 0"/>
-      <geometry>
-        <box size="0.0475 0.0295 0.0340"/>
+      <origin xyz="0 0 0" rpy="0 0 0"/>
+      <geometry>
+        <mesh filename="package://open_manipulator_description/meshes/chain_link1.stl" scale="0.001 0.001 0.001"/>
       </geometry>
     </collision>
@@ -64,7 +64,7 @@
     </visual>
     <collision>
-      <origin xyz="0.0 0.0 0.048" rpy="0 0 0"/>
-      <geometry>
-        <box size="0.0355 0.0550 0.0515"/>
+      <origin xyz="0 0 0.018" rpy="0 0 0"/>
+      <geometry>
+        <mesh filename="package://open_manipulator_description/meshes/chain_link2.stl" scale="0.001 0.001 0.001"/>
       </geometry>
     </collision>
@@ -106,7 +106,7 @@
     </visual>
     <collision>
-      <origin xyz="0.0 0 0.085" rpy="0 0 0"/>
-      <geometry>
-        <box size="0.030 0.055 0.120"/>
+      <origin xyz="0 0 0" rpy="0 0 0"/>
+      <geometry>
+        <mesh filename="package://open_manipulator_description/meshes/chain_link3.stl" scale="0.001 0.001 0.001"/>
       </geometry>
     </collision>
@@ -148,7 +148,7 @@
     </visual>
     <collision>
-      <origin xyz="0.065 0 0.0" rpy="0 0 0"/>
-      <geometry>
-        <box size="0.115 0.055 0.035"/>
+      <origin xyz="0 0 0" rpy="0 0 0"/>
+      <geometry>
+        <mesh filename="package://open_manipulator_description/meshes/chain_link4.stl" scale="0.001 0.001 0.001"/>
       </geometry>
     </collision>
@@ -190,7 +190,7 @@
     </visual>
     <collision>
-      <origin xyz="0.043 0 0.005" rpy="0 0 0"/>
-      <geometry>
-        <box size="0.048 0.120 0.0650"/>
+      <origin xyz="0 0 0" rpy="0 0 0"/>
+      <geometry>
+        <mesh filename="package://open_manipulator_description/meshes/chain_link5.stl" scale="0.001 0.001 0.001"/>
       </geometry>
     </collision>
@@ -213,7 +213,7 @@
     </visual>
     <collision>
-      <origin xyz="0.060 0.033 0" rpy="0 0 0"/>
-      <geometry>
-        <box size="0.065 0.025 0.050"/>
+      <origin xyz="0.028 0.0246 0" rpy="0 0 0"/>
+      <geometry>
+        <mesh filename="package://open_manipulator_description/meshes/chain_link_grip_l.stl" scale="0.001 0.001 0.001"/>
       </geometry>
     </collision>
@@ -255,7 +255,7 @@
     </visual>
     <collision>
-      <origin xyz="0.060 -0.033 0" rpy="0 0 0"/>
-      <geometry>
-        <box size="0.065 0.025 0.050"/>
+      <origin xyz="0.028 -0.0246 0" rpy="0 0 0"/>
+      <geometry>
+        <mesh filename="package://open_manipulator_description/meshes/chain_link_grip_r.stl" scale="0.001 0.001 0.001"/>
       </geometry>
     </collision>

File: open_manipulator_with_tb3/urdf/open_manipulator_chain_with_tb3_waffle_pi.urdf.xacro (robot description, xacro)
@@ -22,7 +22,7 @@
     </visual>
     <collision>
-      <origin xyz="0.0 0.0 0.017" rpy="0 0 0"/>
-      <geometry>
-        <box size="0.0475 0.0295 0.0340"/>
+      <origin xyz="0 0 0" rpy="0 0 0"/>
+      <geometry>
+        <mesh filename="package://open_manipulator_description/meshes/chain_link1.stl" scale="0.001 0.001 0.001"/>
       </geometry>
     </collision>
@@ -64,7 +64,7 @@
     </visual>
     <collision>
-      <origin xyz="0.0 0.0 0.048" rpy="0 0 0"/>
-      <geometry>
-        <box size="0.0355 0.0550 0.0515"/>
+      <origin xyz="0 0 0.018" rpy="0 0 0"/>
+      <geometry>
+        <mesh filename="package://open_manipulator_description/meshes/chain_link2.stl" scale="0.001 0.001 0.001"/>
       </geometry>
     </collision>
@@ -106,7 +106,7 @@
     </visual>
     <collision>
-      <origin xyz="0.0 0 0.085" rpy="0 0 0"/>
-      <geometry>
-        <box size="0.030 0.055 0.120"/>
+      <origin xyz="0 0 0" rpy="0 0 0"/>
+      <geometry>
+        <mesh filename="package://open_manipulator_description/meshes/chain_link3.stl" scale="0.001 0.001 0.001"/>
       </geometry>
     </collision>
@@ -148,7 +148,7 @@
     </visual>
     <collision>
-      <origin xyz="0.065 0 0.0" rpy="0 0 0"/>
-      <geometry>
-        <box size="0.115 0.055 0.035"/>
+      <origin xyz="0 0 0" rpy="0 0 0"/>
+      <geometry>
+        <mesh filename="package://open_manipulator_description/meshes/chain_link4.stl" scale="0.001 0.001 0.001"/>
       </geometry>
     </collision>
@@ -190,7 +190,7 @@
     </visual>
     <collision>
-      <origin xyz="0.043 0 0.005" rpy="0 0 0"/>
-      <geometry>
-        <box size="0.048 0.120 0.0650"/>
+      <origin xyz="0 0 0" rpy="0 0 0"/>
+      <geometry>
+        <mesh filename="package://open_manipulator_description/meshes/chain_link5.stl" scale="0.001 0.001 0.001"/>
       </geometry>
     </collision>
@@ -198,7 +198,7 @@
       <origin xyz="0 0 0" />
       <mass value="0.141" />
-      <inertia ixx="0.1" ixy="0.0" ixz="0.0"
-               iyy="0.1" iyz="0.0"
-               izz="0.1" />
+      <inertia ixx="1" ixy="0.0" ixz="0.0"
+               iyy="1" iyz="0.0"
+               izz="1" />
     </inertial>
   </link>
@@ -213,7 +213,7 @@
     </visual>
     <collision>
-      <origin xyz="0.060 0.033 0" rpy="0 0 0"/>
-      <geometry>
-        <box size="0.065 0.025 0.050"/>
+      <origin xyz="0.028 0.0246 0" rpy="0 0 0"/>
+      <geometry>
+        <mesh filename="package://open_manipulator_description/meshes/chain_link_grip_l.stl" scale="0.001 0.001 0.001"/>
       </geometry>
     </collision>
@@ -221,7 +221,7 @@
       <origin xyz="0 0 0" />
       <mass value="0.017" />
-      <inertia ixx="0.1" ixy="0.0" ixz="0.0"
-               iyy="0.1" iyz="0.0"
-               izz="0.1" />
+      <inertia ixx="1" ixy="0.0" ixz="0.0"
+               iyy="1" iyz="0.0"
+               izz="1" />
     </inertial>
   </link>
@@ -232,5 +232,5 @@
     <origin xyz="0.0536 0.0 0.0" rpy="0 0 0"/>
     <axis xyz="0 -1 0"/>
-    <limit velocity="3.5" effort="100" lower="-0.015" upper="0.0105" />
+    <limit velocity="13.5" effort="10000" lower="-0.015" upper="0.0105" />
   </joint>
   <!-- Transmission 5 -->
@@ -255,7 +255,7 @@
     </visual>
     <collision>
-      <origin xyz="0.060 -0.033 0" rpy="0 0 0"/>
-      <geometry>
-        <box size="0.065 0.025 0.050"/>
+      <origin xyz="0.028 -0.0246 0" rpy="0 0 0"/>
+      <geometry>
+        <mesh filename="package://open_manipulator_description/meshes/chain_link_grip_r.stl" scale="0.001 0.001 0.001"/>
       </geometry>
     </collision>
@@ -274,5 +274,5 @@
     <origin xyz="0.0536 0 0" rpy="0 0 0"/>
     <axis xyz="0 1 0"/>
-    <limit velocity="3.5" effort="100" lower="-0.015" upper="0.0105" />
+    <limit velocity="13.5" effort="10000" lower="-0.015" upper="0.0105" />
   </joint>
   <!-- Transmission 6 -->
