Commit message: add lidar

File: open_manipulator_with_tb3/urdf/open_manipulator_with_tb3_waffle_pi.urdf.xacro (robot description, xacro)
@@ -8,5 +8,6 @@
   <!-- Base fixed joint -->
   <joint name="base_fixed" type="fixed">
-    <origin xyz="-0.005 0.0 0.091" rpy="0 0 0"/>
+<!--    <origin xyz="-0.005 0.0 0.091" rpy="0 0 0"/>-->
+    <origin xyz="-0.084 0.0 0.091" rpy="0 0 0"/>
     <parent link="base_link"/>
     <child link="link1"/>
