Commit message: update inertia

File: open_manipulator_with_tb3/urdf/open_manipulator_with_tb3_waffle.urdf.xacro (robot description, xacro)
@@ -34,4 +34,11 @@
                izz="0.1" />
     </inertial>
+    <!-- <inertial>
+      <origin xyz="3.0876154e-04 0.0000000e+00 -1.2176461e-04" />
+      <mass value="7.9119962e-02" />
+      <inertia ixx="1.2505234e-05" ixy="0.0" ixz="-1.7855208e-07"
+               iyy="2.1898364e-05" iyz="0.0"
+               izz="1.9267361e-05" />
+    </inertial> -->
   </link>
   <!-- Joint 1 -->
@@ -76,4 +83,11 @@
                izz="0.1" />
     </inertial>
+    <!-- <inertial>
+      <origin xyz="-3.0184870e-04 5.4043684e-04 ${0.018 + 2.9433464e-02}" />
+      <mass value="9.8406837e-02" />
+      <inertia ixx="3.4543422e-05" ixy="-1.6031095e-08" ixz="-3.8375155e-07"
+               iyy="3.2689329e-05" iyz="2.8511935e-08"
+               izz="1.8850320e-05" />
+    </inertial> -->
   </link>
   <!--  Joint 2 -->
@@ -118,4 +132,11 @@
                izz="0.1" />
     </inertial>
+    <!-- <inertial>
+      <origin xyz="1.0308393e-02 3.7743363e-04 1.0170197e-01" />
+      <mass value="1.3850917e-01" />
+      <inertia ixx="3.3055381e-04" ixy="-9.7940978e-08" ixz="-3.8505711e-05"
+               iyy="3.4290447e-04" iyz="-1.5717516e-06"
+               izz="6.0346498e-05" />
+    </inertial> -->
   </link>
   <!--  Joint 3 -->
@@ -160,4 +181,11 @@
                izz="0.1" />
     </inertial>
+    <!-- <inertial>
+      <origin xyz="9.0909590e-02 3.8929816e-04 2.2413279e-04" />
+      <mass value="1.3274562e-01" />
+      <inertia ixx="3.0654178e-05" ixy="-1.2764155e-06" ixz="-2.6874417e-07"
+               iyy="2.4230292e-04" iyz="1.1559550e-08"
+               izz="2.5155057e-04" />
+    </inertial> -->
   </link>
   <!--  Joint 4 -->
@@ -202,4 +230,11 @@
                izz="0.1" />
     </inertial>
+    <!-- <inertial>
+      <origin xyz="4.4206755e-02 3.6839985e-07 8.9142216e-03" />
+      <mass value="1.4327573e-01" />
+      <inertia ixx="8.0870749e-05" ixy="0.0" ixz="-1.0157896e-06"
+               iyy="7.5980465e-05" iyz="0.0"
+               izz="9.3127351e-05" />
+    </inertial> -->
   </link>
   <!--  Grip link -->
@@ -225,4 +260,11 @@
                izz="0.1" />
     </inertial>
+    <!-- <inertial>
+      <origin xyz="${0.028 + 8.3720668e-03} ${0.0246 + 9.9696160e-03} -4.2836895e-07" />
+      <mass value="3.2218127e-02" />
+      <inertia ixx="9.5568826e-06" ixy="2.8424644e-06" ixz="-3.2829197e-10"
+               iyy="2.2552871e-05" iyz="-3.1463634e-10"
+               izz="1.7605306e-05" />
+    </inertial> -->
   </link>
   <!--  Grip joint -->
@@ -267,4 +309,11 @@
                izz="0.1" />
     </inertial>
+    <!-- <inertial>
+      <origin xyz="${0.028 + 8.3720668e-03} ${-0.0246 - 9.9696160e-03} -4.2836895e-07" />
+      <mass value="3.2218127e-02" />
+      <inertia ixx="9.5568826e-06" ixy="2.8424644e-06" ixz="-3.2829197e-10"
+               iyy="2.2552871e-05" iyz="-3.1463634e-10"
+               izz="1.7605306e-05" />
+    </inertial> -->
   </link>
   <!--  Grip joint sub -->

File: open_manipulator_with_tb3/urdf/open_manipulator_with_tb3_waffle_pi.urdf.xacro (robot description, xacro)
@@ -34,4 +34,11 @@
                izz="0.1" />
     </inertial>
+    <!-- <inertial>
+      <origin xyz="3.0876154e-04 0.0000000e+00 -1.2176461e-04" />
+      <mass value="7.9119962e-02" />
+      <inertia ixx="1.2505234e-05" ixy="0.0" ixz="-1.7855208e-07"
+               iyy="2.1898364e-05" iyz="0.0"
+               izz="1.9267361e-05" />
+    </inertial> -->
   </link>
   <!-- Joint 1 -->
@@ -76,4 +83,11 @@
                izz="0.1" />
     </inertial>
+    <!-- <inertial>
+      <origin xyz="-3.0184870e-04 5.4043684e-04 ${0.018 + 2.9433464e-02}" />
+      <mass value="9.8406837e-02" />
+      <inertia ixx="3.4543422e-05" ixy="-1.6031095e-08" ixz="-3.8375155e-07"
+               iyy="3.2689329e-05" iyz="2.8511935e-08"
+               izz="1.8850320e-05" />
+    </inertial> -->
   </link>
   <!--  Joint 2 -->
@@ -118,4 +132,11 @@
                izz="0.1" />
     </inertial>
+    <!-- <inertial>
+      <origin xyz="1.0308393e-02 3.7743363e-04 1.0170197e-01" />
+      <mass value="1.3850917e-01" />
+      <inertia ixx="3.3055381e-04" ixy="-9.7940978e-08" ixz="-3.8505711e-05"
+               iyy="3.4290447e-04" iyz="-1.5717516e-06"
+               izz="6.0346498e-05" />
+    </inertial> -->
   </link>
   <!--  Joint 3 -->
@@ -160,4 +181,11 @@
                izz="0.1" />
     </inertial>
+    <!-- <inertial>
+      <origin xyz="9.0909590e-02 3.8929816e-04 2.2413279e-04" />
+      <mass value="1.3274562e-01" />
+      <inertia ixx="3.0654178e-05" ixy="-1.2764155e-06" ixz="-2.6874417e-07"
+               iyy="2.4230292e-04" iyz="1.1559550e-08"
+               izz="2.5155057e-04" />
+    </inertial> -->
   </link>
   <!--  Joint 4 -->
@@ -198,8 +226,15 @@
       <origin xyz="0 0 0" />
       <mass value="0.141" />
-      <inertia ixx="1" ixy="0.0" ixz="0.0"
-               iyy="1" iyz="0.0"
-               izz="1" />
-    </inertial>
+      <inertia ixx="0.1" ixy="0.0" ixz="0.0"
+               iyy="0.1" iyz="0.0"
+               izz="0.1" />
+    </inertial>
+    <!-- <inertial>
+      <origin xyz="4.4206755e-02 3.6839985e-07 8.9142216e-03" />
+      <mass value="1.4327573e-01" />
+      <inertia ixx="8.0870749e-05" ixy="0.0" ixz="-1.0157896e-06"
+               iyy="7.5980465e-05" iyz="0.0"
+               izz="9.3127351e-05" />
+    </inertial> -->
   </link>
   <!--  Grip link -->
@@ -221,8 +256,15 @@
       <origin xyz="0 0 0" />
       <mass value="0.017" />
-      <inertia ixx="1" ixy="0.0" ixz="0.0"
-               iyy="1" iyz="0.0"
-               izz="1" />
-    </inertial>
+      <inertia ixx="0.1" ixy="0.0" ixz="0.0"
+               iyy="0.1" iyz="0.0"
+               izz="0.1" />
+    </inertial>
+    <!-- <inertial>
+      <origin xyz="${0.028 + 8.3720668e-03} ${0.0246 + 9.9696160e-03} -4.2836895e-07" />
+      <mass value="3.2218127e-02" />
+      <inertia ixx="9.5568826e-06" ixy="2.8424644e-06" ixz="-3.2829197e-10"
+               iyy="2.2552871e-05" iyz="-3.1463634e-10"
+               izz="1.7605306e-05" />
+    </inertial> -->
   </link>
   <!--  Grip joint -->
@@ -232,5 +274,5 @@
     <origin xyz="0.0536 0.0 0.0" rpy="0 0 0"/>
     <axis xyz="0 -1 0"/>
-    <limit velocity="13.5" effort="10000" lower="-0.015" upper="0.0105" />
+    <limit velocity="3.5" effort="100" lower="-0.015" upper="0.0105" />
   </joint>
   <!-- Transmission 5 -->
@@ -267,4 +309,11 @@
                izz="0.1" />
     </inertial>
+    <!-- <inertial>
+      <origin xyz="${0.028 + 8.3720668e-03} ${-0.0246 - 9.9696160e-03} -4.2836895e-07" />
+      <mass value="3.2218127e-02" />
+      <inertia ixx="9.5568826e-06" ixy="2.8424644e-06" ixz="-3.2829197e-10"
+               iyy="2.2552871e-05" iyz="-3.1463634e-10"
+               izz="1.7605306e-05" />
+    </inertial> -->
   </link>
   <!--  Grip joint sub -->
@@ -274,5 +323,5 @@
     <origin xyz="0.0536 0 0" rpy="0 0 0"/>
     <axis xyz="0 1 0"/>
-    <limit velocity="13.5" effort="10000" lower="-0.015" upper="0.0105" />
+    <limit velocity="3.5" effort="100" lower="-0.015" upper="0.0105" />
   </joint>
   <!-- Transmission 6 -->

Commit message: update scan param

File: open_manipulator_with_tb3/urdf/open_manipulator_with_tb3_waffle.urdf.xacro (robot description, xacro)
@@ -8,5 +8,5 @@
   <!-- Base fixed joint -->
   <joint name="base_fixed" type="fixed">
-    <origin xyz="-0.005 0.0 0.091" rpy="0 0 0"/>
+    <origin xyz="-0.092 0.0 0.091" rpy="0 0 0"/>
     <parent link="base_link"/>
     <child link="link1"/>

File: open_manipulator_with_tb3/urdf/open_manipulator_with_tb3_waffle_pi.urdf.xacro (robot description, xacro)
@@ -8,6 +8,5 @@
   <!-- Base fixed joint -->
   <joint name="base_fixed" type="fixed">
-<!--    <origin xyz="-0.005 0.0 0.091" rpy="0 0 0"/>-->
-    <origin xyz="-0.084 0.0 0.091" rpy="0 0 0"/>
+    <origin xyz="-0.092 0.0 0.091" rpy="0 0 0"/>
     <parent link="base_link"/>
     <child link="link1"/>

Commit message: change urdf name

File: open_manipulator_with_tb3/urdf/open_manipulator_with_tb3_waffle.urdf.xacro (robot description, xacro)
@@ -3,5 +3,5 @@
 <robot name="open_manipulator_with_tb3" xmlns:xacro="http://www.ros.org/wiki/xacro">
   <!-- Include TurtleBot3 Waffle URDF -->
-  <xacro:include filename="$(find turtlebot3_description)/urdf/turtlebot3_waffle_naked.urdf.xacro" />
+  <xacro:include filename="$(find turtlebot3_description)/urdf/turtlebot3_waffle_for_open_manipulator.urdf.xacro" />
   <!-- Include OpenManipulator Chain Gazebo Parameter -->
   <xacro:include filename="$(find open_manipulator_with_tb3)/urdf/open_manipulator_with_tb3.gazebo.xacro" />

File: open_manipulator_with_tb3/urdf/open_manipulator_with_tb3_waffle_pi.urdf.xacro (robot description, xacro)
@@ -3,5 +3,5 @@
 <robot name="open_manipulator_with_tb3" xmlns:xacro="http://www.ros.org/wiki/xacro">
   <!-- Include TurtleBot3 Waffle URDF -->
-  <xacro:include filename="$(find turtlebot3_description)/urdf/turtlebot3_waffle_pi_naked.urdf.xacro" />
+  <xacro:include filename="$(find turtlebot3_description)/urdf/turtlebot3_waffle_pi_for_open_manipulator.urdf.xacro" />
   <!-- Include OpenManipulator Chain Gazebo Parameter -->
   <xacro:include filename="$(find open_manipulator_with_tb3)/urdf/open_manipulator_with_tb3.gazebo.xacro" />
@@ -11,5 +11,5 @@
     <parent link="base_link"/>
     <child link="link1"/>
-  </joint>
+  </joint>f
   <!-- Link 1 -->
   <link name="link1">
