Commit message: updated urdf files

File: open_manipulator_x_description/urdf/open_manipulator_x_robot.urdf.xacro (robot description, xacro)
@@ -2,7 +2,4 @@
 <!-- OpenManipulator Chain -->
 <robot name="open_manipulator_x" xmlns:xacro="http://ros.org/wiki/xacro">
-  <!-- !!!!!!!!!!!!!!!!!!!!!!!!!!!!!!!! -->
-  <!-- TODO:Xacro files do not work yet -->
-  <!-- !!!!!!!!!!!!!!!!!!!!!!!!!!!!!!!! -->
   <!-- Import Rviz colors -->
   <xacro:include filename="$(find open_manipulator_x_description)/urdf/materials.xacro" />
@@ -13,35 +10,4 @@
   <!-- Import URDF -->
   <xacro:include filename="$(find open_manipulator_x_description)/urdf/open_manipulator_x.urdf.xacro" />
-  <!-- Init colour -->
-  <material name="black">
-    <color rgba="0.0 0.0 0.0 1.0"/>
-  </material>
-  <material name="dark">
-    <color rgba="0.3 0.3 0.3 1.0"/>
-  </material>
-  <material name="light_black">
-    <color rgba="0.4 0.4 0.4 1.0"/>
-  </material>
-  <material name="blue">
-    <color rgba="0.0 0.0 0.8 1.0"/>
-  </material>
-  <material name="green">
-    <color rgba="0.0 0.8 0.0 1.0"/>
-  </material>
-  <material name="grey">
-    <color rgba="0.5 0.5 0.5 1.0"/>
-  </material>
-  <material name="orange">
-    <color rgba="1.0 0.4235 0.0392 1.0"/>
-  </material>
-  <material name="brown">
-    <color rgba="0.8706 0.8118 0.7647 1.0"/>
-  </material>
-  <material name="red">
-    <color rgba="0.8 0.0 0.0 1.0"/>
-  </material>
-  <material name="white">
-    <color rgba="1.0 1.0 1.0 1.0"/>
-  </material>
   <!-- World -->
   <link name="world"/>
@@ -52,4 +18,38 @@
     <child link="link1"/>
   </joint>
+  <!-- !!!!!!!!!!!!!!!!!!!!!!!!!!!!!!!! -->
+  <!-- TODO:Xacro files do not work yet -->
+  <!-- !!!!!!!!!!!!!!!!!!!!!!!!!!!!!!!! -->
+  <!-- Init colour -->
+  <material name="black">
+    <color rgba="0.0 0.0 0.0 1.0"/>
+  </material>
+  <material name="dark">
+    <color rgba="0.3 0.3 0.3 1.0"/>
+  </material>
+  <material name="light_black">
+    <color rgba="0.4 0.4 0.4 1.0"/>
+  </material>
+  <material name="blue">
+    <color rgba="0.0 0.0 0.8 1.0"/>
+  </material>
+  <material name="green">
+    <color rgba="0.0 0.8 0.0 1.0"/>
+  </material>
+  <material name="grey">
+    <color rgba="0.5 0.5 0.5 1.0"/>
+  </material>
+  <material name="orange">
+    <color rgba="1.0 0.4235 0.0392 1.0"/>
+  </material>
+  <material name="brown">
+    <color rgba="0.8706 0.8118 0.7647 1.0"/>
+  </material>
+  <material name="red">
+    <color rgba="0.8 0.0 0.0 1.0"/>
+  </material>
+  <material name="white">
+    <color rgba="1.0 1.0 1.0 1.0"/>
+  </material>
   <!-- Link 1 -->
   <link name="link1">
@@ -98,6 +98,6 @@
       </geometry>
     </collision>
-    <inertial>
-      <origin xyz="3.0184870e-04 5.4043684e-04 0.047433464e-02" />
+     <inertial>
+      <origin xyz="-3.0184870e-04 5.4043684e-04 0.047433464e-02" />
       <mass value="9.8406837e-02" />
       <inertia ixx="3.4543422e-05" ixy="-1.6031095e-08" ixz="-3.8375155e-07"
@@ -199,4 +199,12 @@
     </inertial>
   </link>
+  <!--  Gripper joint -->
+  <joint name="gripper" type="prismatic">
+    <parent link="link5"/>
+    <child link="gripper_link"/>
+    <origin xyz="0.0817 0.021 0.0" rpy="0 0 0"/>
+    <axis xyz="0 1 0"/>
+    <limit velocity="4.8" effort="1" lower="-0.010" upper="0.019" />
+  </joint>
   <!--  Gripper link -->
   <link name="gripper_link">
@@ -222,11 +230,12 @@
     </inertial>
   </link>
-  <!--  Gripper joint -->
-  <joint name="gripper" type="prismatic">
-    <parent link="link5"/>
-    <child link="gripper_link"/>
-    <origin xyz="0.0817 0.021 0.0" rpy="0 0 0"/>
-    <axis xyz="0 1 0"/>
+  <!--  Gripper joint sub -->
+  <joint name="gripper_sub" type="prismatic">
+    <parent link="link5"/>
+    <child link="gripper_link_sub"/>
+    <origin xyz="0.0817 -0.021 0.0" rpy="0 0 0"/>
+    <axis xyz="0 -1 0"/>
     <limit velocity="4.8" effort="1" lower="-0.010" upper="0.019" />
+    <mimic joint="gripper" multiplier="1"/>
   </joint>
   <!--  Gripper link sub -->
@@ -253,13 +262,4 @@
     </inertial>
   </link>
-  <!--  Gripper joint sub -->
-  <joint name="gripper_sub" type="prismatic">
-    <parent link="link5"/>
-    <child link="gripper_link_sub"/>
-    <origin xyz="0.0817 -0.021 0" rpy="0 0 0"/>
-    <axis xyz="0 -1 0"/>
-    <limit velocity="4.8" effort="1" lower="-0.010" upper="0.019" />
-    <mimic joint="gripper" multiplier="1"/>
-  </joint>
   <!-- end effector joint -->
   <joint name="end_effector_joint" type="fixed">
@@ -285,3 +285,11 @@
     </inertial>
   </link>
+  <!-- Realsense Camera Joint Position -->
+  <joint name="camera_joint" type="fixed">
+    <axis xyz="0 1 0" />
+    <origin xyz="0.070 0.032 0.052" rpy="0 0 0"/>
+    <parent link="link5"/>
+    <child link="camera_link"/>
+  </joint>
+  <link name="camera_link"/>
 </robot>

Commit message: updated urdf files

File: open_manipulator_x_description/urdf/open_manipulator_x_robot.urdf.xacro (robot description, xacro)
@@ -21,13 +21,12 @@
   <!-- TODO:Xacro files do not work yet -->
   <!-- !!!!!!!!!!!!!!!!!!!!!!!!!!!!!!!! -->
-  <!-- Init colour -->
   <material name="black">
     <color rgba="0.0 0.0 0.0 1.0"/>
   </material>
-  <material name="dark">
-    <color rgba="0.3 0.3 0.3 1.0"/>
-  </material>
-  <material name="light_black">
-    <color rgba="0.4 0.4 0.4 1.0"/>
+  <material name="white">
+    <color rgba="1.0 1.0 1.0 1.0"/>
+  </material>
+  <material name="red">
+    <color rgba="0.8 0.0 0.0 1.0"/>
   </material>
   <material name="blue">
@@ -41,14 +40,8 @@
   </material>
   <material name="orange">
-    <color rgba="1.0 0.4235 0.0392 1.0"/>
+    <color rgba="${255/255} ${108/255} ${10/255} 1.0"/>
   </material>
   <material name="brown">
-    <color rgba="0.8706 0.8118 0.7647 1.0"/>
-  </material>
-  <material name="red">
-    <color rgba="0.8 0.0 0.0 1.0"/>
-  </material>
-  <material name="white">
-    <color rgba="1.0 1.0 1.0 1.0"/>
+    <color rgba="${222/255} ${207/255} ${195/255} 1.0"/>
   </material>
   <!-- Link 1 -->
