Commit message: Remove obsolete STL files and update URDF/XACRO files for OpenManipulator Y and Follower, including new links and adjustments to inertial properties.

File: open_manipulator_description/urdf/om_y/open_manipulator_y.urdf.xacro (robot description, xacro)
@@ -36,6 +36,6 @@
   </joint>
   <joint name="$(arg prefix)gripper_fixed" type="fixed">
-    <origin xyz="0 -0.05 0" rpy="1.57 1.57 0"/>
-    <parent link="$(arg prefix)link6"/>
+    <origin xyz="0 -0.006 0" rpy="1.57 1.57 0"/>
+    <parent link="$(arg prefix)end_effector_flange_link"/>
     <axis xyz="0 0 0"/>
     <child link="$(arg prefix)rh_p12_rn_base"/>

File: open_manipulator_description/urdf/om_y/open_manipulator_y_arm.urdf.xacro (robot description, xacro)
@@ -1,240 +1,235 @@
-<?xml version="1.0"?>
+<?xml version="1.0" encoding="UTF-8"?>
 <robot xmlns:xacro="http://www.ros.org/wiki/xacro">
-  <xacro:macro name="open_manipulator_y" params="prefix">
-    <xacro:property
-      name="meshes_file_direction"
-      value="package://open_manipulator_description/meshes/om_y/"/>
-    <link name="${prefix}link0">
-      <visual>
-        <origin xyz="0 0 0" rpy="0 0 0"/>
-        <geometry>
-          <mesh filename="${meshes_file_direction}/base_unit.stl" scale="0.001 0.001 0.001"/>
-        </geometry>
-            <material name="grey">
-          <color rgba="0.2 0.2 0.2 1"/>
-        </material>
-      </visual>
-      <collision>
-        <origin xyz="0 0 0" rpy="0 0 0"/>
-        <geometry>
-          <mesh filename="${meshes_file_direction}/base_unit.stl" scale="0.001 0.001 0.001"/>
-        </geometry>
-      </collision>
-       <inertial>
-        <origin xyz="3.0876154e-04 0.0000000e+00 -1.2176461e-04" />
-        <mass value="7.9119962e-02" />
-        <inertia ixx="1.2505234e-05" ixy="0.0" ixz="-1.7855208e-07"
-                 iyy="2.1898364e-05" iyz="0.0"
-                 izz="1.9267361e-05" />
-      </inertial>
-    </link>
-    <joint name="${prefix}joint1" type="revolute">
-      <parent link="${prefix}link0"/>
-      <child link="${prefix}link1"/>
-      <origin xyz="0.0 0.0 0.173" rpy="0 0 0"/>
-      <axis xyz="0 0 1"/>
-      <limit velocity="4.8" effort="1000" lower="${-pi}" upper="${pi}" />
-      <dynamics damping="0.1"/>
-    </joint>
-    <link name="${prefix}link1">
-      <visual>
-        <origin xyz="0 0 0" rpy="0 0 0"/>
-        <geometry>
-          <mesh filename="${meshes_file_direction}/1axis.stl" scale="0.001 0.001 0.001"/>
-        </geometry>
-            <material name="grey">
-          <color rgba="0.2 0.2 0.2 1"/>
-        </material>
-      </visual>
-      <collision>
-        <origin xyz="0 0 0" rpy="0 0 0"/>
-        <geometry>
-          <mesh filename="${meshes_file_direction}/1axis.stl" scale="0.001 0.001 0.001"/>
-        </geometry>
-      </collision>
-       <inertial>
-        <origin xyz="-3.0184870e-04 5.4043684e-04 ${0.018 + 2.9433464e-02}" />
-        <mass value="9.8406837e-02" />
-        <inertia ixx="3.4543422e-05" ixy="-1.6031095e-08" ixz="-3.8375155e-07"
-                 iyy="3.2689329e-05" iyz="2.8511935e-08"
-                 izz="1.8850320e-05" />
-      </inertial>
-    </link>
-    <joint name="${prefix}joint2" type="revolute">
-      <parent link="${prefix}link1"/>
-      <child link="${prefix}link2"/>
-      <origin xyz="0 -0.12 0.0" rpy="0 0 0"/>
-      <axis xyz="0 1 0"/>
-      <limit velocity="4.8" effort="1000" lower="${-pi*0.5}" upper="${pi*0.5}" />
-      <dynamics damping="0.1"/>
-    </joint>
-    <link name="${prefix}link2">
-      <visual>
-        <origin xyz="0 0 0" rpy="0 0 0"/>
-        <geometry>
-          <mesh filename="${meshes_file_direction}/2axis.stl" scale="0.001 0.001 0.001"/>
-        </geometry>
-                <material name="grey">
-          <color rgba="0.2 0.2 0.2 1"/>
-        </material>
-      </visual>
-      <collision>
-        <origin xyz="0 0 0" rpy="0 0 0"/>
-        <geometry>
-          <mesh filename="${meshes_file_direction}/2axis.stl" scale="0.001 0.001 0.001"/>
-        </geometry>
-      </collision>
-       <inertial>
-        <origin xyz="1.0308393e-02 3.7743363e-04 1.0170197e-01" />
-        <mass value="1.3850917e-01" />
-        <inertia ixx="3.3055381e-04" ixy="-9.7940978e-08" ixz="-3.8505711e-05"
-                 iyy="3.4290447e-04" iyz="-1.5717516e-06"
-                 izz="6.0346498e-05" />
-      </inertial>
-    </link>
-    <joint name="${prefix}joint3" type="revolute">
-      <parent link="${prefix}link2"/>
-      <child link="${prefix}link3"/>
-      <origin xyz="0 0.004 0.245" rpy="0 0 0"/>
-      <axis xyz="0 1 0"/>
-      <limit velocity="4.8" effort="1000" lower="${-pi*0.9}" upper="${pi*0.8}" />
-      <dynamics damping="0.1"/>
-    </joint>
-    <link name="${prefix}link3">
-      <visual>
-        <origin xyz="0 0 0" rpy="0 0 0"/>
-        <geometry>
-          <mesh filename="${meshes_file_direction}/3axis.stl" scale="0.001 0.001 0.001"/>
-        </geometry>
-                <material name="grey">
-          <color rgba="0.2 0.2 0.2 1"/>
-        </material>
-      </visual>
-      <collision>
-        <origin xyz="0 0 0" rpy="0 0 0"/>
-        <geometry>
-          <mesh filename="${meshes_file_direction}/3axis.stl" scale="0.001 0.001 0.001"/>
-        </geometry>
-      </collision>
-       <inertial>
-        <origin xyz="9.0909590e-02 3.8929816e-04 2.2413279e-04" />
-        <mass value="1.3274562e-01" />
-        <inertia ixx="3.0654178e-05" ixy="-1.2764155e-06" ixz="-2.6874417e-07"
-                 iyy="2.4230292e-04" iyz="1.1559550e-08"
-                 izz="2.5155057e-04" />
-      </inertial>
-    </link>
-    <joint name="${prefix}joint4" type="revolute">
-      <parent link="${prefix}link3"/>
-      <child link="${prefix}link4"/>
-      <origin xyz="0 0.119 0.2182" rpy="0 0 0"/>
-      <axis xyz="0 1 0"/>
-      <limit velocity="4.8" effort="1000" lower="${-pi*0.8}" upper="${pi*0.8}" />
-      <dynamics damping="0.1"/>
-    </joint>
-    <link name="${prefix}link4">
-      <visual>
-        <origin xyz="0 0 0" rpy="0 0 0"/>
-        <geometry>
-          <mesh filename="${meshes_file_direction}/4axis.stl" scale="0.001 0.001 0.001"/>
-        </geometry>
-                <material name="grey">
-          <color rgba="0.2 0.2 0.2 1"/>
-        </material>
-      </visual>
-      <collision>
-        <origin xyz="0 0 0" rpy="0 0 0"/>
-        <geometry>
-          <mesh filename="${meshes_file_direction}/4axis.stl" scale="0.001 0.001 0.001"/>
-        </geometry>
-      </collision>
-       <inertial>
-        <origin xyz="4.4206755e-02 3.6839985e-07 8.9142216e-03" />
-        <mass value="1.4327573e-01" />
-        <inertia ixx="8.0870749e-05" ixy="0.0" ixz="-1.0157896e-06"
-                 iyy="7.5980465e-05" iyz="0.0"
-                 izz="9.3127351e-05" />
-      </inertial>
-    </link>
-    <joint name="${prefix}joint5" type="revolute">
-      <parent link="${prefix}link4"/>
-      <child link="${prefix}link5"/>
-      <origin xyz="0 -0.115 0" rpy="0 0 0"/>
-      <axis xyz="0 0 1"/>
-      <limit velocity="4.8" effort="1000" lower="${-pi}" upper="${pi}" />
-      <dynamics damping="0.1"/>
-    </joint>
-    <link name="${prefix}link5">
-      <visual>
-        <origin xyz="0 0 0" rpy="0 0 0"/>
-        <geometry>
-          <mesh filename="${meshes_file_direction}/5axis.stl" scale="0.001 0.001 0.001"/>
-        </geometry>
-                <material name="grey">
-          <color rgba="0.2 0.2 0.2 1"/>
-        </material>
-      </visual>
-      <collision>
-        <origin xyz="0 0 0" rpy="0 0 0"/>
-        <geometry>
-          <mesh filename="${meshes_file_direction}/5axis.stl" scale="0.001 0.001 0.001"/>
-        </geometry>
-      </collision>
-       <inertial>
-        <origin xyz="4.4206755e-02 3.6839985e-07 8.9142216e-03" />
-        <mass value="1.4327573e-01" />
-        <inertia ixx="8.0870749e-05" ixy="0.0" ixz="-1.0157896e-06"
-                 iyy="7.5980465e-05" iyz="0.0"
-                 izz="9.3127351e-05" />
-      </inertial>
-    </link>
-    <joint name="${prefix}joint6" type="revolute">
-      <parent link="${prefix}link5"/>
-      <child link="${prefix}link6"/>
-      <origin xyz="0 0 0.1145" rpy="0 0 0"/>
-      <axis xyz="0 1 0"/>
-      <limit velocity="4.8" effort="1000" lower="${-pi*0.5}" upper="${pi*0.5}" />
-      <dynamics damping="0.1"/>
-    </joint>
-    <link name="${prefix}link6">
-      <visual>
-        <origin xyz="0 0 0" rpy="0 0 0"/>
-	    <geometry>
-	      <box size="0.01 0.01 0.01"/>
-	    </geometry>
-        <material name="grey">
-          <color rgba="0.2 0.2 0.2 1"/>
-        </material>
-      </visual>
-      <collision>
-        <origin xyz="0 0 0" rpy="0 0 0"/>
-	    <geometry>
-	      <box size="0.01 0.01 0.01"/>
-	    </geometry>
-      </collision>
-       <inertial>
-        <origin xyz="4.4206755e-02 3.6839985e-07 8.9142216e-03" />
-        <mass value="1.4327573e-01" />
-        <inertia ixx="8.0870749e-05" ixy="0.0" ixz="-1.0157896e-06"
-                 iyy="7.5980465e-05" iyz="0.0"
-                 izz="9.3127351e-05" />
-      </inertial>
-    </link>
-    <joint name="${prefix}end_effector_joint" type="fixed">
-      <parent link="${prefix}link6"/>
-      <child link="${prefix}end_effector_link"/>
-      <origin xyz="0 -0.195 0" rpy="0 0 0"/>
-    </joint>
-    <link name="${prefix}end_effector_link">
-      <visual>
-        <origin xyz="0 0 0" rpy="0 0 0"/>
-        <geometry>
-          <box size="0.01 0.01 0.01" />
-        </geometry>
-        <material name="red">
-          <color rgba="1.0 0.0 0.0 1"/>
-        </material>
-      </visual>
-    </link>
-  </xacro:macro>
+   <xacro:macro name="open_manipulator_y" params="prefix">
+      <xacro:property name="meshes_file_direction" value="package://open_manipulator_description/meshes/om_y/" />
+      <link name="${prefix}link0">
+         <visual>
+            <origin xyz="0 0 0" rpy="0 0 0" />
+            <geometry>
+               <mesh filename="${meshes_file_direction}/base_unit.stl" scale="0.001 0.001 0.001" />
+            </geometry>
+            <material name="grey">
+               <color rgba="0.2 0.2 0.2 1" />
+            </material>
+         </visual>
+         <collision>
+            <origin xyz="0 0 0" rpy="0 0 0" />
+            <geometry>
+               <mesh filename="${meshes_file_direction}/base_unit.stl" scale="0.001 0.001 0.001" />
+            </geometry>
+         </collision>
+         <inertial>
+            <origin xyz="-4.021582400e-03 1.308399100e-03 5.507347000e-02" />
+            <mass value="1.528748600e+00" />
+            <inertia ixx="4.642820300e-03" ixy="4.440553200e-05" ixz="-1.504929600e-04" iyy="4.973695500e-03" iyz="2.075604700e-05" izz="6.407832100e-03" />
+         </inertial>
+      </link>
+      <joint name="${prefix}joint1" type="revolute">
+         <parent link="${prefix}link0" />
+         <child link="${prefix}link1" />
+         <origin xyz="0.0 0.0 0.1715" rpy="0 0 0" />
+         <axis xyz="0 0 1" />
+         <limit velocity="4.8" effort="1000" lower="${-pi*2.0}" upper="${pi*2.0}" />
+         <dynamics damping="0.1" />
+      </joint>
+      <link name="${prefix}link1">
+         <visual>
+            <origin xyz="0 0 0" rpy="0 0 0" />
+            <geometry>
+               <mesh filename="${meshes_file_direction}/link1.stl" scale="0.001 0.001 0.001" />
+            </geometry>
+            <material name="grey">
+               <color rgba="0.2 0.2 0.2 1" />
+            </material>
+         </visual>
+         <collision>
+            <origin xyz="0 0 0" rpy="0 0 0" />
+            <geometry>
+               <mesh filename="${meshes_file_direction}/link1.stl" scale="0.001 0.001 0.001" />
+            </geometry>
+         </collision>
+         <inertial>
+            <origin xyz="-1.106361500e-04 -5.471127000e-03 -1.589773300e-02" />
+            <mass value="2.064883200e+00" />
+            <inertia ixx="3.033219000e-03" ixy="5.179283800e-06" ixz="3.335796100e-06" iyy="2.727672400e-03" iyz="1.793495300e-04" izz="2.282657600e-03" />
+         </inertial>
+      </link>
+      <joint name="${prefix}joint2" type="revolute">
+         <parent link="${prefix}link1" />
+         <child link="${prefix}link2" />
+         <origin xyz="0 -0.1215 0.0" rpy="0 0 0" />
+         <axis xyz="0 1 0" />
+         <limit velocity="4.8" effort="1000" lower="${-pi*2.0}" upper="${pi*2.0}" />
+         <dynamics damping="0.1" />
+      </joint>
+      <link name="${prefix}link2">
+         <visual>
+            <origin xyz="0 0 0" rpy="0 0 0" />
+            <geometry>
+               <mesh filename="${meshes_file_direction}/link2.stl" scale="0.001 0.001 0.001" />
+            </geometry>
+            <material name="grey">
+               <color rgba="0.2 0.2 0.2 1" />
+            </material>
+         </visual>
+         <collision>
+            <origin xyz="0 0 0" rpy="0 0 0" />
+            <geometry>
+               <mesh filename="${meshes_file_direction}/link2.stl" scale="0.001 0.001 0.001" />
+            </geometry>
+         </collision>
+         <inertial>
+            <origin xyz="1.140537900e-05 1.618424400e-02 1.036063400e-01" />
+            <mass value="3.679539500e+00" />
+            <inertia ixx="5.173191800e-02" ixy="2.395881900e-06" ixz="5.789396000e-05" iyy="5.035340100e-02" iyz="-4.382571600e-04" izz="4.501436000e-03" />
+         </inertial>
+      </link>
+      <joint name="${prefix}joint3" type="revolute">
+         <parent link="${prefix}link2" />
+         <child link="${prefix}link3" />
+         <origin xyz="0 0 0.247" rpy="0 0 0" />
+         <axis xyz="0 1 0" />
+         <limit velocity="4.8" effort="1000" lower="${-pi*2.0}" upper="${pi*2.0}" />
+         <dynamics damping="0.1" />
+      </joint>
+      <link name="${prefix}link3">
+         <visual>
+            <origin xyz="0 0 0" rpy="0 0 0" />
+            <geometry>
+               <mesh filename="${meshes_file_direction}/link3.stl" scale="0.001 0.001 0.001" />
+            </geometry>
+            <material name="grey">
+               <color rgba="0.2 0.2 0.2 1" />
+            </material>
+         </visual>
+         <collision>
+            <origin xyz="0 0 0" rpy="0 0 0" />
+            <geometry>
+               <mesh filename="${meshes_file_direction}/link3.stl" scale="0.001 0.001 0.001" />
+            </geometry>
+         </collision>
+         <inertial>
+            <origin xyz="7.814868900e-05 1.071848100e-01 1.411726700e-01" />
+            <mass value="2.386591600e+00" />
+            <inertia ixx="2.269439900e-02" ixy="-9.414242800e-07" ixz="-1.855175700e-05" iyy="2.192008700e-02" iyz="1.917938700e-04" izz="2.776155900e-03" />
+         </inertial>
+      </link>
+      <joint name="${prefix}joint4" type="revolute">
+         <parent link="${prefix}link3" />
+         <child link="${prefix}link4" />
+         <origin xyz="0 0.1215 0.2195" rpy="0 0 0" />
+         <axis xyz="0 1 0" />
+         <limit velocity="4.8" effort="1000" lower="${-pi*2.0}" upper="${pi*2.0}" />
+         <dynamics damping="0.1" />
+      </joint>
+      <link name="${prefix}link4">
+         <visual>
+            <origin xyz="0 0 0" rpy="0 0 0" />
+            <geometry>
+               <mesh filename="${meshes_file_direction}/link4.stl" scale="0.001 0.001 0.001" />
+            </geometry>
+            <material name="grey">
+               <color rgba="0.2 0.2 0.2 1" />
+            </material>
+         </visual>
+         <collision>
+            <origin xyz="0 0 0" rpy="0 0 0" />
+            <geometry>
+               <mesh filename="${meshes_file_direction}/link4.stl" scale="0.001 0.001 0.001" />
+            </geometry>
+         </collision>
+         <inertial>
+            <origin xyz="-1.331825600e-04 -1.074666700e-01 1.909068800e-02" />
+            <mass value="1.400234700e+00" />
+            <inertia ixx="1.754567900e-03" ixy="-4.586337900e-06" ixz="-1.775914200e-06" iyy="1.565214700e-03" iyz="1.533991300e-04" izz="1.215983900e-03" />
+         </inertial>
+      </link>
+      <joint name="${prefix}joint5" type="revolute">
+         <parent link="${prefix}link4" />
+         <child link="${prefix}link5" />
+         <origin xyz="0 -0.113 0" rpy="0 0 0" />
+         <axis xyz="0 0 1" />
+         <limit velocity="4.8" effort="1000" lower="${-pi*2.0}" upper="${pi*2.0}" />
+         <dynamics damping="0.1" />
+      </joint>
+      <link name="${prefix}link5">
+         <visual>
+            <origin xyz="0 0 0" rpy="0 0 0" />
+            <geometry>
+               <mesh filename="${meshes_file_direction}/link5.stl" scale="0.001 0.001 0.001" />
+            </geometry>
+            <material name="grey">
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