Commit message: Remove obsolete STL files and update URDF/XACRO files for OpenManipulator Y and Follower, including new links and adjustments to inertial properties.

File: open_manipulator_description/urdf/om_y/open_manipulator_y_follower.urdf.xacro (robot description, xacro)
@@ -1,232 +1,235 @@
-<?xml version="1.0"?>
+<?xml version="1.0" encoding="UTF-8"?>
 <robot xmlns:xacro="http://www.ros.org/wiki/xacro">
-  <xacro:macro name="open_manipulator_y" params="prefix">
-    <xacro:property
-      name="meshes_file_direction"
-      value="package://open_manipulator_description/meshes/om_y_follower"/>
-    <link name="${prefix}link0">
-      <visual>
-        <origin xyz="0 0 0" rpy="0 0 0"/>
-        <geometry>
-          <mesh filename="${meshes_file_direction}/base_link.stl" scale="0.001 0.001 0.001"/>
-        </geometry>
-        <material name="grey">
-          <color rgba="0.2 0.2 0.2 1"/>
-        </material>      </visual>
-      <collision>
-        <origin xyz="0 0 0" rpy="0 0 0"/>
-        <geometry>
-          <mesh filename="${meshes_file_direction}/base_link.stl" scale="0.001 0.001 0.001"/>
-        </geometry>
-      </collision>
-      <inertial>
-        <origin xyz="-9.9252667e-03 5.7283832e-03 1.9646428e-02" />
-        <mass value="8.2109029e-01" />
-        <inertia ixx="1.1221867e-03" ixy="1.5808720e-04" ixz="-1.3545719e-04"
-                  iyy="1.1909942e-03" iyz="6.8527024e-05"
-                  izz="1.8565038e-03" />
-      </inertial>
-    </link>
-    <joint name="${prefix}joint1" type="revolute">
-      <parent link="${prefix}link0"/>
-      <child link="${prefix}link1"/>
-      <origin xyz="0 0 0.1095" rpy="0 0 0"/>
-      <axis xyz="0 0 1"/>
-      <limit velocity="4.8" effort="1000" lower="${-pi}" upper="${pi}" />
-      <dynamics damping="0.1"/>
-    </joint>
-    <link name="${prefix}link1">
-      <visual>
-        <origin xyz="0 0 0" rpy="0 0 0"/>
-        <geometry>
-          <mesh filename="${meshes_file_direction}/link1.stl" scale="0.001 0.001 0.001"/>
-        </geometry>
-        <material name="grey">
-          <color rgba="0.2 0.2 0.2 1"/>
-        </material>      </visual>
-      <collision>
-        <origin xyz="0 0 0" rpy="0 0 0"/>
-        <geometry>
-          <mesh filename="${meshes_file_direction}/link1.stl" scale="0.001 0.001 0.001"/>
-        </geometry>
-      </collision>
-      <inertial>
-        <origin xyz="-1.1644167e-04 -5.6674143e-03 -1.8215700e-02" />
-        <mass value="1.9612825e+00" />
-        <inertia ixx="2.6855127e-03" ixy="5.1207735e-06" ixz="3.4623807e-06"
-                 iyy="2.4500716e-03" iyz="2.0132042e-04"
-                 izz="2.0463416e-03" />
-      </inertial>
-    </link>
-    <joint name="${prefix}joint2" type="revolute">
-      <parent link="${prefix}link1"/>
-      <child link="${prefix}link2"/>
-      <origin xyz="0 -0.12 0" rpy="0 0 0"/>
-      <axis xyz="0 1 0"/>
-      <limit velocity="4.8" effort="1000" lower="${-pi*0.5}" upper="${pi*0.5}" />
-      <dynamics damping="0.1"/>
-    </joint>
-    <link name="${prefix}link2">
-      <visual>
-        <origin xyz="0 0 0" rpy="0 0 0"/>
-        <geometry>
-          <mesh filename="${meshes_file_direction}/link2.stl" scale="0.001 0.001 0.001"/>
-        </geometry>
-        <material name="grey">
-          <color rgba="0.2 0.2 0.2 1"/>
-        </material>      </visual>
-      <collision>
-        <origin xyz="0 0 0" rpy="0 0 0"/>
-        <geometry>
-          <mesh filename="${meshes_file_direction}/link2.stl" scale="0.001 0.001 0.001"/>
-        </geometry>
-      </collision>
-      <inertial>
-        <origin xyz="1.1553105e-05 1.7742026e-02 1.0293555e-01" />
-        <mass value="3.6177931e+00" />
-        <inertia ixx="4.7663982e-02" ixy="2.3686863e-06" ixz="5.7279093e-05"
-                 iyy="4.6409792e-02" iyz="-3.5412923e-04"
-                 izz="4.1114936e-03" />
-      </inertial>
-    </link>
-    <joint name="${prefix}joint3" type="revolute">
-      <parent link="${prefix}link2"/>
-      <child link="${prefix}link3"/>
-      <origin xyz="0 0 0.245" rpy="0 0 0"/>
-      <axis xyz="0 1 0"/>
-      <limit velocity="4.8" effort="1000" lower="${-pi}" upper="${pi}" />
-      <dynamics damping="0.1"/>
-    </joint>
-    <link name="${prefix}link3">
-      <visual>
-        <origin xyz="0 0 0" rpy="0 0 0"/>
-        <geometry>
-          <mesh filename="${meshes_file_direction}/link3.stl" scale="0.001 0.001 0.001"/>
-        </geometry>
-        <material name="grey">
-          <color rgba="0.2 0.2 0.2 1"/>
-        </material>      </visual>
-      <collision>
-        <origin xyz="0 0 0" rpy="0 0 0"/>
-        <geometry>
-          <mesh filename="${meshes_file_direction}/link3.stl" scale="0.001 0.001 0.001"/>
-        </geometry>
-      </collision>
-      <inertial>
-        <origin xyz="8.1034250e-05 1.0648979e-01 1.4052376e-01" />
-        <mass value="2.3114312e+00" />
-        <inertia ixx="2.0523222e-02" ixy="-1.5172383e-06" ixz="-1.7492562e-05"
-                 iyy="1.9803879e-02" iyz="5.0926723e-04"
-                 izz="2.5171921e-03" />
-      </inertial>
-    </link>
-    <joint name="${prefix}joint4" type="revolute">
-      <parent link="${prefix}link3"/>
-      <child link="${prefix}link4"/>
-      <origin xyz="0 0.124 0.2185" rpy="0 0 0"/>
-      <axis xyz="0 1 0"/>
-      <limit velocity="4.8" effort="1000" lower="${-pi}" upper="${pi}" />
-      <dynamics damping="0.1"/>
-    </joint>
-    <link name="${prefix}link4">
-      <visual>
-        <origin xyz="0 0 0" rpy="0 0 0"/>
-        <geometry>
-          <mesh filename="${meshes_file_direction}/link4.stl" scale="0.001 0.001 0.001"/>
-        </geometry>
-        <material name="grey">
-          <color rgba="0.2 0.2 0.2 1"/>
-        </material>      </visual>
-      <collision>
-        <origin xyz="0 0 0" rpy="0 0 0"/>
-        <geometry>
-          <mesh filename="${meshes_file_direction}/link4.stl" scale="0.001 0.001 0.001"/>
-        </geometry>
-      </collision>
-      <inertial>
-        <origin xyz="-1.4269552e-04 -1.0859083e-01 2.1737711e-02" />
-        <mass value="1.3072456e+00" />
-        <inertia ixx="1.5128575e-03" ixy="-4.5495421e-06" ixz="-2.6871200e-06"
-                 iyy="1.3563546e-03" iyz="1.6468450e-04"
-                 izz="1.0617924e-03" />
-      </inertial>
-    </link>
-    <joint name="${prefix}joint5" type="revolute">
-      <parent link="${prefix}link4"/>
-      <child link="${prefix}link5"/>
-      <origin xyz="0 -0.1145 0" rpy="0 0 0"/>
-      <axis xyz="0 0 1"/>
-      <limit velocity="4.8" effort="1000" lower="${-pi}" upper="${pi}" />
-      <dynamics damping="0.1"/>
-    </joint>
-    <link name="${prefix}link5">
-      <visual>
-        <origin xyz="0 0 0" rpy="0 0 0"/>
-        <geometry>
-          <mesh filename="${meshes_file_direction}/link5.stl" scale="0.001 0.001 0.001"/>
-        </geometry>
-        <material name="grey">
-          <color rgba="0.2 0.2 0.2 1"/>
-        </material>      </visual>
-      <collision>
-        <origin xyz="0 0 0" rpy="0 0 0"/>
-        <geometry>
-          <mesh filename="${meshes_file_direction}/link5.stl" scale="0.001 0.001 0.001"/>
-        </geometry>
-      </collision>
-      <inertial>
-        <origin xyz="1.4269553e-04 -2.1737711e-02 1.0859083e-01" />
-        <mass value="1.3072456e+00" />
-        <inertia ixx="1.5128575e-03" ixy="-2.6871201e-06" ixz="-4.5495419e-06"
-                 iyy="1.0617924e-03" iyz="1.6468450e-04"
-                 izz="1.3563546e-03" />
-      </inertial>
-    </link>
-    <joint name="${prefix}joint6" type="revolute">
-      <parent link="${prefix}link5"/>
-      <child link="${prefix}link6"/>
-      <origin xyz="0 0 0.1145" rpy="0 0 0"/>
-      <axis xyz="0 1 0"/>
-      <limit velocity="4.8" effort="1000" lower="${-pi}" upper="${pi}" />
-      <dynamics damping="0.1"/>
-    </joint>
-    <link name="${prefix}link6">
-      <visual>
-        <origin xyz="0 0 0" rpy="0 0 0"/>
-        <geometry>
-          <mesh filename="${meshes_file_direction}/link6.stl" scale="0.001 0.001 0.001"/>
-        </geometry>
-        <material name="grey">
-          <color rgba="0.2 0.2 0.2 1"/>
-        </material>      </visual>
-      <collision>
-        <origin xyz="0 0 0" rpy="0 0 0"/>
-        <geometry>
-          <mesh filename="${meshes_file_direction}/link6.stl" scale="0.001 0.001 0.001"/>
-        </geometry>
-      </collision>
-      <inertial>
-        <origin xyz="0.0000000e+00 -6.4771193e-02 0.0000000e+00" />
-        <mass value="0" />
-        <inertia ixx="7.1274204e-03" ixy="0.0000000e+00" ixz="-1.4218045e-06"
-                 iyy="1.4682178e-02" iyz="0.0000000e+00"
-                 izz="8.2444760e-03" />
-      </inertial>
-    </link>
-    <joint name="${prefix}end_effector_joint" type="fixed">
-      <parent link="${prefix}link6"/>
-      <child link="${prefix}end_effector_link"/>
-      <origin xyz="0 -0.195 0" rpy="0 0 0"/>
-    </joint>
-    <link name="${prefix}end_effector_link">
-      <visual>
-        <origin xyz="0 0 0" rpy="0 0 0"/>
-        <geometry>
-          <box size="0.01 0.01 0.01" />
-        </geometry>
-        <material name="red">
-          <color rgba="1.0 0.0 0.0 1"/>
-        </material>       </visual>
-    </link>
-  </xacro:macro>
+   <xacro:macro name="open_manipulator_y" params="prefix">
+      <xacro:property name="meshes_file_direction" value="package://open_manipulator_description/meshes/om_y/" />
+      <link name="${prefix}link0">
+         <visual>
+            <origin xyz="0 0 0" rpy="0 0 0" />
+            <geometry>
+               <mesh filename="${meshes_file_direction}/base_unit.stl" scale="0.001 0.001 0.001" />
+            </geometry>
+            <material name="grey">
+               <color rgba="0.2 0.2 0.2 1" />
+            </material>
+         </visual>
+         <collision>
+            <origin xyz="0 0 0" rpy="0 0 0" />
+            <geometry>
+               <mesh filename="${meshes_file_direction}/base_unit.stl" scale="0.001 0.001 0.001" />
+            </geometry>
+         </collision>
+         <inertial>
+            <origin xyz="-4.021582400e-03 1.308399100e-03 5.507347000e-02" />
+            <mass value="1.528748600e+00" />
+            <inertia ixx="4.642820300e-03" ixy="4.440553200e-05" ixz="-1.504929600e-04" iyy="4.973695500e-03" iyz="2.075604700e-05" izz="6.407832100e-03" />
+         </inertial>
+      </link>
+      <joint name="${prefix}joint1" type="revolute">
+         <parent link="${prefix}link0" />
+         <child link="${prefix}link1" />
+         <origin xyz="0.0 0.0 0.1715" rpy="0 0 0" />
+         <axis xyz="0 0 1" />
+         <limit velocity="4.8" effort="1000" lower="${-pi*2.0}" upper="${pi*2.0}" />
+         <dynamics damping="0.1" />
+      </joint>
+      <link name="${prefix}link1">
+         <visual>
+            <origin xyz="0 0 0" rpy="0 0 0" />
+            <geometry>
+               <mesh filename="${meshes_file_direction}/link1.stl" scale="0.001 0.001 0.001" />
+            </geometry>
+            <material name="grey">
+               <color rgba="0.2 0.2 0.2 1" />
+            </material>
+         </visual>
+         <collision>
+            <origin xyz="0 0 0" rpy="0 0 0" />
+            <geometry>
+               <mesh filename="${meshes_file_direction}/link1.stl" scale="0.001 0.001 0.001" />
+            </geometry>
+         </collision>
+         <inertial>
+            <origin xyz="-1.106361500e-04 -5.471127000e-03 -1.589773300e-02" />
+            <mass value="2.064883200e+00" />
+            <inertia ixx="3.033219000e-03" ixy="5.179283800e-06" ixz="3.335796100e-06" iyy="2.727672400e-03" iyz="1.793495300e-04" izz="2.282657600e-03" />
+         </inertial>
+      </link>
+      <joint name="${prefix}joint2" type="revolute">
+         <parent link="${prefix}link1" />
+         <child link="${prefix}link2" />
+         <origin xyz="0 -0.1215 0.0" rpy="0 0 0" />
+         <axis xyz="0 1 0" />
+         <limit velocity="4.8" effort="1000" lower="${-pi*2.0}" upper="${pi*2.0}" />
+         <dynamics damping="0.1" />
+      </joint>
+      <link name="${prefix}link2">
+         <visual>
+            <origin xyz="0 0 0" rpy="0 0 0" />
+            <geometry>
+               <mesh filename="${meshes_file_direction}/link2.stl" scale="0.001 0.001 0.001" />
+            </geometry>
+            <material name="grey">
+               <color rgba="0.2 0.2 0.2 1" />
+            </material>
+         </visual>
+         <collision>
+            <origin xyz="0 0 0" rpy="0 0 0" />
+            <geometry>
+               <mesh filename="${meshes_file_direction}/link2.stl" scale="0.001 0.001 0.001" />
+            </geometry>
+         </collision>
+         <inertial>
+            <origin xyz="1.140537900e-05 1.618424400e-02 1.036063400e-01" />
+            <mass value="3.679539500e+00" />
+            <inertia ixx="5.173191800e-02" ixy="2.395881900e-06" ixz="5.789396000e-05" iyy="5.035340100e-02" iyz="-4.382571600e-04" izz="4.501436000e-03" />
+         </inertial>
+      </link>
+      <joint name="${prefix}joint3" type="revolute">
+         <parent link="${prefix}link2" />
+         <child link="${prefix}link3" />
+         <origin xyz="0 0 0.247" rpy="0 0 0" />
+         <axis xyz="0 1 0" />
+         <limit velocity="4.8" effort="1000" lower="${-pi*2.0}" upper="${pi*2.0}" />
+         <dynamics damping="0.1" />
+      </joint>
+      <link name="${prefix}link3">
+         <visual>
+            <origin xyz="0 0 0" rpy="0 0 0" />
+            <geometry>
+               <mesh filename="${meshes_file_direction}/link3.stl" scale="0.001 0.001 0.001" />
+            </geometry>
+            <material name="grey">
+               <color rgba="0.2 0.2 0.2 1" />
+            </material>
+         </visual>
+         <collision>
+            <origin xyz="0 0 0" rpy="0 0 0" />
+            <geometry>
+               <mesh filename="${meshes_file_direction}/link3.stl" scale="0.001 0.001 0.001" />
+            </geometry>
+         </collision>
+         <inertial>
+            <origin xyz="7.814868900e-05 1.071848100e-01 1.411726700e-01" />
+            <mass value="2.386591600e+00" />
+            <inertia ixx="2.269439900e-02" ixy="-9.414242800e-07" ixz="-1.855175700e-05" iyy="2.192008700e-02" iyz="1.917938700e-04" izz="2.776155900e-03" />
+         </inertial>
+      </link>
+      <joint name="${prefix}joint4" type="revolute">
+         <parent link="${prefix}link3" />
+         <child link="${prefix}link4" />
+         <origin xyz="0 0.1215 0.2195" rpy="0 0 0" />
+         <axis xyz="0 1 0" />
+         <limit velocity="4.8" effort="1000" lower="${-pi*2.0}" upper="${pi*2.0}" />
+         <dynamics damping="0.1" />
+      </joint>
+      <link name="${prefix}link4">
+         <visual>
+            <origin xyz="0 0 0" rpy="0 0 0" />
+            <geometry>
+               <mesh filename="${meshes_file_direction}/link4.stl" scale="0.001 0.001 0.001" />
+            </geometry>
+            <material name="grey">
+               <color rgba="0.2 0.2 0.2 1" />
+            </material>
+         </visual>
+         <collision>
+            <origin xyz="0 0 0" rpy="0 0 0" />
+            <geometry>
+               <mesh filename="${meshes_file_direction}/link4.stl" scale="0.001 0.001 0.001" />
+            </geometry>
+         </collision>
+         <inertial>
+            <origin xyz="-1.331825600e-04 -1.074666700e-01 1.909068800e-02" />
+            <mass value="1.400234700e+00" />
+            <inertia ixx="1.754567900e-03" ixy="-4.586337900e-06" ixz="-1.775914200e-06" iyy="1.565214700e-03" iyz="1.533991300e-04" izz="1.215983900e-03" />
+         </inertial>
+      </link>
+      <joint name="${prefix}joint5" type="revolute">
+         <parent link="${prefix}link4" />
+         <child link="${prefix}link5" />
+         <origin xyz="0 -0.113 0" rpy="0 0 0" />
+         <axis xyz="0 0 1" />
+         <limit velocity="4.8" effort="1000" lower="${-pi*2.0}" upper="${pi*2.0}" />
+         <dynamics damping="0.1" />
+      </joint>
+      <link name="${prefix}link5">
+         <visual>
+            <origin xyz="0 0 0" rpy="0 0 0" />
+            <geometry>
+               <mesh filename="${meshes_file_direction}/link5.stl" scale="0.001 0.001 0.001" />
+            </geometry>
+            <material name="grey">
+               <color rgba="0.2 0.2 0.2 1" />
+            </material>
+         </visual>
+         <collision>
+            <origin xyz="0 0 0" rpy="0 0 0" />
+            <geometry>
+               <mesh filename="${meshes_file_direction}/link5.stl" scale="0.001 0.001 0.001" />
+            </geometry>
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
File: open_manipulator_description/urdf/rh_p12_rn_a.urdf.xacro (robot description, xacro)
@@ -26,5 +26,5 @@
         <origin xyz="0.000 0.000 0.032" rpy="0 0 0"/>
         <mass value="0.236"/>
-        <inertia ixx="1.0" ixy="0.0" ixz="0.0" iyy="1.0" iyz="0.0" izz="1.0" />
+        <inertia ixx="0.000001" ixy="0.0" ixz="0.0" iyy="0.000001" iyz="0.0" izz="0.000001" />
       </inertial>
     </link>
@@ -58,5 +58,5 @@
         <origin xyz="0.000 0.034 0.004" rpy="0 0 0"/>
         <mass value="0.068"/>
-        <inertia ixx="1.0" ixy="0.0" ixz="0.0" iyy="1.0" iyz="0.0" izz="1.0" />
+        <inertia ixx="0.000001" ixy="0.0" ixz="0.0" iyy="0.000001" iyz="0.0" izz="0.000001" />
       </inertial>
     </link>
@@ -91,5 +91,5 @@
         <origin xyz="0.000 0.006 0.011" rpy="0 0 0"/>
         <mass value="0.022"/>
-        <inertia ixx="1.0" ixy="0.0" ixz="0.0" iyy="1.0" iyz="0.0" izz="1.0" />
+        <inertia ixx="0.000001" ixy="0.0" ixz="0.0" iyy="0.000001" iyz="0.0" izz="0.000001" />
       </inertial>
     </link>
@@ -124,5 +124,5 @@
         <origin xyz="0.000 -0.034 0.004" rpy="0 0 0"/>
         <mass value="0.068"/>
-        <inertia ixx="1.0" ixy="0.0" ixz="0.0" iyy="1.0" iyz="0.0" izz="1.0" />
+        <inertia ixx="0.000001" ixy="0.0" ixz="0.0" iyy="0.000001" iyz="0.0" izz="0.000001" />
       </inertial>
     </link>
@@ -157,5 +157,5 @@
         <origin xyz="0.000 -0.006 0.011" rpy="0 0 0"/>
         <mass value="0.022"/>
-        <inertia ixx="1.0" ixy="0.0" ixz="0.0" iyy="1.0" iyz="0.0" izz="1.0" />
+        <inertia ixx="0.000001" ixy="0.0" ixz="0.0" iyy="0.000001" iyz="0.0" izz="0.000001" />
       </inertial>
     </link>
