Commit message: new urdf

File: open_manipulator_description/urdf/om_y/open_manipulator_y_follower.urdf (robot description, URDF)
Before this commit: robot open_manipulator_y, 8 links, 7 joints
Links:
- added link rh_p12_rn_base, mass 0.236; collision mesh filename=package://open_manipulator_description/meshes/rh_p12_rn_a/b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 scale=0.001 0.001 0.001; visual mesh filename=package://open_manipulator_description/meshes/rh_p12_rn_a/b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 scale=0.001 0.001 0.001
- added link rh_p12_rn_l1, mass 0.068; collision mesh filename=package://open_manipulator_description/meshes/rh_p12_rn_a/l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 scale=0.001 0.001 0.001; visual mesh filename=package://open_manipulator_description/meshes/rh_p12_rn_a/l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 scale=0.001 0.001 0.001
- added link rh_p12_rn_l2, mass 0.022; collision mesh filename=package://open_manipulator_description/meshes/rh_p12_rn_a/l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 scale=0.001 0.001 0.001; visual mesh filename=package://open_manipulator_description/meshes/rh_p12_rn_a/l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 scale=0.001 0.001 0.001
- added link rh_p12_rn_r1, mass 0.068; collision mesh filename=package://open_manipulator_description/meshes/rh_p12_rn_a/r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 scale=0.001 0.001 0.001; visual mesh filename=package://open_manipulator_description/meshes/rh_p12_rn_a/r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 scale=0.001 0.001 0.001
- added link rh_p12_rn_r2, mass 0.022; collision mesh filename=package://open_manipulator_description/meshes/rh_p12_rn_a/r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 scale=0.001 0.001 0.001; visual mesh filename=package://open_manipulator_description/meshes/rh_p12_rn_a/r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 scale=0.001 0.001 0.001
Joints:
- added joint gripper_fixed: type fixed, parent end_effector_flange_link, child rh_p12_rn_base, origin xyz=0 -0.006 0 rpy=1.57 1.57 0, axis 0 0 0
- added joint rh_l1: type revolute, parent rh_p12_rn_base, child rh_p12_rn_l1, origin xyz=0.0 -0.008 0.048 rpy=0 0 0, axis -1 0 0, limit lower=0.0 upper=1.1 effort=1000 velocity=6.5, mimic joint=rh_r1_joint multiplier=1
- added joint rh_l2: type revolute, parent rh_p12_rn_l1, child rh_p12_rn_l2, origin xyz=0.0 -0.0493634 0.0285 rpy=0 0 0, axis 1 0 0, limit lower=0.0 upper=1.0 effort=1000 velocity=6.5, mimic joint=rh_r1_joint multiplier=1
- added joint rh_r1_joint: type revolute, parent rh_p12_rn_base, child rh_p12_rn_r1, origin xyz=0.0 0.008 0.048 rpy=0 0 0, axis 1 0 0, limit lower=0.0 upper=1.1 effort=1000 velocity=6.5
- added joint rh_r2: type revolute, parent rh_p12_rn_r1, child rh_p12_rn_r2, origin xyz=0.0 0.0493634 0.0285 rpy=0 0 0, axis -1 0 0, limit lower=0.0 upper=1.0 effort=1000 velocity=6.5, mimic joint=rh_r1_joint multiplier=1
