Commit message: Added self collision function
Signed-off-by: Sungho Woo <wsh@robotis.com>

File: open_manipulator_description/urdf/om_y/open_manipulator_y_arm.urdf.xacro (robot description, xacro)
@@ -14,7 +14,7 @@
          </visual>
          <collision>
-            <origin xyz="0 0 0" rpy="0 0 0" />
-            <geometry>
-               <mesh filename="${meshes_file_direction}/base_unit.stl" scale="0.001 0.001 0.001" />
+            <origin xyz="0 0 0.03" rpy="0 0 0" />
+            <geometry>
+               <cylinder radius="0.08" length="0.05"/>
             </geometry>
          </collision>
@@ -31,5 +31,5 @@
          <axis xyz="0 0 1" />
          <limit velocity="4.8" effort="1000" lower="${-pi*2.0}" upper="${pi*2.0}" />
-         <dynamics damping="0.1" />
+         <dynamics damping="0.05" />
       </joint>
       <link name="${prefix}link1">
@@ -44,7 +44,7 @@
          </visual>
          <collision>
-            <origin xyz="0 0 0" rpy="0 0 0" />
-            <geometry>
-               <mesh filename="${meshes_file_direction}/link1.stl" scale="0.001 0.001 0.001" />
+            <origin xyz="0 0 -0.035" rpy="0 0 0" />
+            <geometry>
+               <cylinder radius="0.055" length="0.1"/>
             </geometry>
          </collision>
@@ -74,7 +74,7 @@
          </visual>
          <collision>
-            <origin xyz="0 0 0" rpy="0 0 0" />
-            <geometry>
-               <mesh filename="${meshes_file_direction}/link2.stl" scale="0.001 0.001 0.001" />
+            <origin xyz="0 -0.02 0.13" rpy="0 0 0" />
+            <geometry>
+               <cylinder radius="0.046" length="0.28"/>
             </geometry>
          </collision>
@@ -104,7 +104,7 @@
          </visual>
          <collision>
-            <origin xyz="0 0 0" rpy="0 0 0" />
-            <geometry>
-               <mesh filename="${meshes_file_direction}/link3.stl" scale="0.001 0.001 0.001" />
+            <origin xyz="0 0.125 0.12" rpy="0 0 0" />
+            <geometry>
+               <cylinder radius="0.042" length="0.23"/>
             </geometry>
          </collision>
@@ -134,7 +134,7 @@
          </visual>
          <collision>
-            <origin xyz="0 0 0" rpy="0 0 0" />
-            <geometry>
-               <mesh filename="${meshes_file_direction}/link4.stl" scale="0.001 0.001 0.001" />
+            <origin xyz="0 0 0" rpy="1.57 0 0" />
+            <geometry>
+               <cylinder radius="0.045" length="0.10"/>
             </geometry>
          </collision>
@@ -164,7 +164,7 @@
          </visual>
          <collision>
-            <origin xyz="0 0 0" rpy="0 0 0" />
-            <geometry>
-               <mesh filename="${meshes_file_direction}/link5.stl" scale="0.001 0.001 0.001" />
+            <origin xyz="0 0 0.01" rpy="0 0 0" />
+            <geometry>
+               <cylinder radius="0.043" length="0.05"/>
             </geometry>
          </collision>
@@ -194,7 +194,7 @@
          </visual>
          <collision>
-            <origin xyz="0 0 0" rpy="0 0 0" />
-            <geometry>
-               <mesh filename="${meshes_file_direction}/link6.stl" scale="0.001 0.001 0.001" />
+            <origin xyz="0 -0.1 0" rpy="1.57 0 0" />
+            <geometry>
+               <cylinder radius="0.07" length="0.25"/>
             </geometry>
          </collision>
@@ -221,7 +221,7 @@
          </visual>
          <collision>
-            <origin xyz="0 0 0" rpy="0 0 0" />
-            <geometry>
-               <mesh filename="${meshes_file_direction}/flange.stl" scale="0.001 0.001 0.001" />
+            <origin xyz="0 0.03 0.04" rpy="0 0 0" />
+            <geometry>
+               <cylinder radius="0.04" length="0.12"/>
             </geometry>
          </collision>

Commit message: Fixed collision config
Signed-off-by: Sungho Woo <wsh@robotis.com>

File: open_manipulator_description/urdf/om_y/open_manipulator_y_arm.urdf.xacro (robot description, xacro)
@@ -44,5 +44,5 @@
          </visual>
          <collision>
-            <origin xyz="0 0 -0.035" rpy="0 0 0" />
+            <origin xyz="0 -0.01 -0.035" rpy="0 0 0" />
             <geometry>
                <cylinder radius="0.055" length="0.1"/>
@@ -74,5 +74,5 @@
          </visual>
          <collision>
-            <origin xyz="0 -0.02 0.13" rpy="0 0 0" />
+            <origin xyz="-0.005 -0.02 0.13" rpy="0 0 0" />
             <geometry>
                <cylinder radius="0.046" length="0.28"/>
@@ -104,7 +104,7 @@
          </visual>
          <collision>
-            <origin xyz="0 0.125 0.12" rpy="0 0 0" />
-            <geometry>
-               <cylinder radius="0.042" length="0.23"/>
+            <origin xyz="0 0.125 0.08" rpy="0 0 0" />
+            <geometry>
+               <cylinder radius="0.042" length="0.19"/>
             </geometry>
          </collision>
@@ -164,5 +164,5 @@
          </visual>
          <collision>
-            <origin xyz="0 0 0.01" rpy="0 0 0" />
+            <origin xyz="0 0.01 0.005" rpy="0 0 0" />
             <geometry>
                <cylinder radius="0.043" length="0.05"/>
@@ -196,5 +196,5 @@
             <origin xyz="0 -0.1 0" rpy="1.57 0 0" />
             <geometry>
-               <cylinder radius="0.07" length="0.25"/>
+               <cylinder radius="0.09" length="0.22"/>
             </geometry>
          </collision>

Commit message: Fixed collision
Signed-off-by: Sungho Woo <wsh@robotis.com>

File: open_manipulator_description/urdf/om_y/open_manipulator_y_arm.urdf.xacro (robot description, xacro)
@@ -223,5 +223,5 @@
             <origin xyz="0 0.03 0.04" rpy="0 0 0" />
             <geometry>
-               <cylinder radius="0.04" length="0.12"/>
+               <cylinder radius="0.03" length="0.12"/>
             </geometry>
          </collision>

File: open_manipulator_description/urdf/om_y_follower/open_manipulator_y_follower_arm.urdf.xacro (robot description, xacro)
@@ -223,5 +223,5 @@
             <origin xyz="0 0.03 0.04" rpy="0 0 0" />
             <geometry>
-               <cylinder radius="0.04" length="0.12"/>
+               <cylinder radius="0.035" length="0.12"/>
             </geometry>
          </collision>
