Commit message: added leader x
Signed-off-by: Sungho Woo <wsh@robotis.com>

File: open_manipulator_description/ros2_control/open_manipulator_x_leader_system.ros2_control.xacro (robot description, xacro)
@@ -1,5 +1,5 @@
 <?xml version="1.0"?>
 <robot xmlns:xacro="http://www.ros.org/wiki/xacro">
-  <xacro:macro name="open_manipulator_x_system" params="name prefix port_name:=/dev/ttyUSB0 use_sim:=^|false use_fake_hardware:=^|false fake_sensor_commands:=^|false">
+  <xacro:macro name="open_manipulator_x_system" params="name prefix port_name:=/dev/ttyUSB1 use_sim:=^|false use_fake_hardware:=^|false fake_sensor_commands:=^|false">
     <ros2_control name="omx" type="system">
       <xacro:if value="$(arg use_sim)">
@@ -17,5 +17,5 @@
           <xacro:unless value="${use_fake_hardware}">
             <plugin>dynamixel_hardware_interface/DynamixelHardware</plugin>
-            <param name="port_name">${port_name}</param>
+            <param name="port_name">/dev/ttyACM0</param>
             <param name="baud_rate">1000000</param>
             <param name="error_timeout_sec">0.2</param>
@@ -43,13 +43,4 @@
             <param name="reboot_dxl_srv_name">dynamixel_hardware_interface/reboot_dxl</param>
             <param name="set_dxl_torque_srv_name">dynamixel_hardware_interface/set_dxl_torque</param>
-              <!-- This parameter is used for a prismatic joint
-            that operates through a revolute mechanism. If the joint does not require this configuration, this parameter can be removed. -->
-            <param name="use_revolute_to_prismatic_gripper">1</param>
-            <param name="revolute_to_prismatic_dxl">dxl5</param>
-            <param name="revolute_max">-1.52</param>
-            <param name="revolute_min">0.92</param>
-            <param name="revolute_to_prismatic_joint">${prefix}gripper_left_joint</param>
-            <param name="prismatic_max">0.019</param>
-            <param name="prismatic_min">-0.01</param>
           </xacro:unless>
         </hardware>
@@ -57,4 +48,5 @@
       <joint name="${prefix}joint1">
         <command_interface name="position"/>
+        <command_interface name="effort"/>
         <state_interface name="position"/>
         <state_interface name="velocity"/>
@@ -63,4 +55,5 @@
       <joint name="${prefix}joint2">
         <command_interface name="position"/>
+        <command_interface name="effort"/>
         <state_interface name="position"/>
         <state_interface name="velocity"/>
@@ -69,4 +62,5 @@
       <joint name="${prefix}joint3">
         <command_interface name="position"/>
+        <command_interface name="effort"/>
         <state_interface name="position"/>
         <state_interface name="velocity"/>
@@ -75,4 +69,5 @@
       <joint name="${prefix}joint4">
         <command_interface name="position"/>
+        <command_interface name="effort"/>
         <state_interface name="position"/>
         <state_interface name="velocity"/>
@@ -81,4 +76,5 @@
       <joint name="${prefix}gripper_left_joint">
         <command_interface name="position"/>
+        <command_interface name="effort"/>
         <state_interface name="position"/>
         <state_interface name="velocity"/>
@@ -96,6 +92,20 @@
       <gpio name="dxl1">
         <param name="type">dxl</param>
-        <param name="ID">11</param>
+        <param name="ID">1</param>
+          <command_interface name="Goal Position"/>
+          <command_interface name="Goal Current"/>
+          <state_interface name="Present Position"/>
+          <state_interface name="Present Velocity"/>
+          <state_interface name="Present Current"/>
+          <state_interface name="Torque Enable"/>
+          <state_interface name="Present Input Voltage"/>
+          <param name="Drive Mode">0</param>
+          <param name="Operating Mode">0</param>
+      </gpio>
+      <gpio name="dxl2">
+        <param name="type">dxl</param>
+        <param name="ID">2</param>
         <command_interface name="Goal Position"/>
+        <command_interface name="Goal Current"/>
         <state_interface name="Present Position"/>
         <state_interface name="Present Velocity"/>
@@ -103,16 +113,12 @@
         <state_interface name="Torque Enable"/>
         <state_interface name="Present Input Voltage"/>
-        <param name="Position P Gain">800</param>
-        <param name="Position I Gain">100</param>
-        <param name="Position D Gain">100</param>
-        <param name="Profile Velocity">200</param>
-        <param name="Profile Acceleration">50</param>
         <param name="Drive Mode">0</param>
-        <param name="Operating Mode">3</param>
+        <param name="Operating Mode">0</param>
       </gpio>
-      <gpio name="dxl2">
+      <gpio name="dxl3">
         <param name="type">dxl</param>
-        <param name="ID">12</param>
+        <param name="ID">3</param>
         <command_interface name="Goal Position"/>
+        <command_interface name="Goal Current"/>
         <state_interface name="Present Position"/>
         <state_interface name="Present Velocity"/>
@@ -120,16 +126,12 @@
         <state_interface name="Torque Enable"/>
         <state_interface name="Present Input Voltage"/>
-        <param name="Position P Gain">800</param>
-        <param name="Position I Gain">100</param>
-        <param name="Position D Gain">100</param>
-        <param name="Profile Velocity">200</param>
-        <param name="Profile Acceleration">50</param>
         <param name="Drive Mode">0</param>
-        <param name="Operating Mode">3</param>
+        <param name="Operating Mode">0</param>
       </gpio>
-      <gpio name="dxl3">
+      <gpio name="dxl4">
         <param name="type">dxl</param>
-        <param name="ID">13</param>
+        <param name="ID">4</param>
         <command_interface name="Goal Position"/>
+        <command_interface name="Goal Current"/>
         <state_interface name="Present Position"/>
         <state_interface name="Present Velocity"/>
@@ -137,16 +139,12 @@
         <state_interface name="Torque Enable"/>
         <state_interface name="Present Input Voltage"/>
-        <param name="Position P Gain">800</param>
-        <param name="Position I Gain">100</param>
-        <param name="Position D Gain">100</param>
-        <param name="Profile Velocity">200</param>
-        <param name="Profile Acceleration">50</param>
         <param name="Drive Mode">0</param>
-        <param name="Operating Mode">3</param>
+        <param name="Operating Mode">0</param>
       </gpio>
-      <gpio name="dxl4">
+      <gpio name="dxl5">
         <param name="type">dxl</param>
-        <param name="ID">14</param>
+        <param name="ID">5</param>
         <command_interface name="Goal Position"/>
+        <command_interface name="Goal Current"/>
         <state_interface name="Present Position"/>
         <state_interface name="Present Velocity"/>
@@ -154,22 +152,6 @@
         <state_interface name="Torque Enable"/>
         <state_interface name="Present Input Voltage"/>
-        <param name="Position P Gain">800</param>
-        <param name="Position I Gain">100</param>
-        <param name="Position D Gain">100</param>
-        <param name="Profile Velocity">200</param>
-        <param name="Profile Acceleration">50</param>
-        <param name="Drive Mode">0</param>
-        <param name="Operating Mode">3</param>
-      </gpio>
-      <gpio name="dxl5">
-        <param name="type">dxl</param>
-        <param name="ID">15</param>
-        <command_interface name="Goal Position"/>
-        <state_interface name="Present Position"/>
-        <state_interface name="Present Velocity"/>
-        <state_interface name="Present Current"/>
-        <state_interface name="Torque Enable"/>
-        <state_interface name="Present Input Voltage"/>
-        <param name="Operating Mode">3</param>
+        <param name="Drive Mode">1</param>
+        <param name="Operating Mode">0</param>
       </gpio>
     </ros2_control>
