Commit message: fix: Unified structure for the omy leader ros2 control config

File: open_manipulator_description/ros2_control/open_manipulator_y_leader_system.ros2_control.xacro (robot description, xacro)
@@ -1,8 +1,19 @@
 <?xml version="1.0"?>
 <robot xmlns:xacro="http://www.ros.org/wiki/xacro">
-    <xacro:macro name="open_manipulator_y_leader_ros2_control" params="name initial_positions_file">
-        <xacro:property name="initial_positions" value="${load_yaml(initial_positions_file)['initial_positions']}"/>
-        <ros2_control name="${name}" type="system">
-          <hardware>
+  <xacro:macro name="open_manipulator_y_leader_system" params="name prefix use_sim:=^|false use_fake_hardware:=^|false fake_sensor_commands:=^|false">
+    <ros2_control name="${name}" type="system">
+      <xacro:if value="$(arg use_sim)">
+        <hardware>
+          <plugin>gz_ros2_control/GazeboSimSystem</plugin>
+        </hardware>
+      </xacro:if>
+      <xacro:unless value="$(arg use_sim)">
+        <hardware>
+          <xacro:if value="${use_fake_hardware}">
+            <plugin>fake_components/GenericSystem</plugin>
+            <param name="fake_sensor_commands">${fake_sensor_commands}</param>
+            <param name="state_following_offset">0.0</param>
+          </xacro:if>
+          <xacro:unless value="${use_fake_hardware}">
             <plugin>dynamixel_hardware_interface/DynamixelHardware</plugin>
             <param name="port_name">/dev/ttyUSB0</param>
@@ -35,146 +46,162 @@
             <param name="reboot_dxl_srv_name">dynamixel_hardware_interface/reboot_dxl</param>
             <param name="set_dxl_torque_srv_name">dynamixel_hardware_interface/set_dxl_torque</param>
-          </hardware>
-          <joint name="joint1">
-            <command_interface name="position"/>
-            <command_interface name="effort"/>
-            <state_interface name="position"/>
-            <state_interface name="velocity"/>
-            <state_interface name="effort"/>
-          </joint>
-          <joint name="joint2">
-            <command_interface name="position"/>
-            <command_interface name="effort"/>
-            <state_interface name="position"/>
-            <state_interface name="velocity"/>
-            <state_interface name="effort"/>
-          </joint>
-          <joint name="joint3">
-            <command_interface name="position"/>
-            <command_interface name="effort"/>
-            <state_interface name="position"/>
-            <state_interface name="velocity"/>
-            <state_interface name="effort"/>
-          </joint>
-          <joint name="joint4">
-            <command_interface name="position"/>
-            <command_interface name="effort"/>
-            <state_interface name="position"/>
-            <state_interface name="velocity"/>
-            <state_interface name="effort"/>
-          </joint>
-          <joint name="joint5">
-            <command_interface name="position"/>
-            <command_interface name="effort"/>
-            <state_interface name="position"/>
-            <state_interface name="velocity"/>
-            <state_interface name="effort"/>
-          </joint>
-          <joint name="joint6">
-            <command_interface name="position"/>
-            <command_interface name="effort"/>
-            <state_interface name="position"/>
-            <state_interface name="velocity"/>
-            <state_interface name="effort"/>
-          </joint>
-          <joint name="rh_r1_joint">
-            <command_interface name="position"/>
-            <command_interface name="effort"/>
-            <state_interface name="position"/>
-            <state_interface name="velocity"/>
-            <state_interface name="effort"/>
-          </joint>
-          <gpio name="dxl1">
-            <param name="type">dxl</param>
-            <param name="ID">1</param>
-            <command_interface name="Goal Position"/>
-            <command_interface name="Goal Current"/>
-            <state_interface name="Present Position"/>
-            <state_interface name="Present Velocity"/>
-            <state_interface name="Present Current"/>
-            <state_interface name="Torque Enable"/>
-            <state_interface name="Present Input Voltage"/>
-            <param name="Drive Mode">0</param>
-            <param name="Operating Mode">0</param>
-          </gpio>
-          <gpio name="dxl2">
-            <param name="type">dxl</param>
-            <param name="ID">2</param>
-            <command_interface name="Goal Position"/>
-            <command_interface name="Goal Current"/>
-            <state_interface name="Present Position"/>
-            <state_interface name="Present Velocity"/>
-            <state_interface name="Present Current"/>
-            <state_interface name="Torque Enable"/>
-            <state_interface name="Present Input Voltage"/>
-            <param name="Drive Mode">0</param>
-            <param name="Operating Mode">0</param>
-          </gpio>
-          <gpio name="dxl3">
-            <param name="type">dxl</param>
-            <param name="ID">3</param>
-            <command_interface name="Goal Position"/>
-            <command_interface name="Goal Current"/>
-            <state_interface name="Present Position"/>
-            <state_interface name="Present Velocity"/>
-            <state_interface name="Present Current"/>
-            <state_interface name="Torque Enable"/>
-            <state_interface name="Present Input Voltage"/>
-            <param name="Drive Mode">1</param>
-            <param name="Operating Mode">0</param>
-          </gpio>
-          <gpio name="dxl4">
-            <param name="type">dxl</param>
-            <param name="ID">4</param>
-            <command_interface name="Goal Position"/>
-            <command_interface name="Goal Current"/>
-            <state_interface name="Present Position"/>
-            <state_interface name="Present Velocity"/>
-            <state_interface name="Present Current"/>
-            <state_interface name="Torque Enable"/>
-            <state_interface name="Present Input Voltage"/>
-            <param name="Drive Mode">0</param>
-            <param name="Operating Mode">0</param>
-          </gpio>
-          <gpio name="dxl5">
-            <param name="type">dxl</param>
-            <param name="ID">5</param>
-            <command_interface name="Goal Position"/>
-            <command_interface name="Goal Current"/>
-            <state_interface name="Present Position"/>
-            <state_interface name="Present Velocity"/>
-            <state_interface name="Present Current"/>
-            <state_interface name="Torque Enable"/>
-            <state_interface name="Present Input Voltage"/>
-            <param name="Drive Mode">0</param>
-            <param name="Operating Mode">0</param>
-          </gpio>
-          <gpio name="dxl6">
-            <param name="type">dxl</param>
-            <param name="ID">6</param>
-            <command_interface name="Goal Position"/>
-            <command_interface name="Goal Current"/>
-            <state_interface name="Present Position"/>
-            <state_interface name="Present Velocity"/>
-            <state_interface name="Present Current"/>
-            <state_interface name="Torque Enable"/>
-            <state_interface name="Present Input Voltage"/>
-            <param name="Drive Mode">0</param>
-            <param name="Operating Mode">0</param>
-          </gpio>
-          <gpio name="dxl7">
-            <param name="type">dxl</param>
-            <param name="ID">7</param>
-            <command_interface name="Goal Position"/>
-            <command_interface name="Goal Current"/>
-            <state_interface name="Present Position"/>
-            <state_interface name="Present Velocity"/>
-            <state_interface name="Present Current"/>
-            <state_interface name="Torque Enable"/>
-            <state_interface name="Present Input Voltage"/>
-            <param name="Drive Mode">0</param>
-            <param name="Operating Mode">0</param>
-          </gpio>
-        </ros2_control>
-    </xacro:macro>
+          </xacro:unless>
+        </hardware>
+      </xacro:unless>
+      <joint name="${prefix}joint1">
+        <command_interface name="position"/>
+        <command_interface name="effort"/>
+        <state_interface name="position"/>
+        <state_interface name="velocity"/>
+        <state_interface name="effort"/>
+      </joint>
+      <joint name="${prefix}joint2">
+        <command_interface name="position"/>
+        <command_interface name="effort"/>
+        <state_interface name="position"/>
+        <state_interface name="velocity"/>
+        <state_interface name="effort"/>
+      </joint>
+      <joint name="${prefix}joint3">
+        <command_interface name="position"/>
+        <command_interface name="effort"/>
+        <state_interface name="position"/>
+        <state_interface name="velocity"/>
+        <state_interface name="effort"/>
+      </joint>
+      <joint name="${prefix}joint4">
+        <command_interface name="position"/>
+        <command_interface name="effort"/>
+        <state_interface name="position"/>
+        <state_interface name="velocity"/>
+        <state_interface name="effort"/>
+      </joint>
+      <joint name="${prefix}joint5">
+        <command_interface name="position"/>
+        <command_interface name="effort"/>
+        <state_interface name="position"/>
+        <state_interface name="velocity"/>
+        <state_interface name="effort"/>
+      </joint>
+      <joint name="${prefix}joint6">
+        <command_interface name="position"/>
+        <command_interface name="effort"/>
+        <state_interface name="position"/>
+        <state_interface name="velocity"/>
+        <state_interface name="effort"/>
+      </joint>
+      <joint name="${prefix}rh_r1_joint">
+        <command_interface name="position"/>
+        <command_interface name="effort"/>
+        <state_interface name="position"/>
+        <state_interface name="velocity"/>
+        <state_interface name="effort"/>
+      </joint>
+      <gpio name="dxl1">
+        <param name="type">dxl</param>
+        <param name="ID">1</param>
+        <command_interface name="Goal Position"/>
+        <command_interface name="Goal Current"/>
+        <state_interface name="Present Position"/>
+        <state_interface name="Present Velocity"/>
+        <state_interface name="Present Current"/>
+        <state_interface name="Torque Enable"/>
+        <state_interface name="Present Input Voltage"/>
+        <param name="Drive Mode">0</param>
+        <param name="Operating Mode">0</param>
+        <param name="Return Delay Time">0</param>
+        <param name="Baud Rate">6</param>
+      </gpio>
+      <gpio name="dxl2">
+        <param name="type">dxl</param>
+        <param name="ID">2</param>
+        <command_interface name="Goal Position"/>
+        <command_interface name="Goal Current"/>
+        <state_interface name="Present Position"/>
+        <state_interface name="Present Velocity"/>
+        <state_interface name="Present Current"/>
+        <state_interface name="Torque Enable"/>
+        <state_interface name="Present Input Voltage"/>
+        <param name="Drive Mode">1</param>
+        <param name="Operating Mode">0</param>
+        <param name="Return Delay Time">0</param>
+        <param name="Baud Rate">6</param>
+      </gpio>
+      <gpio name="dxl3">
+        <param name="type">dxl</param>
+        <param name="ID">3</param>
+        <command_interface name="Goal Position"/>
+        <command_interface name="Goal Current"/>
+        <state_interface name="Present Position"/>
+        <state_interface name="Present Velocity"/>
+        <state_interface name="Present Current"/>
+        <state_interface name="Torque Enable"/>
+        <state_interface name="Present Input Voltage"/>
+        <param name="Drive Mode">0</param>
+        <param name="Operating Mode">0</param>
+        <param name="Return Delay Time">0</param>
+        <param name="Baud Rate">6</param>
+      </gpio>
+      <gpio name="dxl4">
+        <param name="type">dxl</param>
+        <param name="ID">4</param>
+        <command_interface name="Goal Position"/>
+        <command_interface name="Goal Current"/>
+        <state_interface name="Present Position"/>
+        <state_interface name="Present Velocity"/>
+        <state_interface name="Present Current"/>
+        <state_interface name="Torque Enable"/>
+        <state_interface name="Present Input Voltage"/>
+        <param name="Drive Mode">1</param>
+        <param name="Operating Mode">0</param>
+        <param name="Return Delay Time">0</param>
+        <param name="Baud Rate">6</param>
+      </gpio>
+      <gpio name="dxl5">
+        <param name="type">dxl</param>
+        <param name="ID">5</param>
+        <command_interface name="Goal Position"/>
+        <command_interface name="Goal Current"/>
+        <state_interface name="Present Position"/>
+        <state_interface name="Present Velocity"/>
+        <state_interface name="Present Current"/>
+        <state_interface name="Torque Enable"/>
+        <state_interface name="Present Input Voltage"/>
+        <param name="Drive Mode">0</param>
+        <param name="Operating Mode">0</param>
+        <param name="Return Delay Time">0</param>
+        <param name="Baud Rate">6</param>
+      </gpio>
+      <gpio name="dxl6">
+        <param name="type">dxl</param>
+        <param name="ID">6</param>
+        <command_interface name="Goal Position"/>
+        <command_interface name="Goal Current"/>
+        <state_interface name="Present Position"/>
+        <state_interface name="Present Velocity"/>
+        <state_interface name="Present Current"/>
+        <state_interface name="Torque Enable"/>
+        <state_interface name="Present Input Voltage"/>
+        <param name="Drive Mode">1</param>
+        <param name="Operating Mode">0</param>
+        <param name="Return Delay Time">0</param>
+        <param name="Baud Rate">6</param>
+      </gpio>
+      <gpio name="dxl7">
+        <param name="type">dxl</param>
+        <param name="ID">7</param>
+        <command_interface name="Goal Position"/>
+        <command_interface name="Goal Current"/>
+        <state_interface name="Present Position"/>
+        <state_interface name="Present Velocity"/>
+        <state_interface name="Present Current"/>
+        <state_interface name="Torque Enable"/>
+        <state_interface name="Present Input Voltage"/>
+        <param name="Drive Mode">0</param>
+        <param name="Operating Mode">0</param>
+        <param name="Return Delay Time">0</param>
+        <param name="Baud Rate">6</param>
+      </gpio>
+    </ros2_control>
+  </xacro:macro>
 </robot>
