Commit message: - modified open manipulator xacro file (fake_components -> mock_components) - modified open_manipulator urdf (meshes_file_direction)

File: open_manipulator_description/ros2_control/open_manipulator_x_system.ros2_control.xacro (robot description, xacro)
@@ -11,5 +11,5 @@
         <hardware>
           <xacro:if value="${use_fake_hardware}">
-            <plugin>fake_components/GenericSystem</plugin>
+            <plugin>mock_components/GenericSystem</plugin>
             <param name="fake_sensor_commands">${fake_sensor_commands}</param>
             <param name="state_following_offset">0.0</param>

File: open_manipulator_description/ros2_control/open_manipulator_y_end_unit.ros2_control.xacro (robot description, xacro)
@@ -11,5 +11,5 @@
         <hardware>
           <xacro:if value="${use_fake_hardware}">
-            <plugin>fake_components/GenericSystem</plugin>
+            <plugin>mock_components/GenericSystem</plugin>
             <param name="fake_sensor_commands">${fake_sensor_commands}</param>
             <param name="state_following_offset">0.0</param>

File: open_manipulator_description/ros2_control/open_manipulator_y_follower_system.ros2_control.xacro (robot description, xacro)
@@ -11,5 +11,5 @@
         <hardware>
           <xacro:if value="${use_fake_hardware}">
-            <plugin>fake_components/GenericSystem</plugin>
+            <plugin>mock_components/GenericSystem</plugin>
             <param name="fake_sensor_commands">${fake_sensor_commands}</param>
             <param name="state_following_offset">0.0</param>

File: open_manipulator_description/ros2_control/open_manipulator_y_leader_system.ros2_control.xacro (robot description, xacro)
@@ -11,5 +11,5 @@
         <hardware>
           <xacro:if value="${use_fake_hardware}">
-            <plugin>fake_components/GenericSystem</plugin>
+            <plugin>mock_components/GenericSystem</plugin>
             <param name="fake_sensor_commands">${fake_sensor_commands}</param>
             <param name="state_following_offset">0.0</param>

File: open_manipulator_description/ros2_control/open_manipulator_y_system.ros2_control.xacro (robot description, xacro)
@@ -11,5 +11,5 @@
         <hardware>
           <xacro:if value="${use_fake_hardware}">
-            <plugin>fake_components/GenericSystem</plugin>
+            <plugin>mock_components/GenericSystem</plugin>
             <param name="fake_sensor_commands">${fake_sensor_commands}</param>
             <param name="state_following_offset">0.0</param>

File: open_manipulator_description/urdf/om_y/open_manipulator_y_arm.urdf.xacro (robot description, xacro)
@@ -2,5 +2,5 @@
 <robot xmlns:xacro="http://www.ros.org/wiki/xacro">
    <xacro:macro name="open_manipulator_y" params="prefix">
-      <xacro:property name="meshes_file_direction" value="package://open_manipulator_description/meshes/om_y/" />
+      <xacro:property name="meshes_file_direction" value="package://open_manipulator_description/meshes/om_y" />
       <link name="${prefix}link0">
          <visual>

File: open_manipulator_description/urdf/om_y_follower/open_manipulator_y_follower_arm.urdf.xacro (robot description, xacro)
@@ -2,5 +2,5 @@
 <robot xmlns:xacro="http://www.ros.org/wiki/xacro">
    <xacro:macro name="open_manipulator_y" params="prefix">
-      <xacro:property name="meshes_file_direction" value="package://open_manipulator_description/meshes/om_y/" />
+      <xacro:property name="meshes_file_direction" value="package://open_manipulator_description/meshes/om_y_follower" />
       <link name="${prefix}link0">
          <visual>
