Commit message: fix: Updated ros2 control for the omy follower
 - New End unit hardware is now fixed

File: open_manipulator_description/ros2_control/open_manipulator_y_follower_system.ros2_control.xacro (robot description, xacro)
@@ -17,27 +17,25 @@
           <xacro:unless value="${use_fake_hardware}">
             <plugin>dynamixel_hardware_interface/DynamixelHardware</plugin>
-            <param name="port_name">/dev/ttyACM0</param>
-            <param name="baud_rate">4000000</param>
+            <param name="port_name">/dev/ttyAMA2</param>
+            <param name="baud_rate">6250000</param>
             <param name="error_timeout_ms">500</param>
             <param name="dynamixel_model_folder">/param/dxl_model</param>
-            <param name="number_of_joints">7</param>
-            <param name="number_of_transmissions">7</param>
+            <param name="number_of_joints">6</param>
+            <param name="number_of_transmissions">6</param>
             <param name="transmission_to_joint_matrix">
-              1, 0, 0, 0, 0, 0, 0,
-              0, 1, 0, 0, 0, 0, 0,
-              0, 0, 1, 0, 0, 0, 0,
-              0, 0, 0, 1, 0, 0, 0,
-              0, 0, 0, 0, 1, 0, 0,
-              0, 0, 0, 0, 0, 1, 0,
-              0, 0, 0, 0, 0, 0, 1
+              1, 0, 0, 0, 0, 0,
+              0, 1, 0, 0, 0, 0,
+              0, 0, 1, 0, 0, 0,
+              0, 0, 0, 1, 0, 0,
+              0, 0, 0, 0, 1, 0,
+              0, 0, 0, 0, 0, 1
             </param>
             <param name="joint_to_transmission_matrix">
-              1, 0, 0, 0, 0, 0, 0,
-              0, 1, 0, 0, 0, 0, 0,
-              0, 0, 1, 0, 0, 0, 0,
-              0, 0, 0, 1, 0, 0, 0,
-              0, 0, 0, 0, 1, 0, 0,
-              0, 0, 0, 0, 0, 1, 0,
-              0, 0, 0, 0, 0, 0, 1
+              1, 0, 0, 0, 0, 0,
+              0, 1, 0, 0, 0, 0,
+              0, 0, 1, 0, 0, 0,
+              0, 0, 0, 1, 0, 0,
+              0, 0, 0, 0, 1, 0,
+              0, 0, 0, 0, 0, 1
             </param>
             <param name="dynamixel_state_pub_msg_name">dynamixel_hardware_interface/dxl_state</param>
@@ -85,10 +83,4 @@
         <state_interface name="effort"/>
       </joint>
-      <joint name="${prefix}rh_r1_joint">
-        <command_interface name="position"/>
-        <state_interface name="position"/>
-        <state_interface name="velocity"/>
-        <state_interface name="effort"/>
-      </joint>
       <gpio name="dxl1">
         <param name="type">dxl</param>
@@ -105,5 +97,5 @@
         <param name="Profile Velocity">3591</param>
         <param name="Profile Acceleration">8050</param>
-        <param name="Homing Offset">-131072</param>
+        <param name="Homing Offset">0</param>
         <param name="Return Delay Time">0</param>
         <param name="Position P Gain">1583185</param>
@@ -121,5 +113,5 @@
         <state_interface name="Torque Enable"/>
         <state_interface name="Present Input Voltage"/>
-        <param name="Drive Mode">0</param>
+        <param name="Drive Mode">1</param>
         <param name="Velocity Limit">3591</param>
         <param name="Acceleration Limit">8050</param>
@@ -141,4 +133,24 @@
         <state_interface name="Torque Enable"/>
         <state_interface name="Present Input Voltage"/>
+        <param name="Drive Mode">0</param>
+        <param name="Velocity Limit">6486</param>
+        <param name="Acceleration Limit">8050</param>
+        <param name="Profile Velocity">6486</param>
+        <param name="Profile Acceleration">8050</param>
+        <param name="Return Delay Time">0</param>
+        <param name="Position P Gain">1583185</param>
+        <param name="Velocity P Gain">18184</param>
+        <param name="Velocity I Gain">1585331</param>
+        <param name="Operating Mode">3</param>
+      </gpio>
+      <gpio name="dxl4">
+        <param name="type">dxl</param>
+        <param name="ID">4</param>
+        <command_interface name="Goal Position"/>
+        <state_interface name="Present Position"/>
+        <state_interface name="Present Velocity"/>
+        <state_interface name="Present Current"/>
+        <state_interface name="Torque Enable"/>
+        <state_interface name="Present Input Voltage"/>
         <param name="Drive Mode">1</param>
         <param name="Velocity Limit">6486</param>
@@ -152,7 +164,7 @@
         <param name="Operating Mode">3</param>
       </gpio>
-      <gpio name="dxl4">
-        <param name="type">dxl</param>
-        <param name="ID">4</param>
+      <gpio name="dxl5">
+        <param name="type">dxl</param>
+        <param name="ID">5</param>
         <command_interface name="Goal Position"/>
         <state_interface name="Present Position"/>
@@ -172,24 +184,4 @@
         <param name="Operating Mode">3</param>
       </gpio>
-      <gpio name="dxl5">
-        <param name="type">dxl</param>
-        <param name="ID">5</param>
-        <command_interface name="Goal Position"/>
-        <state_interface name="Present Position"/>
-        <state_interface name="Present Velocity"/>
-        <state_interface name="Present Current"/>
-        <state_interface name="Torque Enable"/>
-        <state_interface name="Present Input Voltage"/>
-        <param name="Drive Mode">0</param>
-        <param name="Velocity Limit">6486</param>
-        <param name="Acceleration Limit">8050</param>
-        <param name="Profile Velocity">6486</param>
-        <param name="Profile Acceleration">8050</param>
-        <param name="Return Delay Time">0</param>
-        <param name="Position P Gain">1583185</param>
-        <param name="Velocity P Gain">18184</param>
-        <param name="Velocity I Gain">1585331</param>
-        <param name="Operating Mode">3</param>
-      </gpio>
       <gpio name="dxl6">
         <param name="type">dxl</param>
@@ -201,26 +193,26 @@
         <state_interface name="Torque Enable"/>
         <state_interface name="Present Input Voltage"/>
-        <param name="Drive Mode">0</param>
-        <param name="Velocity Limit">6486</param>
-        <param name="Acceleration Limit">8050</param>
-        <param name="Profile Velocity">6486</param>
-        <param name="Profile Acceleration">8050</param>
-        <param name="Return Delay Time">0</param>
-        <param name="Position P Gain">1583185</param>
-        <param name="Velocity P Gain">18184</param>
-        <param name="Velocity I Gain">1585331</param>
-        <param name="Operating Mode">3</param>
-      </gpio>
-      <gpio name="dxl7">
-        <param name="type">dxl</param>
-        <param name="ID">7</param>
-        <command_interface name="Goal Position"/>
-        <state_interface name="Present Position"/>
-        <state_interface name="Present Velocity"/>
-        <state_interface name="Present Current"/>
-        <state_interface name="Torque Enable"/>
-        <state_interface name="Present Input Voltage"/>
-        <param name="Operating Mode">5</param>
-        <param name="Return Delay Time">0</param>
+        <param name="Drive Mode">1</param>
+        <param name="Velocity Limit">6486</param>
+        <param name="Acceleration Limit">8050</param>
+        <param name="Profile Velocity">6486</param>
+        <param name="Profile Acceleration">8050</param>
+        <param name="Return Delay Time">0</param>
+        <param name="Position P Gain">1583185</param>
+        <param name="Velocity P Gain">18184</param>
+        <param name="Velocity I Gain">1585331</param>
+        <param name="Operating Mode">3</param>
+      </gpio>
+      <gpio name="omy_hat">
+        <param name="type">controller</param>
+        <param name="ID">200</param>
+        <param name="Power Enable">1</param>
+        <param name="Voltage Control Enable">1</param>
+        <param name="R LED">200</param>
+        <param name="G LED">200</param>
+        <param name="B LED">120</param>
+        <param name="Baud Rate (Bus)">8</param>
+        <param name="DXL Baud Rate">8</param>
+        <param name="Status">0</param>
       </gpio>
     </ros2_control>
