Commit message: feat: Modify for generic DXL arms

File: open_manipulator_description/ros2_control/open_manipulator_y_follower_system.ros2_control.xacro (robot description, xacro)
@@ -1,5 +1,5 @@
 <?xml version="1.0"?>
 <robot xmlns:xacro="http://www.ros.org/wiki/xacro">
-  <xacro:macro name="open_manipulator_y_system" params="name prefix port_name:=^|/dev/ttyAMA2 use_sim:=^|false use_fake_hardware:=^|false fake_sensor_commands:=^|false">
+  <xacro:macro name="open_manipulator_y_system" params="name prefix port_name:=^|/dev/ttyACM0 use_sim:=^|false use_fake_hardware:=^|false fake_sensor_commands:=^|false">
     <ros2_control name="${name}" type="system">
       <xacro:if value="$(arg use_sim)">
@@ -18,5 +18,5 @@
             <plugin>dynamixel_hardware_interface/DynamixelHardware</plugin>
             <param name="port_name">${port_name}</param>
-            <param name="baud_rate">6250000</param>
+            <param name="baud_rate">1000000</param>
             <param name="error_timeout_ms">500</param>
             <param name="dynamixel_model_folder">/param/dxl_model</param>
@@ -85,134 +85,98 @@
       <gpio name="dxl1">
         <param name="type">dxl</param>
-        <param name="ID">1</param>
+        <param name="ID">11</param>
         <command_interface name="Goal Position"/>
         <state_interface name="Present Position"/>
         <state_interface name="Present Velocity"/>
         <state_interface name="Present Current"/>
-        <state_interface name="Torque Enable"/>
-        <state_interface name="Present Input Voltage"/>
         <param name="Drive Mode">0</param>
-        <param name="Velocity Limit">3591</param>
-        <param name="Acceleration Limit">8050</param>
-        <param name="Profile Velocity">3591</param>
-        <param name="Profile Acceleration">8050</param>
-        <param name="Homing Offset">0</param>
+        <param name="Operating Mode">3</param>
         <param name="Return Delay Time">0</param>
-        <param name="Position P Gain">1583185</param>
-        <param name="Velocity P Gain">41387</param>
-        <param name="Velocity I Gain">1565630</param>
-        <param name="Operating Mode">3</param>
+        <param name="Position P Gain">1500</param>
+        <param name="Position I Gain">400</param>
+        <param name="Position D Gain">400</param>
+        <param name="Profile Velocity">0</param>
+        <param name="Profile Acceleration">0</param>
       </gpio>
       <gpio name="dxl2">
         <param name="type">dxl</param>
-        <param name="ID">2</param>
+        <param name="ID">12</param>
         <command_interface name="Goal Position"/>
         <state_interface name="Present Position"/>
         <state_interface name="Present Velocity"/>
         <state_interface name="Present Current"/>
-        <state_interface name="Torque Enable"/>
-        <state_interface name="Present Input Voltage"/>
-        <param name="Drive Mode">1</param>
-        <param name="Velocity Limit">3591</param>
-        <param name="Acceleration Limit">8050</param>
-        <param name="Profile Velocity">3591</param>
-        <param name="Profile Acceleration">8050</param>
+        <param name="Drive Mode">0</param>
+        <param name="Operating Mode">3</param>
         <param name="Return Delay Time">0</param>
-        <param name="Position P Gain">1583185</param>
-        <param name="Velocity P Gain">41387</param>
-        <param name="Velocity I Gain">1565630</param>
-        <param name="Operating Mode">3</param>
+        <param name="Position P Gain">1500</param>
+        <param name="Position I Gain">400</param>
+        <param name="Position D Gain">400</param>
+        <param name="Profile Velocity">0</param>
+        <param name="Profile Acceleration">0</param>
       </gpio>
       <gpio name="dxl3">
         <param name="type">dxl</param>
-        <param name="ID">3</param>
+        <param name="ID">13</param>
         <command_interface name="Goal Position"/>
         <state_interface name="Present Position"/>
         <state_interface name="Present Velocity"/>
         <state_interface name="Present Current"/>
-        <state_interface name="Torque Enable"/>
-        <state_interface name="Present Input Voltage"/>
         <param name="Drive Mode">0</param>
-        <param name="Velocity Limit">6486</param>
-        <param name="Acceleration Limit">8050</param>
-        <param name="Profile Velocity">6486</param>
-        <param name="Profile Acceleration">8050</param>
+        <param name="Operating Mode">3</param>
         <param name="Return Delay Time">0</param>
-        <param name="Position P Gain">1583185</param>
-        <param name="Velocity P Gain">18184</param>
-        <param name="Velocity I Gain">1585331</param>
-        <param name="Operating Mode">3</param>
+        <param name="Position P Gain">1500</param>
+        <param name="Position I Gain">400</param>
+        <param name="Position D Gain">400</param>
+        <param name="Profile Velocity">0</param>
+        <param name="Profile Acceleration">0</param>
       </gpio>
       <gpio name="dxl4">
         <param name="type">dxl</param>
-        <param name="ID">4</param>
+        <param name="ID">14</param>
         <command_interface name="Goal Position"/>
         <state_interface name="Present Position"/>
         <state_interface name="Present Velocity"/>
         <state_interface name="Present Current"/>
-        <state_interface name="Torque Enable"/>
-        <state_interface name="Present Input Voltage"/>
-        <param name="Drive Mode">1</param>
-        <param name="Velocity Limit">6486</param>
-        <param name="Acceleration Limit">8050</param>
-        <param name="Profile Velocity">6486</param>
-        <param name="Profile Acceleration">8050</param>
+        <param name="Drive Mode">0</param>
+        <param name="Operating Mode">3</param>
         <param name="Return Delay Time">0</param>
-        <param name="Position P Gain">1583185</param>
-        <param name="Velocity P Gain">18184</param>
-        <param name="Velocity I Gain">1585331</param>
-        <param name="Operating Mode">3</param>
+        <param name="Position P Gain">1500</param>
+        <param name="Position I Gain">400</param>
+        <param name="Position D Gain">400</param>
+        <param name="Profile Velocity">0</param>
+        <param name="Profile Acceleration">0</param>
       </gpio>
       <gpio name="dxl5">
         <param name="type">dxl</param>
-        <param name="ID">5</param>
+        <param name="ID">15</param>
         <command_interface name="Goal Position"/>
         <state_interface name="Present Position"/>
         <state_interface name="Present Velocity"/>
         <state_interface name="Present Current"/>
-        <state_interface name="Torque Enable"/>
-        <state_interface name="Present Input Voltage"/>
         <param name="Drive Mode">0</param>
-        <param name="Velocity Limit">6486</param>
-        <param name="Acceleration Limit">8050</param>
-        <param name="Profile Velocity">6486</param>
-        <param name="Profile Acceleration">8050</param>
+        <param name="Operating Mode">3</param>
         <param name="Return Delay Time">0</param>
-        <param name="Position P Gain">1583185</param>
-        <param name="Velocity P Gain">18184</param>
-        <param name="Velocity I Gain">1585331</param>
-        <param name="Operating Mode">3</param>
+        <param name="Position P Gain">1500</param>
+        <param name="Position I Gain">400</param>
+        <param name="Position D Gain">400</param>
+        <param name="Profile Velocity">0</param>
+        <param name="Profile Acceleration">0</param>
       </gpio>
       <gpio name="dxl6">
         <param name="type">dxl</param>
-        <param name="ID">6</param>
+        <param name="ID">16</param>
         <command_interface name="Goal Position"/>
         <state_interface name="Present Position"/>
         <state_interface name="Present Velocity"/>
         <state_interface name="Present Current"/>
-        <state_interface name="Torque Enable"/>
-        <state_interface name="Present Input Voltage"/>
-        <param name="Drive Mode">1</param>
-        <param name="Velocity Limit">6486</param>
-        <param name="Acceleration Limit">8050</param>
-        <param name="Profile Velocity">6486</param>
-        <param name="Profile Acceleration">8050</param>
+        <param name="Drive Mode">0</param>
+        <param name="Operating Mode">5</param>
         <param name="Return Delay Time">0</param>
-        <param name="Position P Gain">1583185</param>
-        <param name="Velocity P Gain">18184</param>
-        <param name="Velocity I Gain">1585331</param>
-        <param name="Operating Mode">3</param>
-      </gpio>
-      <gpio name="omy_hat">
-        <param name="type">controller</param>
-        <param name="ID">200</param>
-        <param name="Power Enable">1</param>
-        <param name="Voltage Control Enable">1</param>
-        <param name="R LED">200</param>
-        <param name="G LED">200</param>
-        <param name="B LED">120</param>
-        <param name="Baud Rate (Bus)">8</param>
-        <param name="DXL Baud Rate">8</param>
-        <param name="Status">0</param>
+        <param name="Position P Gain">1500</param>
+        <param name="Position I Gain">400</param>
+        <param name="Position D Gain">400</param>
+        <param name="Profile Velocity">0</param>
+        <param name="Profile Acceleration">0</param>
+        <param name="Goal Current">700</param>
       </gpio>
     </ros2_control>

File: open_manipulator_description/ros2_control/open_manipulator_y_leader_system.ros2_control.xacro (robot description, xacro)
@@ -17,27 +17,25 @@
           <xacro:unless value="${use_fake_hardware}">
             <plugin>dynamixel_hardware_interface/DynamixelHardware</plugin>
-            <param name="port_name">/dev/ttyUSB0</param>
-            <param name="baud_rate">4000000</param>
+            <param name="port_name">/dev/ttyACM1</param>
+            <param name="baud_rate">1000000</param>
             <param name="error_timeout_ms">500</param>
             <param name="dynamixel_model_folder">/param/dxl_model</param>
-            <param name="number_of_joints">7</param>
-            <param name="number_of_transmissions">7</param>
+            <param name="number_of_joints">6</param>
+            <param name="number_of_transmissions">6</param>
             <param name="transmission_to_joint_matrix">
-              1, 0, 0, 0, 0, 0, 0,
-              0, 1, 0, 0, 0, 0, 0,
-              0, 0, 1, 0, 0, 0, 0,
-              0, 0, 0, 1, 0, 0, 0,
-              0, 0, 0, 0, 1, 0, 0,
-              0, 0, 0, 0, 0, 1, 0,
-              0, 0, 0, 0, 0, 0, 1
+              1, 0, 0, 0, 0, 0,
+              0, 1, 0, 0, 0, 0,
+              0, 0, 1, 0, 0, 0,
+              0, 0, 0, 1, 0, 0,
+              0, 0, 0, 0, 1, 0,
+              0, 0, 0, 0, 0, 1
             </param>
             <param name="joint_to_transmission_matrix">
-              1, 0, 0, 0, 0, 0, 0,
-              0, 1, 0, 0, 0, 0, 0,
-              0, 0, 1, 0, 0, 0, 0,
-              0, 0, 0, 1, 0, 0, 0,
-              0, 0, 0, 0, 1, 0, 0,
-              0, 0, 0, 0, 0, 1, 0,
-              0, 0, 0, 0, 0, 0, 1
+              1, 0, 0, 0, 0, 0,
+              0, 1, 0, 0, 0, 0,
+              0, 0, 1, 0, 0, 0,
+              0, 0, 0, 1, 0, 0,
+              0, 0, 0, 0, 1, 0,
+              0, 0, 0, 0, 0, 1
             </param>
             <param name="dynamixel_state_pub_msg_name">dynamixel_hardware_interface/dxl_state</param>
@@ -50,5 +48,4 @@
       </xacro:unless>
       <joint name="${prefix}joint1">
-        <command_interface name="position"/>
         <command_interface name="effort"/>
         <state_interface name="position"/>
@@ -57,5 +54,4 @@
       </joint>
       <joint name="${prefix}joint2">
-        <command_interface name="position"/>
         <command_interface name="effort"/>
         <state_interface name="position"/>
@@ -64,5 +60,4 @@
       </joint>
       <joint name="${prefix}joint3">
-        <command_interface name="position"/>
         <command_interface name="effort"/>
         <state_interface name="position"/>
@@ -71,5 +66,4 @@
       </joint>
       <joint name="${prefix}joint4">
-        <command_interface name="position"/>
         <command_interface name="effort"/>
         <state_interface name="position"/>
@@ -78,5 +72,4 @@
       </joint>
       <joint name="${prefix}joint5">
-        <command_interface name="position"/>
         <command_interface name="effort"/>
         <state_interface name="position"/>
@@ -85,12 +78,4 @@
       </joint>
       <joint name="${prefix}joint6">
-        <command_interface name="position"/>
-        <command_interface name="effort"/>
-        <state_interface name="position"/>
-        <state_interface name="velocity"/>
-        <state_interface name="effort"/>
-      </joint>
-      <joint name="${prefix}rh_r1_joint">
-        <command_interface name="position"/>
         <command_interface name="effort"/>
         <state_interface name="position"/>
@@ -100,106 +85,73 @@
       <gpio name="dxl1">
         <param name="type">dxl</param>
-        <param name="ID">1</param>
-        <command_interface name="Goal Position"/>
+        <param name="ID">11</param>
         <command_interface name="Goal Current"/>
         <state_interface name="Present Position"/>
         <state_interface name="Present Velocity"/>
         <state_interface name="Present Current"/>
-        <state_interface name="Torque Enable"/>
-        <state_interface name="Present Input Voltage"/>
+        <param name="Torque Enable">0</param>
         <param name="Drive Mode">0</param>
         <param name="Operating Mode">0</param>
         <param name="Return Delay Time">0</param>
-        <param name="Baud Rate">6</param>
       </gpio>
       <gpio name="dxl2">
         <param name="type">dxl</param>
-        <param name="ID">2</param>
-        <command_interface name="Goal Position"/>
+        <param name="ID">12</param>
         <command_interface name="Goal Current"/>
         <state_interface name="Present Position"/>
         <state_interface name="Present Velocity"/>
         <state_interface name="Present Current"/>
-        <state_interface name="Torque Enable"/>
-        <state_interface name="Present Input Voltage"/>
-        <param name="Drive Mode">1</param>
+        <param name="Torque Enable">0</param>
+        <param name="Drive Mode">0</param>
         <param name="Operating Mode">0</param>
         <param name="Return Delay Time">0</param>
-        <param name="Baud Rate">6</param>
       </gpio>
       <gpio name="dxl3">
         <param name="type">dxl</param>
-        <param name="ID">3</param>
-        <command_interface name="Goal Position"/>
+        <param name="ID">13</param>
         <command_interface name="Goal Current"/>
         <state_interface name="Present Position"/>
         <state_interface name="Present Velocity"/>
         <state_interface name="Present Current"/>
-        <state_interface name="Torque Enable"/>
-        <state_interface name="Present Input Voltage"/>
+        <param name="Torque Enable">0</param>
         <param name="Drive Mode">0</param>
         <param name="Operating Mode">0</param>
         <param name="Return Delay Time">0</param>
-        <param name="Baud Rate">6</param>
       </gpio>
       <gpio name="dxl4">
         <param name="type">dxl</param>
-        <param name="ID">4</param>
-        <command_interface name="Goal Position"/>
+        <param name="ID">14</param>
         <command_interface name="Goal Current"/>
         <state_interface name="Present Position"/>
         <state_interface name="Present Velocity"/>
         <state_interface name="Present Current"/>
-        <state_interface name="Torque Enable"/>
-        <state_interface name="Present Input Voltage"/>
-        <param name="Drive Mode">1</param>
+        <param name="Torque Enable">0</param>
+        <param name="Drive Mode">0</param>
         <param name="Operating Mode">0</param>
         <param name="Return Delay Time">0</param>
-        <param name="Baud Rate">6</param>
       </gpio>
       <gpio name="dxl5">
         <param name="type">dxl</param>
-        <param name="ID">5</param>
-        <command_interface name="Goal Position"/>
+        <param name="ID">15</param>
         <command_interface name="Goal Current"/>
         <state_interface name="Present Position"/>
         <state_interface name="Present Velocity"/>
         <state_interface name="Present Current"/>
-        <state_interface name="Torque Enable"/>
-        <state_interface name="Present Input Voltage"/>
+        <param name="Torque Enable">0</param>
         <param name="Drive Mode">0</param>
         <param name="Operating Mode">0</param>
         <param name="Return Delay Time">0</param>
-        <param name="Baud Rate">6</param>
       </gpio>
       <gpio name="dxl6">
         <param name="type">dxl</param>
-        <param name="ID">6</param>
-        <command_interface name="Goal Position"/>
+        <param name="ID">16</param>
         <command_interface name="Goal Current"/>
         <state_interface name="Present Position"/>
         <state_interface name="Present Velocity"/>
         <state_interface name="Present Current"/>
-        <state_interface name="Torque Enable"/>
-        <state_interface name="Present Input Voltage"/>
-        <param name="Drive Mode">1</param>
-        <param name="Operating Mode">0</param>
-        <param name="Return Delay Time">0</param>
-        <param name="Baud Rate">6</param>
-      </gpio>
-      <gpio name="dxl7">
-        <param name="type">dxl</param>
-        <param name="ID">7</param>
-        <command_interface name="Goal Position"/>
-        <command_interface name="Goal Current"/>
-        <state_interface name="Present Position"/>
-        <state_interface name="Present Velocity"/>
-        <state_interface name="Present Current"/>
-        <state_interface name="Torque Enable"/>
-        <state_interface name="Present Input Voltage"/>
+        <param name="Torque Enable">0</param>
         <param name="Drive Mode">0</param>
         <param name="Operating Mode">0</param>
         <param name="Return Delay Time">0</param>
-        <param name="Baud Rate">6</param>
       </gpio>
     </ros2_control>

File: open_manipulator_description/urdf/om_y_follower/open_manipulator_y_follower.urdf.xacro (robot description, xacro)
@@ -17,5 +17,4 @@
   <!-- Include OpenManipulator-Y ros2 control macro -->
   <xacro:include filename="$(find open_manipulator_description)/ros2_control/open_manipulator_y_follower_system.ros2_control.xacro" />
-  <xacro:include filename="$(find open_manipulator_description)/ros2_control/open_manipulator_y_end_unit.ros2_control.xacro" />
   <!-- World -->
   <link name="world"/>
@@ -40,8 +39,4 @@
     use_fake_hardware="$(arg use_fake_hardware)"
     fake_sensor_commands="$(arg fake_sensor_commands)"/>
-  <xacro:open_manipulator_y_end_unit
-    name="OpenManipulatorYEndUnit" prefix="$(arg prefix)" use_sim="$(arg use_sim)"
-    use_fake_hardware="$(arg use_fake_hardware)"
-    fake_sensor_commands="$(arg fake_sensor_commands)"/>
   <gazebo>
     <plugin filename="gz_ros2_control-system" name="gz_ros2_control::GazeboSimROS2ControlPlugin">
