Commit message: OMY-3m bringup gazebo
Signed-off-by: Wonho Yun <ywh@robotis.com>

File: open_manipulator_description/ros2_control/omy_3m_end_unit.ros2_control.xacro (robot description, xacro)
@@ -3,9 +3,4 @@
   <xacro:macro name="omy_3m_end_unit" params="name prefix port_name:=^|/dev/ttyAMA4 use_sim:=^|false use_fake_hardware:=^|false fake_sensor_commands:=^|false">
     <ros2_control name="${name}" type="system">
-      <xacro:if value="$(arg use_sim)">
-        <hardware>
-          <plugin>gz_ros2_control/GazeboSimSystem</plugin>
-        </hardware>
-      </xacro:if>
       <xacro:unless value="$(arg use_sim)">
         <hardware>
@@ -37,10 +32,10 @@
         </hardware>
       </xacro:unless>
-      <joint name="${prefix}rh_r1_joint">
+      <!-- <joint name="${prefix}rh_r1_joint">
         <command_interface name="position"/>
         <state_interface name="position"/>
         <state_interface name="velocity"/>
         <state_interface name="effort"/>
-      </joint>
+      </joint> -->
       <!-- <gpio name="dxl7">
         <param name="type">dxl</param>

File: open_manipulator_description/urdf/omy_3m/omy_3m.urdf.xacro (robot description, xacro)
@@ -34,5 +34,5 @@
   <gazebo>
     <plugin filename="gz_ros2_control-system" name="gz_ros2_control::GazeboSimROS2ControlPlugin">
-      <parameters>$(find open_manipulator_bringup)/config/omy_3m/gazebo_controller_manager.yaml</parameters>
+      <parameters>$(find open_manipulator_bringup)/config/omy_3m/hardware_controller_manager.yaml</parameters>
     </plugin>
   </gazebo>

Commit message: Removed the unused files
Signed-off-by: Wonho Yun <ywh@robotis.com>

File: open_manipulator_description/ros2_control/omy_3m_end_unit.ros2_control.xacro (robot description, xacro)
@@ -32,10 +32,4 @@
         </hardware>
       </xacro:unless>
-      <!-- <joint name="${prefix}rh_r1_joint">
-        <command_interface name="position"/>
-        <state_interface name="position"/>
-        <state_interface name="velocity"/>
-        <state_interface name="effort"/>
-      </joint> -->
       <!-- <gpio name="dxl7">
         <param name="type">dxl</param>
