Commit message: Refactor ROS2 control xacro files

File: open_manipulator_description/ros2_control/omx.ros2_control.xacro (robot description, xacro)
@@ -42,6 +42,4 @@
             <param name="reboot_dxl_srv_name">dynamixel_hardware_interface/reboot_dxl</param>
             <param name="set_dxl_torque_srv_name">dynamixel_hardware_interface/set_dxl_torque</param>
-            <!-- This parameter is used for a prismatic joint that operates through a revolute mechanism.
-            If the joint does not require this configuration, this parameter can be removed. -->
             <param name="use_revolute_to_prismatic_gripper">1</param>
             <param name="revolute_to_prismatic_dxl">dxl5</param>
@@ -100,6 +98,4 @@
         <state_interface name="Present Velocity"/>
         <state_interface name="Present Current"/>
-        <state_interface name="Torque Enable"/>
-        <state_interface name="Present Input Voltage"/>
         <param name="Position P Gain">800</param>
         <param name="Position I Gain">100</param>
@@ -116,6 +112,4 @@
         <state_interface name="Present Velocity"/>
         <state_interface name="Present Current"/>
-        <state_interface name="Torque Enable"/>
-        <state_interface name="Present Input Voltage"/>
         <param name="Position P Gain">800</param>
         <param name="Position I Gain">100</param>
@@ -132,6 +126,4 @@
         <state_interface name="Present Velocity"/>
         <state_interface name="Present Current"/>
-        <state_interface name="Torque Enable"/>
-        <state_interface name="Present Input Voltage"/>
         <param name="Position P Gain">800</param>
         <param name="Position I Gain">100</param>
@@ -148,6 +140,4 @@
         <state_interface name="Present Velocity"/>
         <state_interface name="Present Current"/>
-        <state_interface name="Torque Enable"/>
-        <state_interface name="Present Input Voltage"/>
         <param name="Position P Gain">800</param>
         <param name="Position I Gain">100</param>
@@ -164,6 +154,4 @@
         <state_interface name="Present Velocity"/>
         <state_interface name="Present Current"/>
-        <state_interface name="Torque Enable"/>
-        <state_interface name="Present Input Voltage"/>
       </gpio>
     </ros2_control>

File: open_manipulator_description/ros2_control/omy_3m_end_unit.ros2_control.xacro (robot description, xacro)
@@ -1,6 +1,11 @@
 <?xml version="1.0"?>
 <robot xmlns:xacro="http://www.ros.org/wiki/xacro">
-  <xacro:macro name="omy_3m_end_unit" params="name prefix port_name:=^|/dev/ttyAMA4 use_sim:=^|false use_fake_hardware:=^|false fake_sensor_commands:=^|false">
+  <xacro:macro name="omy_3m_end_unit_system" params="name prefix port_name:=^|/dev/ttyAMA4 use_sim:=^|false use_fake_hardware:=^|false fake_sensor_commands:=^|false">
     <ros2_control name="${name}" type="system">
+      <xacro:if value="$(arg use_sim)">
+        <hardware>
+          <plugin>gz_ros2_control/GazeboSimSystem</plugin>
+        </hardware>
+      </xacro:if>
       <xacro:unless value="$(arg use_sim)">
         <hardware>
@@ -32,24 +37,5 @@
         </hardware>
       </xacro:unless>
-      <!-- <gpio name="dxl7">
-        <param name="type">dxl</param>
-        <param name="ID">7</param>
-        <command_interface name="Goal Position"/>
-        <state_interface name="Present Position"/>
-        <state_interface name="Present Velocity"/>
-        <state_interface name="Present Current"/>
-        <state_interface name="Torque Enable"/>
-        <state_interface name="Present Input Voltage"/>
-        <param name="Operating Mode">5</param>
-        <param name="Return Delay Time">0</param>
-      </gpio> -->
       <gpio name="omy_end">
-        <command_interface name="Goal Position"/>
-        <!-- <command_interface name="Goal Velocity"/> -->
-        <!-- <command_interface name="Goal Current"/> -->
-        <state_interface name="Present Position"/>
-        <state_interface name="Present Velocity"/>
-        <state_interface name="Present Current"/>
-        <state_interface name="Torque Enable"/>
         <param name="type">dxl</param>
         <param name="ID">210</param>

File: open_manipulator_description/ros2_control/omy_f3m_end_unit.ros2_control.xacro (robot description, xacro)
@@ -1,5 +1,5 @@
 <?xml version="1.0"?>
 <robot xmlns:xacro="http://www.ros.org/wiki/xacro">
-  <xacro:macro name="omy_f3m_end_unit" params="name prefix port_name:=^|/dev/ttyAMA4 use_sim:=^|false use_fake_hardware:=^|false fake_sensor_commands:=^|false">
+  <xacro:macro name="omy_f3m_end_unit_system" params="name prefix port_name:=^|/dev/ttyAMA4 use_sim:=^|false use_fake_hardware:=^|false fake_sensor_commands:=^|false">
     <ros2_control name="${name}" type="system">
       <xacro:if value="$(arg use_sim)">
@@ -43,24 +43,38 @@
         <state_interface name="effort"/>
       </joint>
-      <!-- <gpio name="dxl7">
-        <param name="type">dxl</param>
-        <param name="ID">7</param>
+      <xacro:if value="$(arg use_sim)">
+        <joint name="${prefix}rh_r2">
+          <param name="mimic">${prefix}rh_r1_joint</param>
+          <param name="multiplier">1</param>
+          <state_interface name="position"/>
+          <state_interface name="velocity"/>
+          <state_interface name="effort"/>
+          <state_interface name="torque_enable"/>
+          <state_interface name="hardware_state"/>
+        </joint>
+        <joint name="${prefix}rh_l1">
+          <param name="mimic">${prefix}rh_r1_joint</param>
+          <param name="multiplier">1</param>
+          <state_interface name="position"/>
+          <state_interface name="velocity"/>
+          <state_interface name="effort"/>
+          <state_interface name="torque_enable"/>
+          <state_interface name="hardware_state"/>
+        </joint>
+        <joint name="${prefix}rh_l2">
+          <param name="mimic">${prefix}rh_r1_joint</param>
+          <param name="multiplier">1</param>
+          <state_interface name="position"/>
+          <state_interface name="velocity"/>
+          <state_interface name="effort"/>
+          <state_interface name="torque_enable"/>
+          <state_interface name="hardware_state"/>
+        </joint>
+      </xacro:if>
+      <gpio name="omy_end">
         <command_interface name="Goal Position"/>
         <state_interface name="Present Position"/>
         <state_interface name="Present Velocity"/>
         <state_interface name="Present Current"/>
-        <state_interface name="Torque Enable"/>
-        <state_interface name="Present Input Voltage"/>
-        <param name="Operating Mode">5</param>
-        <param name="Return Delay Time">0</param>
-      </gpio> -->
-      <gpio name="omy_end">
-        <command_interface name="Goal Position"/>
-        <!-- <command_interface name="Goal Velocity"/> -->
-        <!-- <command_interface name="Goal Current"/> -->
-        <state_interface name="Present Position"/>
-        <state_interface name="Present Velocity"/>
-        <state_interface name="Present Current"/>
-        <state_interface name="Torque Enable"/>
         <param name="type">dxl</param>
         <param name="ID">210</param>

File: open_manipulator_description/ros2_control/omy_l100_system.ros2_control.xacro (robot description, xacro)
@@ -1,5 +1,5 @@
 <?xml version="1.0"?>
 <robot xmlns:xacro="http://www.ros.org/wiki/xacro">
-  <xacro:macro name="omy_l100_system" params="name prefix use_sim:=^|false use_fake_hardware:=^|false fake_sensor_commands:=^|false">
+  <xacro:macro name="omy_l100_system" params="name prefix port_name:=^|/dev/ttyUSB0 use_sim:=^|false use_fake_hardware:=^|false fake_sensor_commands:=^|false">
     <ros2_control name="${name}" type="system">
       <xacro:if value="$(arg use_sim)">
@@ -17,5 +17,5 @@
           <xacro:unless value="${use_fake_hardware}">
             <plugin>dynamixel_hardware_interface/DynamixelHardware</plugin>
-            <param name="port_name">/dev/ttyUSB0</param>
+            <param name="port_name">${port_name}</param>
             <param name="baud_rate">4000000</param>
             <param name="error_timeout_ms">500</param>
@@ -50,5 +50,4 @@
       </xacro:unless>
       <joint name="${prefix}joint1">
-        <command_interface name="position"/>
         <command_interface name="effort"/>
         <state_interface name="position"/>
@@ -57,5 +56,4 @@
       </joint>
       <joint name="${prefix}joint2">
-        <command_interface name="position"/>
         <command_interface name="effort"/>
         <state_interface name="position"/>
@@ -64,5 +62,4 @@
       </joint>
       <joint name="${prefix}joint3">
-        <command_interface name="position"/>
         <command_interface name="effort"/>
         <state_interface name="position"/>
@@ -71,5 +68,4 @@
       </joint>
       <joint name="${prefix}joint4">
-        <command_interface name="position"/>
         <command_interface name="effort"/>
         <state_interface name="position"/>
@@ -78,5 +74,4 @@
       </joint>
       <joint name="${prefix}joint5">
-        <command_interface name="position"/>
         <command_interface name="effort"/>
         <state_interface name="position"/>
@@ -85,5 +80,4 @@
       </joint>
       <joint name="${prefix}joint6">
-        <command_interface name="position"/>
         <command_interface name="effort"/>
         <state_interface name="position"/>
@@ -92,5 +86,4 @@
       </joint>
       <joint name="${prefix}rh_r1_joint">
-        <command_interface name="position"/>
         <command_interface name="effort"/>
         <state_interface name="position"/>
@@ -101,11 +94,8 @@
         <param name="type">dxl</param>
         <param name="ID">1</param>
-        <command_interface name="Goal Position"/>
         <command_interface name="Goal Current"/>
         <state_interface name="Present Position"/>
         <state_interface name="Present Velocity"/>
         <state_interface name="Present Current"/>
-        <state_interface name="Torque Enable"/>
-        <state_interface name="Present Input Voltage"/>
         <param name="Drive Mode">0</param>
         <param name="Operating Mode">0</param>
@@ -116,11 +106,8 @@
         <param name="type">dxl</param>
         <param name="ID">2</param>
-        <command_interface name="Goal Position"/>
         <command_interface name="Goal Current"/>
         <state_interface name="Present Position"/>
         <state_interface name="Present Velocity"/>
         <state_interface name="Present Current"/>
-        <state_interface name="Torque Enable"/>
-        <state_interface name="Present Input Voltage"/>
         <param name="Drive Mode">1</param>
         <param name="Operating Mode">0</param>
@@ -131,11 +118,8 @@
         <param name="type">dxl</param>
         <param name="ID">3</param>
-        <command_interface name="Goal Position"/>
         <command_interface name="Goal Current"/>
         <state_interface name="Present Position"/>
         <state_interface name="Present Velocity"/>
         <state_interface name="Present Current"/>
-        <state_interface name="Torque Enable"/>
-        <state_interface name="Present Input Voltage"/>
         <param name="Drive Mode">0</param>
         <param name="Operating Mode">0</param>
@@ -146,11 +130,8 @@
         <param name="type">dxl</param>
         <param name="ID">4</param>
-        <command_interface name="Goal Position"/>
         <command_interface name="Goal Current"/>
         <state_interface name="Present Position"/>
         <state_interface name="Present Velocity"/>
         <state_interface name="Present Current"/>
-        <state_interface name="Torque Enable"/>
-        <state_interface name="Present Input Voltage"/>
         <param name="Drive Mode">1</param>
         <param name="Operating Mode">0</param>
@@ -161,11 +142,8 @@
         <param name="type">dxl</param>
         <param name="ID">5</param>
-        <command_interface name="Goal Position"/>
         <command_interface name="Goal Current"/>
         <state_interface name="Present Position"/>
         <state_interface name="Present Velocity"/>
         <state_interface name="Present Current"/>
-        <state_interface name="Torque Enable"/>
-        <state_interface name="Present Input Voltage"/>
         <param name="Drive Mode">0</param>
         <param name="Operating Mode">0</param>
@@ -176,11 +154,8 @@
         <param name="type">dxl</param>
         <param name="ID">6</param>
-        <command_interface name="Goal Position"/>
         <command_interface name="Goal Current"/>
         <state_interface name="Present Position"/>
         <state_interface name="Present Velocity"/>
         <state_interface name="Present Current"/>
-        <state_interface name="Torque Enable"/>
-        <state_interface name="Present Input Voltage"/>
         <param name="Drive Mode">1</param>
         <param name="Operating Mode">0</param>
@@ -191,11 +166,8 @@
         <param name="type">dxl</param>
         <param name="ID">7</param>
-        <command_interface name="Goal Position"/>
         <command_interface name="Goal Current"/>
         <state_interface name="Present Position"/>
         <state_interface name="Present Velocity"/>
         <state_interface name="Present Current"/>
-        <state_interface name="Torque Enable"/>
-        <state_interface name="Present Input Voltage"/>
         <param name="Drive Mode">0</param>
         <param name="Operating Mode">0</param>

Commit message: feat: Add 'disable_torque_at_init' parameter to various robot configurations and adjust profile settings in omx and omy files

File: open_manipulator_description/ros2_control/omx.ros2_control.xacro (robot description, xacro)
@@ -23,4 +23,5 @@
             <param name="number_of_joints">5</param>
             <param name="number_of_transmissions">5</param>
+            <param name="disable_torque_at_init">true</param>
             <param name="transmission_to_joint_matrix">
               1, 0, 0, 0, 0,
@@ -98,10 +99,11 @@
         <state_interface name="Present Velocity"/>
         <state_interface name="Present Current"/>
+        <param name="Operating Mode">3</param>
         <param name="Position P Gain">800</param>
         <param name="Position I Gain">100</param>
         <param name="Position D Gain">100</param>
-        <param name="Profile Velocity">200</param>
-        <param name="Profile Acceleration">50</param>
-        <param name="Drive Mode">0</param>
+        <param name="Profile Velocity">11</param>
+        <param name="Profile Acceleration">2</param>
+        <param name="Drive Mode">4</param>
         <param name="Return Delay Time">0</param>
       </gpio>
@@ -113,10 +115,11 @@
         <state_interface name="Present Velocity"/>
         <state_interface name="Present Current"/>
+        <param name="Operating Mode">3</param>
         <param name="Position P Gain">800</param>
         <param name="Position I Gain">100</param>
         <param name="Position D Gain">100</param>
-        <param name="Profile Velocity">200</param>
-        <param name="Profile Acceleration">50</param>
-        <param name="Drive Mode">0</param>
+        <param name="Profile Velocity">11</param>
+        <param name="Profile Acceleration">2</param>
+        <param name="Drive Mode">4</param>
         <param name="Return Delay Time">0</param>
       </gpio>
@@ -128,10 +131,11 @@
         <state_interface name="Present Velocity"/>
         <state_interface name="Present Current"/>
+        <param name="Operating Mode">3</param>
         <param name="Position P Gain">800</param>
         <param name="Position I Gain">100</param>
         <param name="Position D Gain">100</param>
-        <param name="Profile Velocity">200</param>
-        <param name="Profile Acceleration">50</param>
-        <param name="Drive Mode">0</param>
+        <param name="Profile Velocity">11</param>
+        <param name="Profile Acceleration">2</param>
+        <param name="Drive Mode">4</param>
         <param name="Return Delay Time">0</param>
       </gpio>
@@ -143,10 +147,11 @@
         <state_interface name="Present Velocity"/>
         <state_interface name="Present Current"/>
+        <param name="Operating Mode">3</param>
         <param name="Position P Gain">800</param>
         <param name="Position I Gain">100</param>
         <param name="Position D Gain">100</param>
-        <param name="Profile Velocity">200</param>
-        <param name="Profile Acceleration">50</param>
-        <param name="Drive Mode">0</param>
+        <param name="Profile Velocity">11</param>
+        <param name="Profile Acceleration">2</param>
+        <param name="Drive Mode">4</param>
         <param name="Return Delay Time">0</param>
       </gpio>
@@ -158,5 +163,10 @@
         <state_interface name="Present Velocity"/>
         <state_interface name="Present Current"/>
+        <param name="Operating Mode">5</param>
+        <param name="Profile Velocity">11</param>
+        <param name="Profile Acceleration">2</param>
+        <param name="Drive Mode">4</param>
         <param name="Return Delay Time">0</param>
+        <param name="Goal Current">200</param>
       </gpio>
     </ros2_control>

File: open_manipulator_description/ros2_control/omy_3m.ros2_control.xacro (robot description, xacro)
@@ -23,4 +23,5 @@
             <param name="number_of_joints">6</param>
             <param name="number_of_transmissions">6</param>
+            <param name="disable_torque_at_init">true</param>
             <param name="transmission_to_joint_matrix">
               1, 0, 0, 0, 0, 0,

File: open_manipulator_description/ros2_control/omy_3m_end_unit.ros2_control.xacro (robot description, xacro)
@@ -18,4 +18,5 @@
             <param name="number_of_joints">0</param>
             <param name="number_of_transmissions">0</param>
+            <param name="disable_torque_at_init">true</param>
             <param name="transmission_to_joint_matrix"></param>
             <param name="joint_to_transmission_matrix"></param>

File: open_manipulator_description/ros2_control/omy_f3m.ros2_control.xacro (robot description, xacro)
@@ -23,4 +23,5 @@
             <param name="number_of_joints">6</param>
             <param name="number_of_transmissions">6</param>
+            <param name="disable_torque_at_init">true</param>
             <param name="transmission_to_joint_matrix">
               1, 0, 0, 0, 0, 0,

File: open_manipulator_description/ros2_control/omy_f3m_end_unit.ros2_control.xacro (robot description, xacro)
@@ -23,4 +23,5 @@
             <param name="number_of_joints">1</param>
             <param name="number_of_transmissions">1</param>
+            <param name="disable_torque_at_init">true</param>
             <param name="transmission_to_joint_matrix">
               1

File: open_manipulator_description/ros2_control/omy_l100.ros2_control.xacro (robot description, xacro)
@@ -23,4 +23,5 @@
             <param name="number_of_joints">7</param>
             <param name="number_of_transmissions">7</param>
+            <param name="disable_torque_at_init">true</param>
             <param name="transmission_to_joint_matrix">
               1, 0, 0, 0, 0, 0, 0,

File: open_manipulator_description/urdf/omx/omx_arm.urdf.xacro (robot description, xacro)
@@ -162,5 +162,5 @@
       <origin xyz="0.0817 0.021 0.0" rpy="0 0 0"/>
       <axis xyz="0 1 0"/>
-      <limit velocity="4.8" effort="1000" lower="-0.010" upper="0.019" />
+      <limit velocity="4.8" effort="1000" lower="-0.011" upper="0.02" />
       <dynamics damping="0.1"/>
     </joint>
@@ -194,5 +194,5 @@
       <origin xyz="0.0817 -0.021 0" rpy="0 0 0"/>
       <axis xyz="0 -1 0"/>
-      <limit velocity="4.8" effort="1000" lower="-0.010" upper="0.019" />
+      <limit velocity="4.8" effort="1000" lower="-0.011" upper="0.02" />
       <dynamics damping="0.7"/>
       <mimic joint="${prefix}gripper_left_joint" multiplier="1"/>
