Commit message: update robot arm name
Signed-off-by: Junha Cha <ckwnsgk1@gachon.ac.kr>

File: open_manipulator_description/ros2_control/omx_follower.ros2_control.xacro (robot description, xacro)
@@ -1,6 +1,6 @@
 <?xml version="1.0"?>
 <robot xmlns:xacro="http://www.ros.org/wiki/xacro">
-  <xacro:macro name="omx6_leader_system" params="name prefix port_name:=^|/dev/ttyACM0 use_sim:=^|false use_fake_hardware:=^|false fake_sensor_commands:=^|false">
-    <ros2_control name="${name}" type="system">
+  <xacro:macro name="omx_follower_system" params="name prefix port_name:=^|/dev/ttyACM1 use_sim:=^|false use_fake_hardware:=^|false fake_sensor_commands:=^|false">
+    <ros2_control name="${name}" type="system" is_async="true">
       <xacro:if value="$(arg use_sim)">
         <hardware>
@@ -49,30 +49,30 @@
       </xacro:unless>
       <joint name="${prefix}joint1">
-        <command_interface name="effort"/>
+        <command_interface name="position"/>
         <state_interface name="position"/>
         <state_interface name="velocity"/>
       </joint>
       <joint name="${prefix}joint2">
-        <command_interface name="effort"/>
+        <command_interface name="position"/>
         <state_interface name="position"/>
         <state_interface name="velocity"/>
       </joint>
       <joint name="${prefix}joint3">
-        <command_interface name="effort"/>
+        <command_interface name="position"/>
         <state_interface name="position"/>
         <state_interface name="velocity"/>
       </joint>
       <joint name="${prefix}joint4">
-        <command_interface name="effort"/>
+        <command_interface name="position"/>
         <state_interface name="position"/>
         <state_interface name="velocity"/>
       </joint>
       <joint name="${prefix}joint5">
-        <command_interface name="effort"/>
+        <command_interface name="position"/>
         <state_interface name="position"/>
         <state_interface name="velocity"/>
       </joint>
       <joint name="${prefix}joint6">
-        <command_interface name="effort"/>
+        <command_interface name="position"/>
         <state_interface name="position"/>
         <state_interface name="velocity"/>
@@ -81,63 +81,90 @@
         <param name="type">dxl</param>
         <param name="ID">1</param>
+        <command_interface name="Goal Position"/>
         <state_interface name="Present Position"/>
         <state_interface name="Present Velocity"/>
-        <param name="Torque Enable">0</param>
-        <param name="Drive Mode">0</param>
+        <param name="Drive Mode">4</param>
         <param name="Operating Mode">3</param>
         <param name="Return Delay Time">0</param>
+        <param name="Position P Gain">800</param>
+        <param name="Position I Gain">100</param>
+        <param name="Position D Gain">100</param>
+        <param name="Profile Velocity">20</param>
+        <param name="Profile Acceleration">10</param>
       </gpio>
       <gpio name="dxl2">
         <param name="type">dxl</param>
         <param name="ID">2</param>
+        <command_interface name="Goal Position"/>
         <state_interface name="Present Position"/>
         <state_interface name="Present Velocity"/>
-        <param name="Torque Enable">0</param>
-        <param name="Drive Mode">0</param>
+        <param name="Drive Mode">5</param>
         <param name="Operating Mode">3</param>
         <param name="Return Delay Time">0</param>
+        <param name="Position P Gain">800</param>
+        <param name="Position I Gain">100</param>
+        <param name="Position D Gain">100</param>
+        <param name="Profile Velocity">20</param>
+        <param name="Profile Acceleration">10</param>
       </gpio>
       <gpio name="dxl3">
         <param name="type">dxl</param>
         <param name="ID">3</param>
+        <command_interface name="Goal Position"/>
         <state_interface name="Present Position"/>
         <state_interface name="Present Velocity"/>
-        <param name="Torque Enable">0</param>
-        <param name="Drive Mode">0</param>
+        <param name="Drive Mode">5</param>
         <param name="Operating Mode">3</param>
         <param name="Return Delay Time">0</param>
+        <param name="Position P Gain">800</param>
+        <param name="Position I Gain">100</param>
+        <param name="Position D Gain">100</param>
+        <param name="Profile Velocity">20</param>
+        <param name="Profile Acceleration">10</param>
       </gpio>
       <gpio name="dxl4">
         <param name="type">dxl</param>
         <param name="ID">4</param>
+        <command_interface name="Goal Position"/>
         <state_interface name="Present Position"/>
         <state_interface name="Present Velocity"/>
-        <param name="Torque Enable">0</param>
-        <param name="Drive Mode">0</param>
+        <param name="Drive Mode">5</param>
         <param name="Operating Mode">3</param>
         <param name="Return Delay Time">0</param>
+        <param name="Position P Gain">800</param>
+        <param name="Position I Gain">100</param>
+        <param name="Position D Gain">100</param>
+        <param name="Profile Velocity">20</param>
+        <param name="Profile Acceleration">10</param>
       </gpio>
       <gpio name="dxl5">
         <param name="type">dxl</param>
         <param name="ID">5</param>
+        <command_interface name="Goal Position"/>
         <state_interface name="Present Position"/>
         <state_interface name="Present Velocity"/>
-        <param name="Torque Enable">0</param>
-        <param name="Drive Mode">0</param>
+        <param name="Drive Mode">4</param>
         <param name="Operating Mode">3</param>
         <param name="Return Delay Time">0</param>
+        <param name="Position P Gain">800</param>
+        <param name="Position I Gain">100</param>
+        <param name="Position D Gain">100</param>
+        <param name="Profile Velocity">20</param>
+        <param name="Profile Acceleration">10</param>
       </gpio>
       <gpio name="dxl6">
         <param name="type">dxl</param>
         <param name="ID">6</param>
+        <command_interface name="Goal Position"/>
         <state_interface name="Present Position"/>
         <state_interface name="Present Velocity"/>
-        <param name="Torque Enable">1</param>
-        <param name="Drive Mode">0</param>
+        <param name="Drive Mode">4</param>
         <param name="Operating Mode">5</param>
         <param name="Return Delay Time">0</param>
         <param name="Position P Gain">800</param>
-        <param name="Position D Gain">3000</param>
-        <param name="Current Limit">50</param>
+        <param name="Position I Gain">100</param>
+        <param name="Position D Gain">100</param>
+        <param name="Profile Velocity">20</param>
+        <param name="Profile Acceleration">10</param>
       </gpio>
     </ros2_control>

File: open_manipulator_description/ros2_control/omx_leader.ros2_control.xacro (robot description, xacro)
@@ -1,6 +1,6 @@
 <?xml version="1.0"?>
 <robot xmlns:xacro="http://www.ros.org/wiki/xacro">
-  <xacro:macro name="omx6_follower_system" params="name prefix port_name:=^|/dev/ttyACM1 use_sim:=^|false use_fake_hardware:=^|false fake_sensor_commands:=^|false">
-    <ros2_control name="${name}" type="system" is_async="true">
+  <xacro:macro name="omx_leader_system" params="name prefix port_name:=^|/dev/ttyACM0 use_sim:=^|false use_fake_hardware:=^|false fake_sensor_commands:=^|false">
+    <ros2_control name="${name}" type="system">
       <xacro:if value="$(arg use_sim)">
         <hardware>
@@ -49,30 +49,30 @@
       </xacro:unless>
       <joint name="${prefix}joint1">
-        <command_interface name="position"/>
+        <command_interface name="effort"/>
         <state_interface name="position"/>
         <state_interface name="velocity"/>
       </joint>
       <joint name="${prefix}joint2">
-        <command_interface name="position"/>
+        <command_interface name="effort"/>
         <state_interface name="position"/>
         <state_interface name="velocity"/>
       </joint>
       <joint name="${prefix}joint3">
-        <command_interface name="position"/>
+        <command_interface name="effort"/>
         <state_interface name="position"/>
         <state_interface name="velocity"/>
       </joint>
       <joint name="${prefix}joint4">
-        <command_interface name="position"/>
+        <command_interface name="effort"/>
         <state_interface name="position"/>
         <state_interface name="velocity"/>
       </joint>
       <joint name="${prefix}joint5">
-        <command_interface name="position"/>
+        <command_interface name="effort"/>
         <state_interface name="position"/>
         <state_interface name="velocity"/>
       </joint>
       <joint name="${prefix}joint6">
-        <command_interface name="position"/>
+        <command_interface name="effort"/>
         <state_interface name="position"/>
         <state_interface name="velocity"/>
@@ -81,90 +81,63 @@
         <param name="type">dxl</param>
         <param name="ID">1</param>
-        <command_interface name="Goal Position"/>
         <state_interface name="Present Position"/>
         <state_interface name="Present Velocity"/>
-        <param name="Drive Mode">4</param>
+        <param name="Torque Enable">0</param>
+        <param name="Drive Mode">0</param>
         <param name="Operating Mode">3</param>
         <param name="Return Delay Time">0</param>
-        <param name="Position P Gain">800</param>
-        <param name="Position I Gain">100</param>
-        <param name="Position D Gain">100</param>
-        <param name="Profile Velocity">20</param>
-        <param name="Profile Acceleration">10</param>
       </gpio>
       <gpio name="dxl2">
         <param name="type">dxl</param>
         <param name="ID">2</param>
-        <command_interface name="Goal Position"/>
         <state_interface name="Present Position"/>
         <state_interface name="Present Velocity"/>
-        <param name="Drive Mode">5</param>
+        <param name="Torque Enable">0</param>
+        <param name="Drive Mode">0</param>
         <param name="Operating Mode">3</param>
         <param name="Return Delay Time">0</param>
-        <param name="Position P Gain">800</param>
-        <param name="Position I Gain">100</param>
-        <param name="Position D Gain">100</param>
-        <param name="Profile Velocity">20</param>
-        <param name="Profile Acceleration">10</param>
       </gpio>
       <gpio name="dxl3">
         <param name="type">dxl</param>
         <param name="ID">3</param>
-        <command_interface name="Goal Position"/>
         <state_interface name="Present Position"/>
         <state_interface name="Present Velocity"/>
-        <param name="Drive Mode">5</param>
+        <param name="Torque Enable">0</param>
+        <param name="Drive Mode">0</param>
         <param name="Operating Mode">3</param>
         <param name="Return Delay Time">0</param>
-        <param name="Position P Gain">800</param>
-        <param name="Position I Gain">100</param>
-        <param name="Position D Gain">100</param>
-        <param name="Profile Velocity">20</param>
-        <param name="Profile Acceleration">10</param>
       </gpio>
       <gpio name="dxl4">
         <param name="type">dxl</param>
         <param name="ID">4</param>
-        <command_interface name="Goal Position"/>
         <state_interface name="Present Position"/>
         <state_interface name="Present Velocity"/>
-        <param name="Drive Mode">5</param>
+        <param name="Torque Enable">0</param>
+        <param name="Drive Mode">0</param>
         <param name="Operating Mode">3</param>
         <param name="Return Delay Time">0</param>
-        <param name="Position P Gain">800</param>
-        <param name="Position I Gain">100</param>
-        <param name="Position D Gain">100</param>
-        <param name="Profile Velocity">20</param>
-        <param name="Profile Acceleration">10</param>
       </gpio>
       <gpio name="dxl5">
         <param name="type">dxl</param>
         <param name="ID">5</param>
-        <command_interface name="Goal Position"/>
         <state_interface name="Present Position"/>
         <state_interface name="Present Velocity"/>
-        <param name="Drive Mode">4</param>
+        <param name="Torque Enable">0</param>
+        <param name="Drive Mode">0</param>
         <param name="Operating Mode">3</param>
         <param name="Return Delay Time">0</param>
-        <param name="Position P Gain">800</param>
-        <param name="Position I Gain">100</param>
-        <param name="Position D Gain">100</param>
-        <param name="Profile Velocity">20</param>
-        <param name="Profile Acceleration">10</param>
       </gpio>
       <gpio name="dxl6">
         <param name="type">dxl</param>
         <param name="ID">6</param>
-        <command_interface name="Goal Position"/>
         <state_interface name="Present Position"/>
         <state_interface name="Present Velocity"/>
-        <param name="Drive Mode">4</param>
+        <param name="Torque Enable">1</param>
+        <param name="Drive Mode">0</param>
         <param name="Operating Mode">5</param>
         <param name="Return Delay Time">0</param>
         <param name="Position P Gain">800</param>
-        <param name="Position I Gain">100</param>
-        <param name="Position D Gain">100</param>
-        <param name="Profile Velocity">20</param>
-        <param name="Profile Acceleration">10</param>
+        <param name="Position D Gain">3000</param>
+        <param name="Current Limit">50</param>
       </gpio>
     </ros2_control>

File: open_manipulator_description/urdf/omx_follower/omx_follower.urdf.xacro (robot description, xacro)
@@ -1,11 +1,12 @@
 <?xml version="1.0"?>
-<robot name="omx6_leader" xmlns:xacro="http://www.ros.org/wiki/xacro">
+<robot name="omx_follower" xmlns:xacro="http://www.ros.org/wiki/xacro">
   <xacro:arg name="prefix" default="" />
   <xacro:arg name="use_sim" default="false" />
   <xacro:arg name="use_fake_hardware" default="false" />
   <xacro:arg name="fake_sensor_commands" default="false" />
+  <xacro:arg name="config_type" default="omx_follower" />
+  <xacro:arg name="ros2_control_type" default="omx_follower" />
   <xacro:arg name="port_name" default="/dev/ttyACM1" />
-  <xacro:arg name="ros2_control_type" default="omx6_leader" />
-  <xacro:include filename="$(find open_manipulator_description)/urdf/omx6_leader/omx6_leader_arm.urdf" />
+  <xacro:include filename="$(find open_manipulator_description)/urdf/omx_follower/omx_follower_arm.urdf.xacro" />
   <xacro:include filename="$(find open_manipulator_description)/ros2_control/$(arg ros2_control_type).ros2_control.xacro" />
   <link name="world"/>
@@ -15,9 +16,10 @@
     <origin xyz="0.0 0.0 0.0" rpy="0 0 0"/>
   </joint>
-  <xacro:omx6_leader prefix="$(arg prefix)" />
-  <xacro:omx6_leader_system
-    name="OMX6LEADERSYSTEM" prefix="$(arg prefix)" use_sim="$(arg use_sim)"
+  <xacro:omx_follower prefix="$(arg prefix)" />
+  <xacro:omx_follower_system
+    name="OMXFOLLOWERSystem" prefix="$(arg prefix)" use_sim="$(arg use_sim)"
     use_fake_hardware="$(arg use_fake_hardware)"
     fake_sensor_commands="$(arg fake_sensor_commands)"
-    port_name="$(arg port_name)"/>
+    port_name="$(arg port_name)"
+    />
 </robot>

File: open_manipulator_description/urdf/omx_follower/omx_follower_arm.urdf.xacro (robot description, xacro)
@@ -1,5 +1,5 @@
 <?xml version="1.0" encoding="UTF-8"?>
 <robot xmlns:xacro="http://www.ros.org/wiki/xacro">
-   <xacro:macro name="omx6_follower" params="prefix">
+   <xacro:macro name="omx_follower" params="prefix">
       <link name="${prefix}link0" />
       <joint name="${prefix}joint1" type="revolute">

File: open_manipulator_description/urdf/omx_leader/omx_leader.urdf.xacro (robot description, xacro)
@@ -1,12 +1,11 @@
 <?xml version="1.0"?>
-<robot name="omx6_follower" xmlns:xacro="http://www.ros.org/wiki/xacro">
+<robot name="omx_leader" xmlns:xacro="http://www.ros.org/wiki/xacro">
   <xacro:arg name="prefix" default="" />
   <xacro:arg name="use_sim" default="false" />
   <xacro:arg name="use_fake_hardware" default="false" />
   <xacro:arg name="fake_sensor_commands" default="false" />
-  <xacro:arg name="config_type" default="omx6_follower" />
-  <xacro:arg name="ros2_control_type" default="omx6_follower" />
   <xacro:arg name="port_name" default="/dev/ttyACM1" />
-  <xacro:include filename="$(find open_manipulator_description)/urdf/omx6_follower/omx6_follower_arm.urdf.xacro" />
+  <xacro:arg name="ros2_control_type" default="omx_leader" />
+  <xacro:include filename="$(find open_manipulator_description)/urdf/omx_leader/omx_leader_arm.urdf" />
   <xacro:include filename="$(find open_manipulator_description)/ros2_control/$(arg ros2_control_type).ros2_control.xacro" />
   <link name="world"/>
@@ -16,10 +15,9 @@
     <origin xyz="0.0 0.0 0.0" rpy="0 0 0"/>
   </joint>
-  <xacro:omx6_follower prefix="$(arg prefix)" />
-  <xacro:omx6_follower_system
-    name="OMX6FOLLOWERSystem" prefix="$(arg prefix)" use_sim="$(arg use_sim)"
+  <xacro:omx_leader prefix="$(arg prefix)" />
+  <xacro:omx_leader_system
+    name="OMXLEADERSYSTEM" prefix="$(arg prefix)" use_sim="$(arg use_sim)"
     use_fake_hardware="$(arg use_fake_hardware)"
     fake_sensor_commands="$(arg fake_sensor_commands)"
-    port_name="$(arg port_name)"
-    />
+    port_name="$(arg port_name)"/>
 </robot>
