Commit message: Refactor: rename joint6 to gripper_joint_1 in configuration and URDF files for consistency across hardware controller and initial positions

File: open_manipulator_description/ros2_control/omx_l.ros2_control.xacro (robot description, xacro)
@@ -68,5 +68,5 @@
         <state_interface name="velocity"/>
       </joint>
-      <joint name="${prefix}joint6">
+      <joint name="${prefix}gripper_joint_1">
         <command_interface name="position"/>
         <state_interface name="position"/>

File: open_manipulator_description/urdf/omx_f/omx_f_arm.urdf.xacro (robot description, xacro)
@@ -48,5 +48,5 @@
       </joint>
       <link name="${prefix}link5" />
-      <joint name="${prefix}joint6" type="revolute">
+      <joint name="${prefix}gripper_joint_1" type="revolute">
          <parent link="${prefix}link5" />
          <child link="${prefix}link6" />
