Commit message: update OMX launch file without URDF file
Signed-off-by: Junha Cha <ckwnsgk1@gachon.ac.kr>

File: open_manipulator_description/ros2_control/omx_f.ros2_control.xacro (robot description, xacro)
@@ -1,5 +1,5 @@
 <?xml version="1.0"?>
 <robot xmlns:xacro="http://www.ros.org/wiki/xacro">
-  <xacro:macro name="omx_follower_system" params="name prefix port_name:=^|/dev/ttyACM1 use_sim:=^|false use_fake_hardware:=^|false fake_sensor_commands:=^|false">
+  <xacro:macro name="omx_f_system" params="name prefix port_name:=^|/dev/ttyACM1 use_sim:=^|false use_fake_hardware:=^|false fake_sensor_commands:=^|false">
     <ros2_control name="${name}" type="system" is_async="true">
       <xacro:if value="$(arg use_sim)">
@@ -85,8 +85,8 @@
         <state_interface name="Present Velocity"/>
         <param name="Drive Mode">4</param>
-        <param name="Operating Mode">3</param>
+        <param name="Operating Mode">4</param>
         <param name="Return Delay Time">0</param>
-        <param name="Position P Gain">800</param>
-        <param name="Position I Gain">100</param>
+        <param name="Position P Gain">1000</param>
+        <param name="Position I Gain">0</param>
         <param name="Position D Gain">100</param>
         <param name="Profile Velocity">100</param>
@@ -102,6 +102,6 @@
         <param name="Operating Mode">3</param>
         <param name="Return Delay Time">0</param>
-        <param name="Position P Gain">800</param>
-        <param name="Position I Gain">100</param>
+        <param name="Position P Gain">1000</param>
+        <param name="Position I Gain">0</param>
         <param name="Position D Gain">100</param>
         <param name="Profile Velocity">100</param>
@@ -117,6 +117,6 @@
         <param name="Operating Mode">3</param>
         <param name="Return Delay Time">0</param>
-        <param name="Position P Gain">800</param>
-        <param name="Position I Gain">100</param>
+        <param name="Position P Gain">1000</param>
+        <param name="Position I Gain">0</param>
         <param name="Position D Gain">100</param>
         <param name="Profile Velocity">100</param>
@@ -132,6 +132,6 @@
         <param name="Operating Mode">3</param>
         <param name="Return Delay Time">0</param>
-        <param name="Position P Gain">800</param>
-        <param name="Position I Gain">100</param>
+        <param name="Position P Gain">1000</param>
+        <param name="Position I Gain">0</param>
         <param name="Position D Gain">100</param>
         <param name="Profile Velocity">100</param>
@@ -145,8 +145,8 @@
         <state_interface name="Present Velocity"/>
         <param name="Drive Mode">4</param>
-        <param name="Operating Mode">3</param>
+        <param name="Operating Mode">4</param>
         <param name="Return Delay Time">0</param>
-        <param name="Position P Gain">800</param>
-        <param name="Position I Gain">100</param>
+        <param name="Position P Gain">1000</param>
+        <param name="Position I Gain">0</param>
         <param name="Position D Gain">100</param>
         <param name="Profile Velocity">100</param>
@@ -159,9 +159,9 @@
         <state_interface name="Present Position"/>
         <state_interface name="Present Velocity"/>
-        <param name="Drive Mode">4</param>
+        <param name="Drive Mode">5</param>
         <param name="Operating Mode">5</param>
         <param name="Return Delay Time">0</param>
-        <param name="Position P Gain">800</param>
-        <param name="Position I Gain">100</param>
+        <param name="Position P Gain">1000</param>
+        <param name="Position I Gain">0</param>
         <param name="Position D Gain">100</param>
         <param name="Profile Velocity">100</param>

File: open_manipulator_description/ros2_control/omx_l.ros2_control.xacro (robot description, xacro)
@@ -1,5 +1,5 @@
 <?xml version="1.0"?>
 <robot xmlns:xacro="http://www.ros.org/wiki/xacro">
-  <xacro:macro name="omx_leader_system" params="name prefix port_name:=^|/dev/ttyACM0 use_sim:=^|false use_fake_hardware:=^|false fake_sensor_commands:=^|false">
+  <xacro:macro name="omx_l_system" params="name prefix port_name:=^|/dev/ttyACM0 use_sim:=^|false use_fake_hardware:=^|false fake_sensor_commands:=^|false">
     <ros2_control name="${name}" type="system">
       <xacro:if value="$(arg use_sim)">
@@ -85,5 +85,5 @@
         <param name="Torque Enable">0</param>
         <param name="Drive Mode">0</param>
-        <param name="Operating Mode">3</param>
+        <param name="Operating Mode">4</param>
         <param name="Return Delay Time">0</param>
       </gpio>
@@ -125,5 +125,5 @@
         <param name="Torque Enable">0</param>
         <param name="Drive Mode">0</param>
-        <param name="Operating Mode">3</param>
+        <param name="Operating Mode">4</param>
         <param name="Return Delay Time">0</param>
       </gpio>
@@ -139,5 +139,5 @@
         <param name="Position P Gain">800</param>
         <param name="Position D Gain">3000</param>
-        <param name="Current Limit">50</param>
+        <param name="Current Limit">300</param>
       </gpio>
     </ros2_control>

File: open_manipulator_description/urdf/omx_f/omx_f.urdf.xacro (robot description, xacro)
@@ -1,12 +1,12 @@
 <?xml version="1.0"?>
-<robot name="omx_follower" xmlns:xacro="http://www.ros.org/wiki/xacro">
+<robot name="omx_f" xmlns:xacro="http://www.ros.org/wiki/xacro">
   <xacro:arg name="prefix" default="" />
   <xacro:arg name="use_sim" default="false" />
   <xacro:arg name="use_fake_hardware" default="false" />
   <xacro:arg name="fake_sensor_commands" default="false" />
-  <xacro:arg name="config_type" default="omx_follower" />
-  <xacro:arg name="ros2_control_type" default="omx_follower" />
+  <xacro:arg name="config_type" default="omx_f" />
+  <xacro:arg name="ros2_control_type" default="omx_f" />
   <xacro:arg name="port_name" default="/dev/ttyACM1" />
-  <xacro:include filename="$(find open_manipulator_description)/urdf/omx_follower/omx_follower_arm.urdf.xacro" />
+  <xacro:include filename="$(find open_manipulator_description)/urdf/omx_f/omx_f_arm.urdf.xacro" />
   <xacro:include filename="$(find open_manipulator_description)/ros2_control/$(arg ros2_control_type).ros2_control.xacro" />
   <link name="world"/>
@@ -16,6 +16,6 @@
     <origin xyz="0.0 0.0 0.0" rpy="0 0 0"/>
   </joint>
-  <xacro:omx_follower prefix="$(arg prefix)" />
-  <xacro:omx_follower_system
+  <xacro:omx_f prefix="$(arg prefix)" />
+  <xacro:omx_f_system
     name="OMXFOLLOWERSystem" prefix="$(arg prefix)" use_sim="$(arg use_sim)"
     use_fake_hardware="$(arg use_fake_hardware)"

File: open_manipulator_description/urdf/omx_f/omx_f_arm.urdf.xacro (robot description, xacro)
@@ -1,5 +1,5 @@
 <?xml version="1.0" encoding="UTF-8"?>
 <robot xmlns:xacro="http://www.ros.org/wiki/xacro">
-   <xacro:macro name="omx_leader" params="prefix">
+   <xacro:macro name="omx_f" params="prefix">
       <link name="${prefix}link0" />
       <joint name="${prefix}joint1" type="revolute">

File: open_manipulator_description/urdf/omx_l/omx_l.urdf.xacro (robot description, xacro)
@@ -1,4 +1,4 @@
 <?xml version="1.0"?>
-<robot name="omx_leader" xmlns:xacro="http://www.ros.org/wiki/xacro">
+<robot name="omx_l" xmlns:xacro="http://www.ros.org/wiki/xacro">
   <xacro:arg name="prefix" default="" />
   <xacro:arg name="use_sim" default="false" />
@@ -6,6 +6,6 @@
   <xacro:arg name="fake_sensor_commands" default="false" />
   <xacro:arg name="port_name" default="/dev/ttyACM1" />
-  <xacro:arg name="ros2_control_type" default="omx_leader" />
-  <xacro:include filename="$(find open_manipulator_description)/urdf/omx_leader/omx_leader_arm.urdf" />
+  <xacro:arg name="ros2_control_type" default="omx_l" />
+  <xacro:include filename="$(find open_manipulator_description)/urdf/omx_l/omx_l_arm.urdf" />
   <xacro:include filename="$(find open_manipulator_description)/ros2_control/$(arg ros2_control_type).ros2_control.xacro" />
   <link name="world"/>
@@ -15,6 +15,6 @@
     <origin xyz="0.0 0.0 0.0" rpy="0 0 0"/>
   </joint>
-  <xacro:omx_leader prefix="$(arg prefix)" />
-  <xacro:omx_leader_system
+  <xacro:omx_l prefix="$(arg prefix)" />
+  <xacro:omx_l_system
     name="OMXLEADERSYSTEM" prefix="$(arg prefix)" use_sim="$(arg use_sim)"
     use_fake_hardware="$(arg use_fake_hardware)"

Commit message: adjust GPIO IDs for hardware configuration consistency

File: open_manipulator_description/ros2_control/omx_f.ros2_control.xacro (robot description, xacro)
@@ -73,5 +73,5 @@
         <state_interface name="velocity"/>
       </joint>
-      <joint name="${prefix}joint6">
+      <joint name="${prefix}gripper_joint_1">
         <command_interface name="position"/>
         <state_interface name="position"/>
@@ -80,5 +80,5 @@
       <gpio name="dxl1">
         <param name="type">dxl</param>
-        <param name="ID">1</param>
+        <param name="ID">11</param>
         <command_interface name="Goal Position"/>
         <state_interface name="Present Position"/>
@@ -97,5 +97,5 @@
       <gpio name="dxl2">
         <param name="type">dxl</param>
-        <param name="ID">2</param>
+        <param name="ID">12</param>
         <command_interface name="Goal Position"/>
         <state_interface name="Present Position"/>
@@ -114,5 +114,5 @@
       <gpio name="dxl3">
         <param name="type">dxl</param>
-        <param name="ID">3</param>
+        <param name="ID">13</param>
         <command_interface name="Goal Position"/>
         <state_interface name="Present Position"/>
@@ -131,5 +131,5 @@
       <gpio name="dxl4">
         <param name="type">dxl</param>
-        <param name="ID">4</param>
+        <param name="ID">14</param>
         <command_interface name="Goal Position"/>
         <state_interface name="Present Position"/>
@@ -148,5 +148,5 @@
       <gpio name="dxl5">
         <param name="type">dxl</param>
-        <param name="ID">5</param>
+        <param name="ID">15</param>
         <command_interface name="Goal Position"/>
         <state_interface name="Present Position"/>
@@ -165,5 +165,5 @@
       <gpio name="dxl6">
         <param name="type">dxl</param>
-        <param name="ID">6</param>
+        <param name="ID">16</param>
         <command_interface name="Goal Position"/>
         <state_interface name="Present Position"/>
@@ -177,6 +177,6 @@
         <param name="Profile Velocity">50</param>
         <param name="Profile Acceleration">25</param>
-        <param name="Current Limit">1000</param>
-        <param name="Goal Current">1000</param>
+        <param name="Current Limit">100</param>
+        <param name="Goal Current">100</param>
       </gpio>
     </ros2_control>

Commit message: feat: Add gripper_joint_2 for simulation support in omx_f configuration

File: open_manipulator_description/ros2_control/omx_f.ros2_control.xacro (robot description, xacro)
@@ -78,4 +78,13 @@
         <state_interface name="velocity"/>
       </joint>
+      <xacro:if value="$(arg use_sim)">
+        <joint name="${prefix}gripper_joint_2">
+          <param name="mimic">${prefix}gripper_joint_1</param>
+          <param name="multiplier">-1</param>
+          <state_interface name="position"/>
+          <state_interface name="velocity"/>
+          <state_interface name="effort"/>
+        </joint>
+      </xacro:if>
       <gpio name="dxl1">
         <param name="type">dxl</param>
