Commit message: Add bi manipulation

File: open_manipulator_description/ros2_control/omx_f.ros2_control.xacro (robot description, xacro)
@@ -1,5 +1,5 @@
 <?xml version="1.0"?>
 <robot xmlns:xacro="http://www.ros.org/wiki/xacro">
-  <xacro:macro name="omx_f_system" params="name prefix port_name:=^|/dev/ttyACM1 use_sim:=^|false use_mock_hardware:=^|false mock_sensor_commands:=^|false">
+  <xacro:macro name="omx_f_system" params="name prefix port_name:=^|/dev/ttyACM1 use_sim:=^|false use_mock_hardware:=^|false mock_sensor_commands:=^|false resource_prefix:='' hardware_namespace:=''">
     <ros2_control name="${name}" type="system" is_async="true">
       <xacro:if value="$(arg use_sim)">
@@ -24,9 +24,9 @@
             <param name="number_of_transmissions">6</param>
             <param name="disable_torque_at_init">true</param>
-            <param name="dynamixel_state_pub_msg_name">dynamixel_hardware_interface/dxl_state</param>
-            <param name="get_dynamixel_data_srv_name">dynamixel_hardware_interface/get_dxl_data</param>
-            <param name="set_dynamixel_data_srv_name">dynamixel_hardware_interface/set_dxl_data</param>
-            <param name="reboot_dxl_srv_name">dynamixel_hardware_interface/reboot_dxl</param>
-            <param name="set_dxl_torque_srv_name">dynamixel_hardware_interface/set_dxl_torque</param>
+            <param name="dynamixel_state_pub_msg_name">${hardware_namespace}dynamixel_hardware_interface/dxl_state</param>
+            <param name="get_dynamixel_data_srv_name">${hardware_namespace}dynamixel_hardware_interface/get_dxl_data</param>
+            <param name="set_dynamixel_data_srv_name">${hardware_namespace}dynamixel_hardware_interface/set_dxl_data</param>
+            <param name="reboot_dxl_srv_name">${hardware_namespace}dynamixel_hardware_interface/reboot_dxl</param>
+            <param name="set_dxl_torque_srv_name">${hardware_namespace}dynamixel_hardware_interface/set_dxl_torque</param>
           </xacro:unless>
         </hardware>
@@ -71,5 +71,5 @@
         </joint>
       </xacro:if>
-      <gpio name="dxl11">
+      <gpio name="${resource_prefix}dxl11">
         <param name="type">dxl</param>
         <param name="ID">11</param>
@@ -86,5 +86,5 @@
         <param name="Profile Acceleration">25</param>
       </gpio>
-      <gpio name="dxl12">
+      <gpio name="${resource_prefix}dxl12">
         <param name="type">dxl</param>
         <param name="ID">12</param>
@@ -103,5 +103,5 @@
         <param name="Profile Acceleration">25</param>
       </gpio>
-      <gpio name="dxl13">
+      <gpio name="${resource_prefix}dxl13">
         <param name="type">dxl</param>
         <param name="ID">13</param>
@@ -120,5 +120,5 @@
         <param name="Profile Acceleration">25</param>
       </gpio>
-      <gpio name="dxl14">
+      <gpio name="${resource_prefix}dxl14">
         <param name="type">dxl</param>
         <param name="ID">14</param>
@@ -137,5 +137,5 @@
         <param name="Profile Acceleration">25</param>
       </gpio>
-      <gpio name="dxl15">
+      <gpio name="${resource_prefix}dxl15">
         <param name="type">dxl</param>
         <param name="ID">15</param>
@@ -154,5 +154,5 @@
         <param name="Profile Acceleration">25</param>
       </gpio>
-      <gpio name="dxl16">
+      <gpio name="${resource_prefix}dxl16">
         <param name="type">dxl</param>
         <param name="ID">16</param>

File: open_manipulator_description/ros2_control/omx_l.ros2_control.xacro (robot description, xacro)
@@ -1,5 +1,5 @@
 <?xml version="1.0"?>
 <robot xmlns:xacro="http://www.ros.org/wiki/xacro">
-  <xacro:macro name="omx_l_system" params="name prefix port_name:=^|/dev/ttyACM0 use_sim:=^|false use_mock_hardware:=^|false mock_sensor_commands:=^|false">
+  <xacro:macro name="omx_l_system" params="name prefix port_name:=^|/dev/ttyACM0 use_sim:=^|false use_mock_hardware:=^|false mock_sensor_commands:=^|false resource_prefix:='' hardware_namespace:=''">
     <ros2_control name="${name}" type="system">
       <xacro:if value="$(arg use_sim)">
@@ -24,9 +24,9 @@
             <param name="number_of_transmissions">6</param>
             <param name="disable_torque_at_init">true</param>
-            <param name="dynamixel_state_pub_msg_name">omx_l/dxl_state</param>
-            <param name="get_dynamixel_data_srv_name">omx_l/get_dxl_data</param>
-            <param name="set_dynamixel_data_srv_name">omx_l/set_dxl_data</param>
-            <param name="reboot_dxl_srv_name">omx_l/reboot_dxl</param>
-            <param name="set_dxl_torque_srv_name">omx_l/set_dxl_torque</param>
+            <param name="dynamixel_state_pub_msg_name">${hardware_namespace}omx_l/dxl_state</param>
+            <param name="get_dynamixel_data_srv_name">${hardware_namespace}omx_l/get_dxl_data</param>
+            <param name="set_dynamixel_data_srv_name">${hardware_namespace}omx_l/set_dxl_data</param>
+            <param name="reboot_dxl_srv_name">${hardware_namespace}omx_l/reboot_dxl</param>
+            <param name="set_dxl_torque_srv_name">${hardware_namespace}omx_l/set_dxl_torque</param>
           </xacro:unless>
         </hardware>
@@ -68,5 +68,5 @@
         <!-- <state_interface name="effort"/> -->
       </joint>
-      <gpio name="dxl1">
+      <gpio name="${resource_prefix}dxl1">
         <param name="type">dxl</param>
         <param name="ID">1</param>
@@ -80,5 +80,5 @@
         <param name="Return Delay Time">0</param>
       </gpio>
-      <gpio name="dxl2">
+      <gpio name="${resource_prefix}dxl2">
         <param name="type">dxl</param>
         <param name="ID">2</param>
@@ -92,5 +92,5 @@
         <param name="Return Delay Time">0</param>
       </gpio>
-      <gpio name="dxl3">
+      <gpio name="${resource_prefix}dxl3">
         <param name="type">dxl</param>
         <param name="ID">3</param>
@@ -104,5 +104,5 @@
         <param name="Return Delay Time">0</param>
       </gpio>
-      <gpio name="dxl4">
+      <gpio name="${resource_prefix}dxl4">
         <param name="type">dxl</param>
         <param name="ID">4</param>
@@ -116,5 +116,5 @@
         <param name="Return Delay Time">0</param>
       </gpio>
-      <gpio name="dxl5">
+      <gpio name="${resource_prefix}dxl5">
         <param name="type">dxl</param>
         <param name="ID">5</param>
@@ -128,5 +128,5 @@
         <param name="Return Delay Time">0</param>
       </gpio>
-      <gpio name="dxl6">
+      <gpio name="${resource_prefix}dxl6">
         <param name="type">dxl</param>
         <param name="ID">6</param>
