Commit message: control_changed

File: open_manipulator_description/ros2_control/omy_f3m_end_unit_hx5_right.ros2_control.xacro (robot description, xacro)
@@ -11,5 +11,5 @@
 -->
 <robot xmlns:xacro="http://www.ros.org/wiki/xacro">
-  <xacro:macro name="omy_f3m_end_unit_hx5_right_system" params="name prefix port_name:=^|/dev/rp1ctrluart4 use_sim:=^|false use_mock_hardware:=^|false mock_sensor_commands:=^|false">
+  <xacro:macro name="omy_f3m_end_unit_hx5_right_system" params="name prefix port_name:=^|/dev/ttyAMA4 dynamixel_model_folder:=^|/param/dxl_model configure_hx5_synctable:=^|false use_sim:=^|false use_mock_hardware:=^|false mock_sensor_commands:=^|false">
     <ros2_control name="${name}" type="system" is_async="true">
       <xacro:if value="$(arg use_sim)">
@@ -30,5 +30,5 @@
             <param name="baud_rate">4000000</param>
             <param name="error_timeout_ms">500</param>
-            <param name="dynamixel_model_folder">/param/dxl_model</param>
+            <param name="dynamixel_model_folder">${dynamixel_model_folder}</param>
             <param name="number_of_joints">20</param>
             <param name="number_of_transmissions">20</param>
@@ -188,14 +188,27 @@
         <state_interface name="effort"/>
       </joint>
+      <sensor name="${prefix}finger_r_sensor1"><state_interface name="Present Pressure 5"/></sensor>
+      <sensor name="${prefix}finger_r_sensor2"><state_interface name="Present Pressure 5"/></sensor>
+      <sensor name="${prefix}finger_r_sensor3"><state_interface name="Present Pressure 5"/></sensor>
+      <sensor name="${prefix}finger_r_sensor4"><state_interface name="Present Pressure 5"/></sensor>
+      <sensor name="${prefix}finger_r_sensor5"><state_interface name="Present Pressure 5"/></sensor>
       <!-- OMY END pre-init (disable SyncTable) -->
       <gpio name="omy_end_pre">
+        <state_interface name="Button Status"/>
         <param name="type">controller</param>
         <param name="ID">210</param>
+        <param name="Baud Rate (Bus)">6</param>
         <param name="SyncTable Enable">0</param>
-        <param name="SyncTable Enable HX5">0</param>
         <param name="Tool Analog Enable">0</param>
         <param name="Tool Baud Rate">8</param>
         <param name="Tool Protocol">0</param>
-        <param name="Tool ID">1</param>
+        <param name="Tool ID">110</param>
+        <param name="R LED">200</param>
+        <param name="G LED">200</param>
+        <param name="B LED">120</param>
+        <param name="SyncTable Read Address">634</param>
+        <param name="SyncTable Read Size">125</param>
+        <param name="SyncTable Write Address">799</param>
+        <param name="SyncTable Write Size">80</param>
       </gpio>
       <!-- HX5 hub (ID 110) init + SyncTable config -->
@@ -203,592 +216,17 @@
         <param name="type">controller</param>
         <param name="ID">110</param>
-        <param name="Table Sync Enable">0</param>
-        <param name="Bus Watchdog">100</param>
-        <param name="SyncTable 1 ID 1">111</param>
-        <param name="SyncTable 1 ID 2">112</param>
-        <param name="SyncTable 1 ID 3">113</param>
-        <param name="SyncTable 1 ID 4">114</param>
-        <param name="SyncTable 1 ID 5">115</param>
-        <param name="SyncTable 2 ID 1">116</param>
-        <param name="SyncTable 2 ID 2">117</param>
-        <param name="SyncTable 2 ID 3">118</param>
-        <param name="SyncTable 2 ID 4">119</param>
-        <param name="SyncTable 2 ID 5">120</param>
-        <param name="SyncTable 3 ID 1">121</param>
-        <param name="SyncTable 3 ID 2">122</param>
-        <param name="SyncTable 3 ID 3">123</param>
-        <param name="SyncTable 3 ID 4">124</param>
-        <param name="SyncTable 3 ID 5">125</param>
-        <param name="SyncTable 4 ID 1">126</param>
-        <param name="SyncTable 4 ID 2">127</param>
-        <param name="SyncTable 4 ID 3">128</param>
-        <param name="SyncTable 4 ID 4">129</param>
-        <param name="SyncTable 4 ID 5">130</param>
-        <param name="SyncTable 5 ID 1">131</param>
-        <param name="SyncTable 5 ID 2">132</param>
-        <param name="SyncTable 5 ID 3">133</param>
-        <param name="SyncTable 5 ID 4">134</param>
-        <param name="SyncTable 5 ID 5">135</param>
-        <param name="SyncTable 1 Read Address 1">224</param>
-        <param name="SyncTable 1 Read Address 2">224</param>
-        <param name="SyncTable 1 Read Address 3">224</param>
-        <param name="SyncTable 1 Read Address 4">224</param>
-        <param name="SyncTable 1 Read Address 5">72</param>
-        <param name="SyncTable 1 Read Size 1">6</param>
-        <param name="SyncTable 1 Read Size 2">6</param>
-        <param name="SyncTable 1 Read Size 3">6</param>
-        <param name="SyncTable 1 Read Size 4">6</param>
-        <param name="SyncTable 1 Read Size 5">9</param>
-        <param name="SyncTable 1 Write Address 1">230</param>
-        <param name="SyncTable 1 Write Address 2">230</param>
-        <param name="SyncTable 1 Write Address 3">230</param>
-        <param name="SyncTable 1 Write Address 4">230</param>
-        <param name="SyncTable 1 Write Address 5">0</param>
-        <param name="SyncTable 1 Write Size 1">4</param>
-        <param name="SyncTable 1 Write Size 2">4</param>
-        <param name="SyncTable 1 Write Size 3">4</param>
-        <param name="SyncTable 1 Write Size 4">4</param>
-        <param name="SyncTable 1 Write Size 5">0</param>
-        <param name="SyncTable 2 Read Address 1">224</param>
-        <param name="SyncTable 2 Read Address 2">224</param>
-        <param name="SyncTable 2 Read Address 3">224</param>
-        <param name="SyncTable 2 Read Address 4">224</param>
-        <param name="SyncTable 2 Read Address 5">72</param>
-        <param name="SyncTable 2 Read Size 1">6</param>
-        <param name="SyncTable 2 Read Size 2">6</param>
-        <param name="SyncTable 2 Read Size 3">6</param>
-        <param name="SyncTable 2 Read Size 4">6</param>
-        <param name="SyncTable 2 Read Size 5">9</param>
-        <param name="SyncTable 2 Write Address 1">230</param>
-        <param name="SyncTable 2 Write Address 2">230</param>
-        <param name="SyncTable 2 Write Address 3">230</param>
-        <param name="SyncTable 2 Write Address 4">230</param>
-        <param name="SyncTable 2 Write Address 5">0</param>
-        <param name="SyncTable 2 Write Size 1">4</param>
-        <param name="SyncTable 2 Write Size 2">4</param>
-        <param name="SyncTable 2 Write Size 3">4</param>
-        <param name="SyncTable 2 Write Size 4">4</param>
-        <param name="SyncTable 2 Write Size 5">0</param>
-        <param name="SyncTable 3 Read Address 1">224</param>
-        <param name="SyncTable 3 Read Address 2">224</param>
-        <param name="SyncTable 3 Read Address 3">224</param>
-        <param name="SyncTable 3 Read Address 4">224</param>
-        <param name="SyncTable 3 Read Address 5">72</param>
-        <param name="SyncTable 3 Read Size 1">6</param>
-        <param name="SyncTable 3 Read Size 2">6</param>
-        <param name="SyncTable 3 Read Size 3">6</param>
-        <param name="SyncTable 3 Read Size 4">6</param>
-        <param name="SyncTable 3 Read Size 5">9</param>
-        <param name="SyncTable 3 Write Address 1">230</param>
-        <param name="SyncTable 3 Write Address 2">230</param>
-        <param name="SyncTable 3 Write Address 3">230</param>
-        <param name="SyncTable 3 Write Address 4">230</param>
-        <param name="SyncTable 3 Write Address 5">0</param>
-        <param name="SyncTable 3 Write Size 1">4</param>
-        <param name="SyncTable 3 Write Size 2">4</param>
-        <param name="SyncTable 3 Write Size 3">4</param>
-        <param name="SyncTable 3 Write Size 4">4</param>
-        <param name="SyncTable 3 Write Size 5">0</param>
-        <param name="SyncTable 4 Read Address 1">224</param>
-        <param name="SyncTable 4 Read Address 2">224</param>
-        <param name="SyncTable 4 Read Address 3">224</param>
-        <param name="SyncTable 4 Read Address 4">224</param>
-        <param name="SyncTable 4 Read Address 5">72</param>
-        <param name="SyncTable 4 Read Size 1">6</param>
-        <param name="SyncTable 4 Read Size 2">6</param>
-        <param name="SyncTable 4 Read Size 3">6</param>
-        <param name="SyncTable 4 Read Size 4">6</param>
-        <param name="SyncTable 4 Read Size 5">9</param>
-        <param name="SyncTable 4 Write Address 1">230</param>
-        <param name="SyncTable 4 Write Address 2">230</param>
-        <param name="SyncTable 4 Write Address 3">230</param>
-        <param name="SyncTable 4 Write Address 4">230</param>
-        <param name="SyncTable 4 Write Address 5">0</param>
-        <param name="SyncTable 4 Write Size 1">4</param>
-        <param name="SyncTable 4 Write Size 2">4</param>
-        <param name="SyncTable 4 Write Size 3">4</param>
-        <param name="SyncTable 4 Write Size 4">4</param>
-        <param name="SyncTable 4 Write Size 5">0</param>
-        <param name="SyncTable 5 Read Address 1">224</param>
-        <param name="SyncTable 5 Read Address 2">224</param>
-        <param name="SyncTable 5 Read Address 3">224</param>
-        <param name="SyncTable 5 Read Address 4">224</param>
-        <param name="SyncTable 5 Read Address 5">72</param>
-        <param name="SyncTable 5 Read Size 1">6</param>
-        <param name="SyncTable 5 Read Size 2">6</param>
-        <param name="SyncTable 5 Read Size 3">6</param>
-        <param name="SyncTable 5 Read Size 4">6</param>
-        <param name="SyncTable 5 Read Size 5">9</param>
-        <param name="SyncTable 5 Write Address 1">230</param>
-        <param name="SyncTable 5 Write Address 2">230</param>
-        <param name="SyncTable 5 Write Address 3">230</param>
-        <param name="SyncTable 5 Write Address 4">230</param>
-        <param name="SyncTable 5 Write Address 5">0</param>
-        <param name="SyncTable 5 Write Size 1">4</param>
-        <param name="SyncTable 5 Write Size 2">4</param>
-        <param name="SyncTable 5 Write Size 3">4</param>
-        <param name="SyncTable 5 Write Size 4">4</param>
-        <param name="SyncTable 5 Write Size 5">0</param>
+        <!-- <param name="Bus Watchdog">100</param> -->
       </gpio>
       <!-- Motor init: simplified - only essential params for grasp/release -->
       <!-- Finger 1 motors -->
-      <gpio name="dxl111_init">
-        <param name="type">controller</param>
-        <param name="ID">111</param>
-        <param name="Startup Configuration">2</param>
-        <param name="Operating Mode">5</param>
-        <param name="Drive Mode">13</param>
-        <param name="Bus Watchdog">100</param>
-        <param name="Profile Velocity">100</param>
-        <param name="Profile Acceleration">50</param>
-        <param name="Position P Gain">500</param>
-        <param name="Position D Gain">1000</param>
-        <param name="Homing Offset">0</param>
-        <param name="Indirect Address 1">126</param>
-        <param name="Indirect Address 2">127</param>
-        <param name="Indirect Address 3">128</param>
-        <param name="Indirect Address 4">129</param>
-        <param name="Indirect Address 5">132</param>
-        <param name="Indirect Address 6">133</param>
-        <param name="Indirect Address 7">102</param>
-        <param name="Indirect Address 8">103</param>
-        <param name="Indirect Address 9">116</param>
-        <param name="Indirect Address 10">117</param>
-      </gpio>
-      <gpio name="dxl112_init">
-        <param name="type">controller</param>
-        <param name="ID">112</param>
-        <param name="Startup Configuration">2</param>
-        <param name="Operating Mode">5</param>
-        <param name="Drive Mode">12</param>
-        <param name="Bus Watchdog">100</param>
-        <param name="Profile Velocity">100</param>
-        <param name="Profile Acceleration">50</param>
-        <param name="Position P Gain">500</param>
-        <param name="Position D Gain">1000</param>
-        <param name="Homing Offset">1024</param>
-        <param name="Indirect Address 1">126</param>
-        <param name="Indirect Address 2">127</param>
-        <param name="Indirect Address 3">128</param>
-        <param name="Indirect Address 4">129</param>
-        <param name="Indirect Address 5">132</param>
-        <param name="Indirect Address 6">133</param>
-        <param name="Indirect Address 7">102</param>
-        <param name="Indirect Address 8">103</param>
-        <param name="Indirect Address 9">116</param>
-        <param name="Indirect Address 10">117</param>
-      </gpio>
-      <gpio name="dxl113_init">
-        <param name="type">controller</param>
-        <param name="ID">113</param>
-        <param name="Startup Configuration">2</param>
-        <param name="Operating Mode">5</param>
-        <param name="Drive Mode">13</param>
-        <param name="Bus Watchdog">100</param>
-        <param name="Profile Velocity">100</param>
-        <param name="Profile Acceleration">50</param>
-        <param name="Position P Gain">500</param>
-        <param name="Position D Gain">1000</param>
-        <param name="Indirect Address 1">126</param>
-        <param name="Indirect Address 2">127</param>
-        <param name="Indirect Address 3">128</param>
-        <param name="Indirect Address 4">129</param>
-        <param name="Indirect Address 5">132</param>
-        <param name="Indirect Address 6">133</param>
-        <param name="Indirect Address 7">102</param>
-        <param name="Indirect Address 8">103</param>
-        <param name="Indirect Address 9">116</param>
-        <param name="Indirect Address 10">117</param>
-      </gpio>
-      <gpio name="dxl114_init">
-        <param name="type">controller</param>
-        <param name="ID">114</param>
-        <param name="Startup Configuration">2</param>
-        <param name="Operating Mode">5</param>
-        <param name="Drive Mode">13</param>
-        <param name="Bus Watchdog">100</param>
-        <param name="Profile Velocity">100</param>
-        <param name="Profile Acceleration">50</param>
-        <param name="Position P Gain">500</param>
-        <param name="Position D Gain">1000</param>
-        <param name="Indirect Address 1">126</param>
-        <param name="Indirect Address 2">127</param>
-        <param name="Indirect Address 3">128</param>
-        <param name="Indirect Address 4">129</param>
-        <param name="Indirect Address 5">132</param>
-        <param name="Indirect Address 6">133</param>
-        <param name="Indirect Address 7">102</param>
-        <param name="Indirect Address 8">103</param>
-        <param name="Indirect Address 9">116</param>
-        <param name="Indirect Address 10">117</param>
-      </gpio>
       <!-- Finger 2 motors (simplified - only IDs 116-119) -->
-      <gpio name="dxl116_init">
-        <param name="type">controller</param>
-        <param name="ID">116</param>
-        <param name="Startup Configuration">2</param>
-        <param name="Operating Mode">5</param>
-        <param name="Drive Mode">12</param>
-        <param name="Bus Watchdog">100</param>
-        <param name="Profile Velocity">100</param>
-        <param name="Profile Acceleration">50</param>
-        <param name="Position P Gain">500</param>
-        <param name="Position D Gain">1000</param>
-        <param name="Indirect Address 1">126</param>
-        <param name="Indirect Address 2">127</param>
-        <param name="Indirect Address 3">128</param>
-        <param name="Indirect Address 4">129</param>
-        <param name="Indirect Address 5">132</param>
-        <param name="Indirect Address 6">133</param>
-        <param name="Indirect Address 7">102</param>
-        <param name="Indirect Address 8">103</param>
-        <param name="Indirect Address 9">116</param>
-        <param name="Indirect Address 10">117</param>
-      </gpio>
-      <gpio name="dxl117_init">
-        <param name="type">controller</param>
-        <param name="ID">117</param>
-        <param name="Startup Configuration">2</param>
-        <param name="Operating Mode">5</param>
-        <param name="Drive Mode">12</param>
-        <param name="Bus Watchdog">100</param>
-        <param name="Profile Velocity">100</param>
-        <param name="Profile Acceleration">50</param>
-        <param name="Position P Gain">500</param>
-        <param name="Position D Gain">1000</param>
-        <param name="Homing Offset">1024</param>
-        <param name="Indirect Address 1">126</param>
-        <param name="Indirect Address 2">127</param>
-        <param name="Indirect Address 3">128</param>
-        <param name="Indirect Address 4">129</param>
-        <param name="Indirect Address 5">132</param>
-        <param name="Indirect Address 6">133</param>
-        <param name="Indirect Address 7">102</param>
-        <param name="Indirect Address 8">103</param>
-        <param name="Indirect Address 9">116</param>
-        <param name="Indirect Address 10">117</param>
-      </gpio>
-      <gpio name="dxl118_init">
-        <param name="type">controller</param>
-        <param name="ID">118</param>
-        <param name="Startup Configuration">2</param>
-        <param name="Operating Mode">5</param>
-        <param name="Drive Mode">12</param>
-        <param name="Bus Watchdog">100</param>
-        <param name="Profile Velocity">100</param>
-        <param name="Profile Acceleration">50</param>
-        <param name="Position P Gain">500</param>
-        <param name="Position D Gain">1000</param>
-        <param name="Indirect Address 1">126</param>
-        <param name="Indirect Address 2">127</param>
-        <param name="Indirect Address 3">128</param>
-        <param name="Indirect Address 4">129</param>
-        <param name="Indirect Address 5">132</param>
-        <param name="Indirect Address 6">133</param>
-        <param name="Indirect Address 7">102</param>
-        <param name="Indirect Address 8">103</param>
-        <param name="Indirect Address 9">116</param>
-        <param name="Indirect Address 10">117</param>
-      </gpio>
-      <gpio name="dxl119_init">
-        <param name="type">controller</param>
-        <param name="ID">119</param>
-        <param name="Startup Configuration">2</param>
-        <param name="Operating Mode">5</param>
-        <param name="Drive Mode">12</param>
-        <param name="Bus Watchdog">100</param>
-        <param name="Profile Velocity">100</param>
-        <param name="Profile Acceleration">50</param>
-        <param name="Position P Gain">500</param>
-        <param name="Position D Gain">1000</param>
-        <param name="Indirect Address 1">126</param>
-        <param name="Indirect Address 2">127</param>
-        <param name="Indirect Address 3">128</param>
-        <param name="Indirect Address 4">129</param>
-        <param name="Indirect Address 5">132</param>
-        <param name="Indirect Address 6">133</param>
-        <param name="Indirect Address 7">102</param>
-        <param name="Indirect Address 8">103</param>
-        <param name="Indirect Address 9">116</param>
-        <param name="Indirect Address 10">117</param>
-      </gpio>
       <!-- Finger 3 motors -->
-      <gpio name="dxl121_init">
-        <param name="type">controller</param>
-        <param name="ID">121</param>
-        <param name="Startup Configuration">2</param>
-        <param name="Operating Mode">5</param>
-        <param name="Drive Mode">12</param>
-        <param name="Bus Watchdog">100</param>
-        <param name="Profile Velocity">100</param>
-        <param name="Profile Acceleration">50</param>
-        <param name="Position P Gain">500</param>
-        <param name="Position D Gain">1000</param>
-        <param name="Homing Offset">-171</param>
-        <param name="Indirect Address 1">126</param>
-        <param name="Indirect Address 2">127</param>
-        <param name="Indirect Address 3">128</param>
-        <param name="Indirect Address 4">129</param>
-        <param name="Indirect Address 5">132</param>
-        <param name="Indirect Address 6">133</param>
-        <param name="Indirect Address 7">102</param>
-        <param name="Indirect Address 8">103</param>
-        <param name="Indirect Address 9">116</param>
-        <param name="Indirect Address 10">117</param>
-      </gpio>
-      <gpio name="dxl122_init">
-        <param name="type">controller</param>
-        <param name="ID">122</param>
-        <param name="Startup Configuration">2</param>
-        <param name="Operating Mode">5</param>
-        <param name="Drive Mode">12</param>
-        <param name="Bus Watchdog">100</param>
-        <param name="Profile Velocity">100</param>
-        <param name="Profile Acceleration">50</param>
-        <param name="Position P Gain">500</param>
-        <param name="Position D Gain">1000</param>
-        <param name="Homing Offset">1024</param>
-        <param name="Indirect Address 1">126</param>
-        <param name="Indirect Address 2">127</param>
-        <param name="Indirect Address 3">128</param>
-        <param name="Indirect Address 4">129</param>
-        <param name="Indirect Address 5">132</param>
-        <param name="Indirect Address 6">133</param>
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
File: open_manipulator_description/urdf/omy_f3m/omy_end_hx5_right_standalone.urdf.xacro (robot description, xacro)
@@ -11,4 +11,6 @@
   <xacro:arg name="mock_sensor_commands" default="false" />
   <xacro:arg name="port_name"            default="/dev/ttyAMA4" />
+  <xacro:arg name="dynamixel_model_folder" default="/param/dxl_model" />
+  <xacro:arg name="configure_hx5_synctable" default="false" />
   <!-- HX5 D20 right hand visual/collision links -->
   <xacro:include filename="$(find open_manipulator_description)/urdf/hx5_d20_rev2/hx5_d20_right.urdf.xacro" />
@@ -29,4 +31,6 @@
     prefix="$(arg prefix)"
     port_name="$(arg port_name)"
+    dynamixel_model_folder="$(arg dynamixel_model_folder)"
+    configure_hx5_synctable="$(arg configure_hx5_synctable)"
     use_sim="$(arg use_sim)"
     use_mock_hardware="$(arg use_mock_hardware)"
