Commit message: synctable_watchdog update

File: open_manipulator_description/ros2_control/omy_f3m_end_unit_hx5_right.ros2_control.xacro (robot description, xacro)
@@ -3,14 +3,25 @@
   omy_f3m_end_unit_hx5_right.ros2_control.xacro
   HX5 right hand driven through OMY END (ID 210) SyncTable relay.
-  Simplified version with preset grasp/release motions controlled by trigger.
-  Preset trigger mapping:
-    - trigger closed (t=1.0):  hand fully grasped
-    - trigger open   (t=0.0):  hand fully relaxed
-    - trigger mid    (0<t<1):  blended between grasp and release
-  Joint naming: finger_r_joint1..20 (instead of finger_l_joint)
+  Based on the robotis_hand pattern (hx5_d20_right.ros2_control.xacro):
+  - Reboot the controller, set Table Sync Enable=0
+  - Init each motor (Operating Mode, Drive Mode, gains, Indirect Address …)
+  - Re-set Table Sync Enable=1 with a dummy controller gpio at the end
+  Init order (xacro element order = InitItem execution order):
+    [1] omy_end_pre   (ID 210): Reboot=1, SyncTable Enable=0,
+                                SyncTable Enable HX5=0
+    [2] hand_r_controller (ID 110): Reboot=1, Table Sync Enable=0,
+                                Bus Watchdog, SyncTable 1-5 IDs / Read Addr /
+                                Read Size / Write Addr / Write Size
+    [3] dxl111_init … dxl134_init (ID 111-134): Reboot, Operating Mode=5,
+                                Drive Mode, gains, Indirect Address, Homing Offset
+    [4] hand_r_controller_dummy (ID 110): Table Sync Enable=1
+    [5] virtual_dxl  (dxl111…dxl134)
+        comm_id=210 (relayed via OMY END)
+    [6] omy_end_init  (ID 210): placeholder for additional OMY END RAM init
+    [7] launch file   (ID 210): SyncTable Enable=1, SyncTable Enable HX5=1
 -->
 <robot xmlns:xacro="http://www.ros.org/wiki/xacro">
-  <xacro:macro name="omy_f3m_end_unit_hx5_right_system" params="name prefix port_name:=^|/dev/ttyAMA4 dynamixel_model_folder:=^|/param/dxl_model configure_hx5_synctable:=^|false use_sim:=^|false use_mock_hardware:=^|false mock_sensor_commands:=^|false">
-    <ros2_control name="${name}" type="system" is_async="true">
+  <xacro:macro name="omy_f3m_end_unit_hx5_right_system" params="name prefix port_name:=^|/dev/ttyAMA4 dynamixel_model_folder:=^|/param/dxl_model configure_hx5_synctable:=^|false enable_hx5_motor_torque:=^|false use_sim:=^|false use_mock_hardware:=^|false mock_sensor_commands:=^|false">
+    <ros2_control name="${name}" type="system">
       <xacro:if value="$(arg use_sim)">
         <hardware>
@@ -29,4 +40,8 @@
             <param name="port_name">${port_name}</param>
             <param name="baud_rate">4000000</param>
+            <!-- Match omy_f3m_end_unit.ros2_control.xacro (500 ms) so initial
+                 ping/InitItem failures fall through quickly and the 10-retry
+                 loop in InitDxlComm can recover, instead of stalling for 5 s
+                 per attempt. -->
             <param name="error_timeout_ms">500</param>
             <param name="dynamixel_model_folder">${dynamixel_model_folder}</param>
@@ -42,5 +57,7 @@
         </hardware>
       </xacro:unless>
-      <!-- Joint/Sensor interface declarations -->
+      <!-- ════════════════════════════════════════════════════════════════════
+           Joint / Sensor interface declarations (no InitItem)
+           ════════════════════════════════════════════════════════════════════ -->
       <!-- Finger 1 joints -->
       <joint name="${prefix}finger_r_joint1">
@@ -72,4 +89,15 @@
         <state_interface name="effort"/>
       </joint>
+      <sensor name="${prefix}finger_r_sensor1">
+        <state_interface name="Present Pressure 1"/>
+        <state_interface name="Present Pressure 2"/>
+        <state_interface name="Present Pressure 3"/>
+        <state_interface name="Present Pressure 4"/>
+        <state_interface name="Present Pressure 5"/>
+        <state_interface name="Present Pressure 6"/>
+        <state_interface name="Present Pressure 7"/>
+        <state_interface name="Present Pressure 8"/>
+        <state_interface name="Present Pressure 9"/>
+      </sensor>
       <!-- Finger 2 joints -->
       <joint name="${prefix}finger_r_joint5">
@@ -101,4 +129,15 @@
         <state_interface name="effort"/>
       </joint>
+      <sensor name="${prefix}finger_r_sensor2">
+        <state_interface name="Present Pressure 1"/>
+        <state_interface name="Present Pressure 2"/>
+        <state_interface name="Present Pressure 3"/>
+        <state_interface name="Present Pressure 4"/>
+        <state_interface name="Present Pressure 5"/>
+        <state_interface name="Present Pressure 6"/>
+        <state_interface name="Present Pressure 7"/>
+        <state_interface name="Present Pressure 8"/>
+        <state_interface name="Present Pressure 9"/>
+      </sensor>
       <!-- Finger 3 joints -->
       <joint name="${prefix}finger_r_joint9">
@@ -130,4 +169,15 @@
         <state_interface name="effort"/>
       </joint>
+      <sensor name="${prefix}finger_r_sensor3">
+        <state_interface name="Present Pressure 1"/>
+        <state_interface name="Present Pressure 2"/>
+        <state_interface name="Present Pressure 3"/>
+        <state_interface name="Present Pressure 4"/>
+        <state_interface name="Present Pressure 5"/>
+        <state_interface name="Present Pressure 6"/>
+        <state_interface name="Present Pressure 7"/>
+        <state_interface name="Present Pressure 8"/>
+        <state_interface name="Present Pressure 9"/>
+      </sensor>
       <!-- Finger 4 joints -->
       <joint name="${prefix}finger_r_joint13">
@@ -159,4 +209,15 @@
         <state_interface name="effort"/>
       </joint>
+      <sensor name="${prefix}finger_r_sensor4">
+        <state_interface name="Present Pressure 1"/>
+        <state_interface name="Present Pressure 2"/>
+        <state_interface name="Present Pressure 3"/>
+        <state_interface name="Present Pressure 4"/>
+        <state_interface name="Present Pressure 5"/>
+        <state_interface name="Present Pressure 6"/>
+        <state_interface name="Present Pressure 7"/>
+        <state_interface name="Present Pressure 8"/>
+        <state_interface name="Present Pressure 9"/>
+      </sensor>
       <!-- Finger 5 joints -->
       <joint name="${prefix}finger_r_joint17">
@@ -188,23 +249,51 @@
         <state_interface name="effort"/>
       </joint>
-      <sensor name="${prefix}finger_r_sensor1"><state_interface name="Present Pressure 5"/></sensor>
-      <sensor name="${prefix}finger_r_sensor2"><state_interface name="Present Pressure 5"/></sensor>
-      <sensor name="${prefix}finger_r_sensor3"><state_interface name="Present Pressure 5"/></sensor>
-      <sensor name="${prefix}finger_r_sensor4"><state_interface name="Present Pressure 5"/></sensor>
-      <sensor name="${prefix}finger_r_sensor5"><state_interface name="Present Pressure 5"/></sensor>
-      <!-- OMY END pre-init (disable SyncTable) -->
+      <sensor name="${prefix}finger_r_sensor5">
+        <state_interface name="Present Pressure 1"/>
+        <state_interface name="Present Pressure 2"/>
+        <state_interface name="Present Pressure 3"/>
+        <state_interface name="Present Pressure 4"/>
+        <state_interface name="Present Pressure 5"/>
+        <state_interface name="Present Pressure 6"/>
+        <state_interface name="Present Pressure 7"/>
+        <state_interface name="Present Pressure 8"/>
+        <state_interface name="Present Pressure 9"/>
+      </sensor>
+      <!-- ════════════════════════════════════════════════════════════════════
+           [Step 1] OMY END (ID 210) — disable SyncTable, configure Tool Bus,
+                    reboot.
+                    Tool Bus packet forwarding (Tool Analog Enable=0, Tool
+                    Baud Rate=8 (4 Mbps), Tool Protocol=0, Tool ID=110) is
+                    REQUIRED so that motor init packets to ID 110-134 are
+                    forwarded reliably while SyncTable is OFF. Without these
+                    the pass-through mode is intermittent and InitItem writes
+                    to ID:110 randomly time out after 10-15 packets.
+           ════════════════════════════════════════════════════════════════════ -->
+      <!--
+           Reboot=1 INTENTIONALLY OMITTED for ID 210 / 110.
+           Reason: dynamixel_sdk Protocol2PacketHandler::reboot() allocates
+           a fixed 11-byte stack rxpacket and trusts the LENGTH field of
+           the response to set wait_length. Right after openPort + 4 Mbps
+           setBaudRate, the RP1 UART RX FIFO holds residual bytes / framing
+           noise / RS-485 self-echo, which is not flushed by the SDK
+           between TX and RX (clearPort is only called once at txPacket
+           start). The first reboot to ID 210 deterministically forms a
+           "fake header" pattern, the LENGTH byte slips into a value
+           5..1024, wait_length is bumped past 11, and the next readPort
+           writes past the 11-byte buffer into the stack guard page →
+           SIGSEGV (Invalid permissions for mapped object 0x7ffe…).
+           Letting the first transaction be a ping (rxpacket[14], retried
+           by InitDxlComm) instead avoids the deterministic crash.
+           See log9.txt for the exact stack trace.
+      -->
       <gpio name="omy_end_pre">
-        <state_interface name="Button Status"/>
         <param name="type">controller</param>
         <param name="ID">210</param>
-        <param name="Baud Rate (Bus)">6</param>
         <param name="SyncTable Enable">0</param>
+        <param name="SyncTable Enable HX5">0</param>
         <param name="Tool Analog Enable">0</param>
         <param name="Tool Baud Rate">8</param>
         <param name="Tool Protocol">0</param>
         <param name="Tool ID">110</param>
-        <param name="R LED">200</param>
-        <param name="G LED">200</param>
-        <param name="B LED">120</param>
         <param name="SyncTable Read Address">634</param>
         <param name="SyncTable Read Size">125</param>
@@ -212,290 +301,684 @@
         <param name="SyncTable Write Size">80</param>
       </gpio>
-      <!-- HX5 hub (ID 110) init + SyncTable config -->
+      <xacro:if value="${configure_hx5_synctable}">
+      <!-- ════════════════════════════════════════════════════════════════════
+           [Step 2] HX5 hub (ID 110) — Reboot + Table Sync Enable=0 + bulk
+                    SyncTable configuration.
+                    Mirrors hx5_d20_right.ros2_control.xacro hand_r_controller.
+                    NOTE: Splitting this into a "pre" gpio block (with just
+                    Table Sync Enable=0) plus a "main" gpio block (with the
+                    bulk SyncTable params) caused the hand process to hang
+                    silently after the first InitItem; ros2_control appears
+                    to handle two gpios with the same ID poorly. So we keep
+                    everything in one block and rely on the inter-packet
+                    sleep added inside dynamixel_hardware_interface::WriteItem
+                    to keep the OMY END Tool Bus buffer from overrunning.
+           ════════════════════════════════════════════════════════════════════ -->
       <gpio name="hand_r_controller">
         <param name="type">controller</param>
         <param name="ID">110</param>
-        <!-- <param name="Bus Watchdog">100</param> -->
-      </gpio>
-      <!-- Motor init: simplified - only essential params for grasp/release -->
-      <!-- Finger 1 motors -->
-      <!-- Finger 2 motors (simplified - only IDs 116-119) -->
-      <!-- Finger 3 motors -->
-      <!-- Finger 4 motors -->
-      <!-- Finger 5 motors -->
-      <!-- HX5 hub - enable SyncTable -->
+        <!-- Reboot=1 OMITTED following the omy_ai pattern
+             (omy_f3m_position.ros2_control.xacro and
+              omy_f3m_end_unit.ros2_control.xacro both run on RP1 UART
+              direct at 4-6.25 Mbps with NO Reboot=1 in any gpio block).
+             Reasoning: the SDK's Protocol2PacketHandler::reboot() uses an
+             11-byte stack rxpacket buffer that overflows when the
+             baudrate-transition self-echo on RP1 UART is mis-parsed as a
+             status header with a non-trivial LENGTH field → SIGSEGV.
+             Letting InitDxlComm's ping (14-byte buffer, 10× retry with
+             1 s sleep) be the first transaction lets the line settle
+             naturally. InitItem then overwrites any dirty motor state. -->
+        <param name="Table Sync Enable">0</param>
+        <param name="Bus Watchdog">100</param>
+        <param name="SyncTable 1 ID 1">111</param>
+        <param name="SyncTable 1 ID 2">112</param>
+        <param name="SyncTable 1 ID 3">113</param>
+        <param name="SyncTable 1 ID 4">114</param>
+        <param name="SyncTable 1 ID 5">115</param>
+        <param name="SyncTable 2 ID 1">116</param>
+        <param name="SyncTable 2 ID 2">117</param>
+        <param name="SyncTable 2 ID 3">118</param>
+        <param name="SyncTable 2 ID 4">119</param>
+        <param name="SyncTable 2 ID 5">120</param>
+        <param name="SyncTable 3 ID 1">121</param>
+        <param name="SyncTable 3 ID 2">122</param>
+        <param name="SyncTable 3 ID 3">123</param>
+        <param name="SyncTable 3 ID 4">124</param>
+        <param name="SyncTable 3 ID 5">125</param>
+        <param name="SyncTable 4 ID 1">126</param>
+        <param name="SyncTable 4 ID 2">127</param>
+        <param name="SyncTable 4 ID 3">128</param>
+        <param name="SyncTable 4 ID 4">129</param>
+        <param name="SyncTable 4 ID 5">130</param>
+        <param name="SyncTable 5 ID 1">131</param>
+        <param name="SyncTable 5 ID 2">132</param>
+        <param name="SyncTable 5 ID 3">133</param>
+        <param name="SyncTable 5 ID 4">134</param>
+        <param name="SyncTable 5 ID 5">135</param>
+        <param name="SyncTable 1 Read Address 1">224</param>
+        <param name="SyncTable 1 Read Address 2">224</param>
+        <param name="SyncTable 1 Read Address 3">224</param>
+        <param name="SyncTable 1 Read Address 4">224</param>
+        <param name="SyncTable 1 Read Address 5">72</param>
+        <param name="SyncTable 1 Read Size 1">6</param>
+        <param name="SyncTable 1 Read Size 2">6</param>
+        <param name="SyncTable 1 Read Size 3">6</param>
+        <param name="SyncTable 1 Read Size 4">6</param>
+        <param name="SyncTable 1 Read Size 5">9</param>
+        <param name="SyncTable 1 Write Address 1">230</param>
+        <param name="SyncTable 1 Write Address 2">230</param>
+        <param name="SyncTable 1 Write Address 3">230</param>
+        <param name="SyncTable 1 Write Address 4">230</param>
+        <param name="SyncTable 1 Write Address 5">0</param>
+        <param name="SyncTable 1 Write Size 1">4</param>
+        <param name="SyncTable 1 Write Size 2">4</param>
+        <param name="SyncTable 1 Write Size 3">4</param>
+        <param name="SyncTable 1 Write Size 4">4</param>
+        <param name="SyncTable 1 Write Size 5">0</param>
+        <param name="SyncTable 2 Read Address 1">224</param>
+        <param name="SyncTable 2 Read Address 2">224</param>
+        <param name="SyncTable 2 Read Address 3">224</param>
+        <param name="SyncTable 2 Read Address 4">224</param>
+        <param name="SyncTable 2 Read Address 5">72</param>
+        <param name="SyncTable 2 Read Size 1">6</param>
+        <param name="SyncTable 2 Read Size 2">6</param>
+        <param name="SyncTable 2 Read Size 3">6</param>
+        <param name="SyncTable 2 Read Size 4">6</param>
+        <param name="SyncTable 2 Read Size 5">9</param>
+        <param name="SyncTable 2 Write Address 1">230</param>
+        <param name="SyncTable 2 Write Address 2">230</param>
+        <param name="SyncTable 2 Write Address 3">230</param>
+        <param name="SyncTable 2 Write Address 4">230</param>
+        <param name="SyncTable 2 Write Address 5">0</param>
+        <param name="SyncTable 2 Write Size 1">4</param>
+        <param name="SyncTable 2 Write Size 2">4</param>
+        <param name="SyncTable 2 Write Size 3">4</param>
+        <param name="SyncTable 2 Write Size 4">4</param>
+        <param name="SyncTable 2 Write Size 5">0</param>
+        <param name="SyncTable 3 Read Address 1">224</param>
+        <param name="SyncTable 3 Read Address 2">224</param>
+        <param name="SyncTable 3 Read Address 3">224</param>
+        <param name="SyncTable 3 Read Address 4">224</param>
+        <param name="SyncTable 3 Read Address 5">72</param>
+        <param name="SyncTable 3 Read Size 1">6</param>
+        <param name="SyncTable 3 Read Size 2">6</param>
+        <param name="SyncTable 3 Read Size 3">6</param>
+        <param name="SyncTable 3 Read Size 4">6</param>
+        <param name="SyncTable 3 Read Size 5">9</param>
+        <param name="SyncTable 3 Write Address 1">230</param>
+        <param name="SyncTable 3 Write Address 2">230</param>
+        <param name="SyncTable 3 Write Address 3">230</param>
+        <param name="SyncTable 3 Write Address 4">230</param>
+        <param name="SyncTable 3 Write Address 5">0</param>
+        <param name="SyncTable 3 Write Size 1">4</param>
+        <param name="SyncTable 3 Write Size 2">4</param>
+        <param name="SyncTable 3 Write Size 3">4</param>
+        <param name="SyncTable 3 Write Size 4">4</param>
+        <param name="SyncTable 3 Write Size 5">0</param>
+        <param name="SyncTable 4 Read Address 1">224</param>
+        <param name="SyncTable 4 Read Address 2">224</param>
+        <param name="SyncTable 4 Read Address 3">224</param>
+        <param name="SyncTable 4 Read Address 4">224</param>
+        <param name="SyncTable 4 Read Address 5">72</param>
+        <param name="SyncTable 4 Read Size 1">6</param>
+        <param name="SyncTable 4 Read Size 2">6</param>
+        <param name="SyncTable 4 Read Size 3">6</param>
+        <param name="SyncTable 4 Read Size 4">6</param>
+        <param name="SyncTable 4 Read Size 5">9</param>
+        <param name="SyncTable 4 Write Address 1">230</param>
+        <param name="SyncTable 4 Write Address 2">230</param>
+        <param name="SyncTable 4 Write Address 3">230</param>
+        <param name="SyncTable 4 Write Address 4">230</param>
+        <param name="SyncTable 4 Write Address 5">0</param>
+        <param name="SyncTable 4 Write Size 1">4</param>
+        <param name="SyncTable 4 Write Size 2">4</param>
+        <param name="SyncTable 4 Write Size 3">4</param>
+        <param name="SyncTable 4 Write Size 4">4</param>
+        <param name="SyncTable 4 Write Size 5">0</param>
+        <param name="SyncTable 5 Read Address 1">224</param>
+        <param name="SyncTable 5 Read Address 2">224</param>
+        <param name="SyncTable 5 Read Address 3">224</param>
+        <param name="SyncTable 5 Read Address 4">224</param>
+        <param name="SyncTable 5 Read Address 5">72</param>
+        <param name="SyncTable 5 Read Size 1">6</param>
+        <param name="SyncTable 5 Read Size 2">6</param>
+        <param name="SyncTable 5 Read Size 3">6</param>
+        <param name="SyncTable 5 Read Size 4">6</param>
+        <param name="SyncTable 5 Read Size 5">9</param>
+        <param name="SyncTable 5 Write Address 1">230</param>
+        <param name="SyncTable 5 Write Address 2">230</param>
+        <param name="SyncTable 5 Write Address 3">230</param>
+        <param name="SyncTable 5 Write Address 4">230</param>
+        <param name="SyncTable 5 Write Address 5">0</param>
+        <param name="SyncTable 5 Write Size 1">4</param>
+        <param name="SyncTable 5 Write Size 2">4</param>
+        <param name="SyncTable 5 Write Size 3">4</param>
+        <param name="SyncTable 5 Write Size 4">4</param>
+        <param name="SyncTable 5 Write Size 5">0</param>
+      </gpio>
+      <!-- ════════════════════════════════════════════════════════════════════
+           [Step 3] HX5 motors (ID 111-134) init
+                    Operating Mode=5  (Current-based Position Control)
+                    Drive Mode=12 or 13, Indirect Address 1-10 mapping etc.
+                    Mirrors hx5_d20_right.ros2_control.xacro dxlNNN_init blocks.
+                    NOTE: Reboot=1 OMITTED from every motor init block,
+                    following the omy_ai pattern (see header comment on
+                    omy_end_pre / hand_r_controller for the SDK
+                    rxpacket[11] stack overflow rationale). InitItem
+                    overwrites stale motor state regardless of reboot.
+           ════════════════════════════════════════════════════════════════════ -->
+      <gpio name="dxl111_init">
+        <param name="type">controller</param>
+        <param name="ID">111</param>
+        <param name="Startup Configuration">2</param>
+        <param name="Operating Mode">5</param>
+        <param name="Drive Mode">13</param>
+        <param name="Bus Watchdog">100</param>
+        <param name="Profile Velocity">100</param>
+        <param name="Profile Acceleration">50</param>
+        <param name="Position P Gain">500</param>
+        <param name="Position D Gain">1000</param>
+        <param name="Homing Offset">0</param>
+        <param name="Indirect Address 1">126</param>
+        <param name="Indirect Address 2">127</param>
+        <param name="Indirect Address 3">128</param>
+        <param name="Indirect Address 4">129</param>
+        <param name="Indirect Address 5">132</param>
+        <param name="Indirect Address 6">133</param>
+        <param name="Indirect Address 7">102</param>
+        <param name="Indirect Address 8">103</param>
+        <param name="Indirect Address 9">116</param>
+        <param name="Indirect Address 10">117</param>
+      </gpio>
+      <gpio name="dxl112_init">
+        <param name="type">controller</param>
+        <param name="ID">112</param>
+        <param name="Startup Configuration">2</param>
+        <param name="Operating Mode">5</param>
+        <param name="Drive Mode">12</param>
+        <param name="Bus Watchdog">100</param>
+        <param name="Profile Velocity">100</param>
+        <param name="Profile Acceleration">50</param>
+        <param name="Position P Gain">500</param>
+        <param name="Position D Gain">1000</param>
+        <param name="Homing Offset">1024</param>
+        <param name="Indirect Address 1">126</param>
+        <param name="Indirect Address 2">127</param>
+        <param name="Indirect Address 3">128</param>
+        <param name="Indirect Address 4">129</param>
+        <param name="Indirect Address 5">132</param>
+        <param name="Indirect Address 6">133</param>
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