Commit message: synctable_watchdog update

File: open_manipulator_description/urdf/omy_f3m/omy_end_hx5_right_standalone.urdf.xacro (robot description, xacro)
@@ -13,4 +13,5 @@
   <xacro:arg name="dynamixel_model_folder" default="/param/dxl_model" />
   <xacro:arg name="configure_hx5_synctable" default="false" />
+  <xacro:arg name="enable_hx5_motor_torque" default="false" />
   <!-- HX5 D20 right hand visual/collision links -->
   <xacro:include filename="$(find open_manipulator_description)/urdf/hx5_d20_rev2/hx5_d20_right.urdf.xacro" />
@@ -33,4 +34,5 @@
     dynamixel_model_folder="$(arg dynamixel_model_folder)"
     configure_hx5_synctable="$(arg configure_hx5_synctable)"
+    enable_hx5_motor_torque="$(arg enable_hx5_motor_torque)"
     use_sim="$(arg use_sim)"
     use_mock_hardware="$(arg use_mock_hardware)"

File: open_manipulator_description/urdf/omy_f3m/omy_f3m_arm_only.urdf.xacro (robot description, xacro)
@@ -7,5 +7,5 @@
   (OMY END + P12 gripper combo on /dev/ttyAMA4, ID 210). When the
   F3M arm is run together with a separately-loaded HX5 hand (which owns
-  OMY END through OMYF3MEndUnitHX5LeftSystem in its own controller_manager),
+  OMY END through an HX5 end-unit system in its own controller_manager),
   two ros2_control hardware components fight for the same OMY END device.
   This causes endless [ID:210] COMM_ERROR : There is no status packet!
