Commit message: test leader
Signed-off-by: Hyunwoo Nam <nhw@robotis.com>

File: open_manipulator_description/ros2_control/omy_l100_current.ros2_control.xacro (robot description, xacro)
@@ -21,6 +21,6 @@
             <param name="error_timeout_ms">500</param>
             <param name="dynamixel_model_folder">/param/dxl_model</param>
-            <param name="number_of_joints">7</param>
-            <param name="number_of_transmissions">7</param>
+            <param name="number_of_joints">6</param>
+            <param name="number_of_transmissions">6</param>
             <param name="disable_torque_at_init">true</param>
             <param name="dynamixel_state_pub_msg_name">dynamixel_hardware_interface/dxl_state</param>
@@ -68,10 +68,10 @@
         <state_interface name="effort"/>
       </joint>
-      <joint name="${prefix}rh_r1_joint">
+      <!-- <joint name="${prefix}rh_r1_joint">
         <command_interface name="effort"/>
         <state_interface name="position"/>
         <state_interface name="velocity"/>
         <state_interface name="effort"/>
-      </joint>
+      </joint> -->
       <gpio name="dxl1">
         <param name="type">dxl</param>
@@ -146,5 +146,5 @@
         <param name="Baud Rate">6</param>
       </gpio>
-      <gpio name="dxl7">
+      <!-- <gpio name="dxl7">
         <param name="type">dxl</param>
         <param name="ID">7</param>
@@ -157,5 +157,5 @@
         <param name="Return Delay Time">0</param>
         <param name="Baud Rate">6</param>
-      </gpio>
+      </gpio> -->
     </ros2_control>
   </xacro:macro>

File: open_manipulator_description/ros2_control/omy_l100_position.ros2_control.xacro (robot description, xacro)
@@ -21,6 +21,6 @@
             <param name="error_timeout_ms">500</param>
             <param name="dynamixel_model_folder">/param/dxl_model</param>
-            <param name="number_of_joints">7</param>
-            <param name="number_of_transmissions">7</param>
+            <param name="number_of_joints">6</param>
+            <param name="number_of_transmissions">6</param>
             <param name="disable_torque_at_init">true</param>
             <param name="dynamixel_state_pub_msg_name">dynamixel_hardware_interface/dxl_state</param>
@@ -68,10 +68,10 @@
         <state_interface name="effort"/>
       </joint>
-      <joint name="${prefix}rh_r1_joint">
+      <!-- <joint name="${prefix}rh_r1_joint">
         <command_interface name="position"/>
         <state_interface name="position"/>
         <state_interface name="velocity"/>
         <state_interface name="effort"/>
-      </joint>
+      </joint> -->
       <gpio name="dxl1">
         <param name="type">dxl</param>
@@ -170,5 +170,5 @@
         <param name="Position D Gain">200</param>
       </gpio>
-      <gpio name="dxl7">
+      <!-- <gpio name="dxl7">
         <param name="type">dxl</param>
         <param name="ID">7</param>
@@ -185,5 +185,5 @@
         <param name="Position I Gain">0</param>
         <param name="Position D Gain">200</param>
-      </gpio>
+      </gpio> -->
     </ros2_control>
   </xacro:macro>

File: open_manipulator_description/urdf/omy_l100/omy_l100_arm.urdf.xacro (robot description, xacro)
@@ -199,5 +199,5 @@
          </inertial>
       </link>
-      <joint name="rh_r1_joint" type="revolute">
+      <joint name="rh_r1_joint" type="fixed">
          <parent link="${prefix}link6" />
          <child link="${prefix}link7" />

Commit message: Update hardware controller configuration for right-hand manipulation and add new mesh files
- Changed controller names and parameters in `hardware_controller_manager.yaml` and `initial_positions.yaml` to reflect right-hand configuration.
- Updated launch file to initialize right-hand controllers and adjusted the `init_position` argument.
- Added new STL mesh files for the right-hand components.
- Introduced a new ROS 2 control configuration for the right-hand system in `omy_f3m_hx5_right_end.ros2_control.xacro`.
- Updated URDF files to include the right-hand model and its components.

File: open_manipulator_description/ros2_control/omy_l100_current.ros2_control.xacro (robot description, xacro)
@@ -21,6 +21,6 @@
             <param name="error_timeout_ms">500</param>
             <param name="dynamixel_model_folder">/param/dxl_model</param>
-            <param name="number_of_joints">6</param>
-            <param name="number_of_transmissions">6</param>
+            <param name="number_of_joints">7</param>
+            <param name="number_of_transmissions">7</param>
             <param name="disable_torque_at_init">true</param>
             <param name="dynamixel_state_pub_msg_name">dynamixel_hardware_interface/dxl_state</param>
@@ -68,10 +68,10 @@
         <state_interface name="effort"/>
       </joint>
-      <!-- <joint name="${prefix}rh_r1_joint">
+      <joint name="${prefix}rh_r1_joint">
         <command_interface name="effort"/>
         <state_interface name="position"/>
         <state_interface name="velocity"/>
         <state_interface name="effort"/>
-      </joint> -->
+      </joint>
       <gpio name="dxl1">
         <param name="type">dxl</param>
@@ -146,5 +146,5 @@
         <param name="Baud Rate">6</param>
       </gpio>
-      <!-- <gpio name="dxl7">
+      <gpio name="dxl7">
         <param name="type">dxl</param>
         <param name="ID">7</param>
@@ -157,5 +157,5 @@
         <param name="Return Delay Time">0</param>
         <param name="Baud Rate">6</param>
-      </gpio> -->
+      </gpio>
     </ros2_control>
   </xacro:macro>

File: open_manipulator_description/urdf/omy_f3m/omy_f3m_hx5.urdf.xacro (robot description, xacro)
@@ -11,8 +11,8 @@
   <!-- <xacro:include filename="$(find open_manipulator_description)/urdf/omy_f3m/rh_p12_rn_a.urdf.xacro" /> -->
   <!-- <xacro:include filename="$(find open_manipulator_description)/gazebo/rh_p12_rn_a.gazebo.xacro" /> -->
-  <xacro:include filename="$(find open_manipulator_description)/urdf/omy_f3m/hx5_d20_left.urdf.xacro" />
+  <xacro:include filename="$(find open_manipulator_description)/urdf/omy_f3m/hx5_d20_right.urdf.xacro" />
   <xacro:include filename="$(find open_manipulator_description)/ros2_control/$(arg ros2_control_type).ros2_control.xacro" />
-  <!-- <xacro:include filename="$(find open_manipulator_description)/ros2_control/omy_f3m_end_unit.ros2_control.xacro" /> -->
-  <xacro:include filename="$(find open_manipulator_description)/ros2_control/omy_f3m_hx5.ros2_control.xacro" />
+  <!-- End Unit compatibility ID 210 and downstream right Hand ID 110 share ttyAMA4. -->
+  <xacro:include filename="$(find open_manipulator_description)/ros2_control/omy_f3m_hx5_right_end.ros2_control.xacro" />
   <link name="world"/>
   <joint name="$(arg prefix)world_fixed" type="fixed">
@@ -27,8 +27,11 @@
     <child link="$(arg prefix)rh_p12_rn_base"/>
   </joint> -->
-  <xacro:hx5_d20_left parent="$(arg prefix)end_effector_flange_link" prefix="$(arg prefix)">
+  <joint name="$(arg prefix)hx5_d20_right_fixed" type="fixed">
+    <parent link="$(arg prefix)end_effector_flange_link"/>
+    <child link="$(arg prefix)hx5_d20_right_base"/>
     <origin xyz="0 0 0" rpy="0 1.5708 -1.5708"/>
-  </xacro:hx5_d20_left>
-  <!-- <joint name="$(arg prefix)end_effector_joint" type="fixed">
+  </joint>
+  <xacro:hx5_d20_right prefix="$(arg prefix)"/>
+  <joint name="$(arg prefix)end_effector_joint" type="fixed">
     <parent link="$(arg prefix)end_effector_flange_link"/>
     <child link="$(arg prefix)end_effector_link"/>
@@ -45,5 +48,5 @@
       </material>
     </visual>
-  </link> -->
+  </link>
   <xacro:omy_f3m prefix="$(arg prefix)" />
   <xacro:omy_f3m_gazebo prefix="$(arg prefix)" />
@@ -54,6 +57,7 @@
     use_mock_hardware="$(arg use_mock_hardware)"
     mock_sensor_commands="$(arg mock_sensor_commands)"/>
-  <xacro:hx5_left_system
-    name="HX5LeftSystem" prefix="$(arg prefix)" use_sim="$(arg use_sim)"
+  <xacro:omy_f3m_hx5_right_end_system
+    name="OMYF3MEndHX5RightSystem" prefix="$(arg prefix)" port_name="/dev/ttyAMA4"
+    use_pressure_sensors="false" use_sim="$(arg use_sim)"
     use_mock_hardware="$(arg use_mock_hardware)"
     mock_sensor_commands="$(arg mock_sensor_commands)"/>

File: open_manipulator_description/urdf/omy_l100/omy_l100_arm.urdf.xacro (robot description, xacro)
@@ -199,5 +199,5 @@
          </inertial>
       </link>
-      <joint name="rh_r1_joint" type="fixed">
+      <joint name="rh_r1_joint" type="revolute">
          <parent link="${prefix}link6" />
          <child link="${prefix}link7" />
