Commit message: Supported jazzy version
Signed-off-by: Sungho Woo <wsh@robotis.com>

File: open_manipulator_description/gazebo/open_manipulator_x.gazebo.xacro (robot description, xacro)
@@ -22,5 +22,4 @@
       <maxVel>1.0</maxVel>
       <minDepth>0.001</minDepth>
-      <material>Gazebo/DarkGrey</material>
     </gazebo>
   </xacro:macro>
@@ -33,5 +32,4 @@
   <xacro:Link reference="${prefix}gripper_right_link"/>
   <gazebo reference="${prefix}end_effector_link">
-    <material>Gazebo/Red</material>
   </gazebo>
   <xacro:SimpleTransmission trans="${prefix}trans1" joint="${prefix}joint1" actuator="${prefix}actuator1" />

File: open_manipulator_description/ros2_control/open_manipulator_x_system.ros2_control.xacro (robot description, xacro)
@@ -2,8 +2,8 @@
 <robot xmlns:xacro="http://www.ros.org/wiki/xacro">
   <xacro:macro name="open_manipulator_x_system" params="name prefix port_name:=/dev/ttyUSB0 use_sim:=^|false use_fake_hardware:=^|false fake_sensor_commands:=^|false">
-    <ros2_control name="${name}" type="system">
+    <ros2_control name="omx" type="system">
       <xacro:if value="$(arg use_sim)">
         <hardware>
-          <plugin>gazebo_ros2_control/GazeboSystem</plugin>
+          <plugin>gz_ros2_control/GazeboSimSystem</plugin>
         </hardware>
       </xacro:if>
@@ -21,5 +21,5 @@
             <param name="error_timeout_sec">0.2</param>
             <param name="dynamixel_model_folder">/param/dxl_model</param>
-            <param name="number_of_joints">6</param>
+            <param name="number_of_joints">5</param>
             <param name="number_of_transmissions">5</param>
             <param name="transmission_to_joint_matrix">
@@ -28,13 +28,12 @@
               0, 0, 1, 0, 0,
               0, 0, 0, 1, 0,
-              0, 0, 0, 0, 1,
-              0, 0, 0, 0, 0
+              0, 0, 0, 0, 1
             </param>
             <param name="joint_to_transmission_matrix">
-              1, 0, 0, 0, 0, 0,
-              0, 1, 0, 0, 0, 0,
-              0, 0, 1, 0, 0, 0,
-              0, 0, 0, 1, 0, 0,
-              0, 0, 0, 0, 1, 0
+              1, 0, 0, 0, 0,
+              0, 1, 0, 0, 0,
+              0, 0, 1, 0, 0,
+              0, 0, 0, 1, 0,
+              0, 0, 0, 0, 1
             </param>
             <param name="ros_update_freq">200</param>
@@ -86,12 +85,13 @@
         <state_interface name="effort"/>
       </joint>
-      <joint name="${prefix}gripper_right_joint">
-        <param name="mimic">${prefix}gripper_left_joint</param>
-        <param name="multiplier">1</param>
-        <command_interface name="position"/>
-        <state_interface name="position"/>
-        <state_interface name="velocity"/>
-        <state_interface name="effort"/>
-      </joint>
+      <xacro:if value="$(arg use_sim)">
+        <joint name="${prefix}gripper_right_joint">
+          <param name="mimic">${prefix}gripper_left_joint</param>
+          <param name="multiplier">1</param>
+          <state_interface name="position"/>
+          <state_interface name="velocity"/>
+          <state_interface name="effort"/>
+        </joint>
+      </xacro:if>
       <gpio name="dxl1">
         <param name="type">dxl</param>

Commit message: add gripper camera

File: open_manipulator_description/gazebo/open_manipulator_x.gazebo.xacro (robot description, xacro)
@@ -39,4 +39,34 @@
   <xacro:SimpleTransmission trans="${prefix}trans5" joint="${prefix}gripper_left_joint" actuator="${prefix}actuator5" />
   <xacro:SimpleTransmission trans="${prefix}trans6" joint="${prefix}gripper_right_joint" actuator="${prefix}actuator6" />
+  <gazebo reference="${prefix}gripper_camera_link">
+    <sensor name="camera" type="camera">
+      <camera>
+        <horizontal_fov>1.3962634</horizontal_fov>
+        <image>
+          <width>640</width>
+          <height>480</height>
+          <format>R8G8B8</format>
+        </image>
+        <clip>
+          <near>0.01</near>
+          <far>15</far>
+        </clip>
+        <noise>
+          <type>gaussian</type>
+          <!-- Noise is sampled independently per pixel on each frame.
+               That pixel's noise value is added to each of its color
+               channels, which at that point lie in the range [0,1]. -->
+          <mean>0.0</mean>
+          <stddev>0.007</stddev>
+        </noise>
+        <optical_frame_id>${prefix}gripper_camera_link_optical</optical_frame_id>
+        <camera_info_topic>${prefix}gripper_camera/camera_info</camera_info_topic>
+      </camera>
+      <always_on>1</always_on>
+      <update_rate>20</update_rate>
+      <visualize>true</visualize>
+      <topic>${prefix}gripper_camera/image</topic>
+    </sensor>
+  </gazebo>
   </xacro:macro>
 </robot>

File: open_manipulator_description/urdf/om_x/open_manipulator_x_arm.urdf.xacro (robot description, xacro)
@@ -238,4 +238,36 @@
       </visual>
     </link>
+    <!-- Gripper camera -->
+    <joint type="fixed" name="${prefix}gripper_camera_joint">
+      <origin xyz="0.08 0.0 0.0" rpy="0 0 0"/>
+      <child link="${prefix}gripper_camera_link"/>
+      <parent link="${prefix}link5"/>
+    </joint>
+    <link name='${prefix}gripper_camera_link'>
+      <pose>0 0 0 0 0 0</pose>
+      <inertial>
+        <mass value="1.0e-03"/>
+        <origin xyz="0 0 0" rpy="0 0 0"/>
+        <inertia
+            ixx="1e-6" ixy="0" ixz="0"
+            iyy="1e-6" iyz="0"
+            izz="1e-6"
+        />
+      </inertial>
+      <visual>
+        <origin xyz="0 0 0" rpy="0 0 0"/>
+        <geometry>
+          <box size=".01 .01 .01"/>
+        </geometry>
+        <material name="red"/>
+      </visual>
+    </link>
+    <joint type="fixed" name="${prefix}gripper_camera_optical_joint">
+      <origin xyz="0 0 0" rpy="-1.5707 0 -1.5707"/>
+      <child link="${prefix}gripper_camera_link_optical"/>
+      <parent link="${prefix}gripper_camera_link"/>
+    </joint>
+    <link name="${prefix}gripper_camera_link_optical">
+    </link>
   </xacro:macro>
 </robot>
