Commit message: description omx
Signed-off-by: Wonho Yun <ywh@robotis.com>

File: open_manipulator_description/gazebo/omx.gazebo.xacro (robot description, xacro)
@@ -1,5 +1,5 @@
 <?xml version="1.0"?>
 <robot xmlns:xacro="http://ros.org/wiki/xacro">
-  <xacro:macro name="open_manipulator_x_gazebo" params="prefix">
+  <xacro:macro name="omx_gazebo" params="prefix">
   <xacro:macro name="SimpleTransmission" params="trans joint actuator">
     <transmission name="${trans}">

File: open_manipulator_description/ros2_control/omx.ros2_control.xacro (robot description, xacro)
@@ -1,5 +1,5 @@
 <?xml version="1.0"?>
 <robot xmlns:xacro="http://www.ros.org/wiki/xacro">
-  <xacro:macro name="open_manipulator_x_system" params="name prefix port_name:=^|/dev/ttyUSB0 use_sim:=^|false use_fake_hardware:=^|false fake_sensor_commands:=^|false">
+  <xacro:macro name="omx_system" params="name prefix port_name:=^|/dev/ttyUSB0 use_sim:=^|false use_fake_hardware:=^|false fake_sensor_commands:=^|false">
     <ros2_control name="${name}" type="system">
       <xacro:if value="$(arg use_sim)">

File: open_manipulator_description/urdf/omx/omx.urdf.xacro (robot description, xacro)
@@ -1,5 +1,5 @@
 <?xml version="1.0"?>
 <!-- OpenManipulator Chain -->
-<robot name="open_manipulator_x" xmlns:xacro="http://ros.org/wiki/xacro">
+<robot name="omx" xmlns:xacro="http://ros.org/wiki/xacro">
   <xacro:arg name="prefix" default="" />
   <xacro:arg name="use_sim" default="false" />
@@ -8,12 +8,12 @@
   <xacro:arg name="port_name" default="/dev/ttyUSB0" />
   <!-- Import all Gazebo-customization elements, including Gazebo colors -->
-  <xacro:include filename="$(find open_manipulator_description)/gazebo/open_manipulator_x.gazebo.xacro" />
+  <xacro:include filename="$(find open_manipulator_description)/gazebo/omx.gazebo.xacro" />
   <!-- Import URDF -->
-  <xacro:include filename="$(find open_manipulator_description)/urdf/om_x/open_manipulator_x_arm.urdf.xacro" />
-  <xacro:include filename="$(find open_manipulator_description)/ros2_control/open_manipulator_x_system.ros2_control.xacro" />
-  <xacro:open_manipulator_x prefix="$(arg prefix)" />
-  <xacro:open_manipulator_x_gazebo prefix="$(arg prefix)" />
-  <xacro:open_manipulator_x_system
-    name="OpenManipulatorXSystem" prefix="$(arg prefix)" use_sim="$(arg use_sim)"
+  <xacro:include filename="$(find open_manipulator_description)/urdf/omx/omx_arm.urdf.xacro" />
+  <xacro:include filename="$(find open_manipulator_description)/ros2_control/omx.ros2_control.xacro" />
+  <xacro:omx prefix="$(arg prefix)" />
+  <xacro:omx_gazebo prefix="$(arg prefix)" />
+  <xacro:omx_system
+    name="OMXSystem" prefix="$(arg prefix)" use_sim="$(arg use_sim)"
     use_fake_hardware="$(arg use_fake_hardware)"
     fake_sensor_commands="$(arg fake_sensor_commands)"

File: open_manipulator_description/urdf/omx/omx_arm.urdf.xacro (robot description, xacro)
@@ -1,8 +1,8 @@
 <?xml version="1.0"?>
 <robot xmlns:xacro="http://www.ros.org/wiki/xacro">
-  <xacro:macro name="open_manipulator_x" params="prefix=''">
+  <xacro:macro name="omx" params="prefix=''">
     <xacro:property
       name="meshes_file_direction"
-      value="package://open_manipulator_description/meshes/om_x"/>
+      value="package://open_manipulator_description/meshes/omx"/>
     <link name="${prefix}link1">
       <visual>
