Commit message: fix: Updated omy leader urdfs

File: open_manipulator_description/urdf/om_y_leader/open_manipulator_y_leader.urdf.xacro (robot description, xacro)
@@ -1,10 +1,25 @@
 <?xml version="1.0"?>
-<robot xmlns:xacro="http://www.ros.org/wiki/xacro" name="open_manipulator_y_leader">
-    <xacro:arg name="initial_positions_file" default="initial_positions.yaml" />
-    <xacro:property name="om_y_model" value="$(env OM_Y_MODEL)" />
-    <!-- Import open_manipulator_y_leader urdf file -->
-    <xacro:include filename="$(find open_manipulator_description)/urdf/om_y_leader/open_manipulator_y_leader_arm.urdf" />
-    <!-- Import control_xacro -->
-    <xacro:include filename="$(find open_manipulator_description)/ros2_control/open_manipulator_y_leader_system.ros2_control.xacro" />
-    <xacro:open_manipulator_y_leader_ros2_control name="open_manipulator_y_leader" initial_positions_file="$(arg initial_positions_file)"/>
+<robot name="open_manipulator_y_leader" xmlns:xacro="http://www.ros.org/wiki/xacro">
+  <xacro:arg name="prefix" default="" />
+  <xacro:arg name="use_sim" default="false" />
+  <xacro:arg name="use_fake_hardware" default="false" />
+  <xacro:arg name="fake_sensor_commands" default="false" />
+  <xacro:property name="robot_model" value="$(env ROBOT_MODEL)" />
+  <!-- Include OpenManipulator-Y_leader urdf macro -->
+  <xacro:include filename="$(find open_manipulator_description)/urdf/om_y_leader/open_manipulator_y_leader_arm.urdf" />
+  <!-- Include OpenManipulator-Y Leader ros2 control macro -->
+  <xacro:include filename="$(find open_manipulator_description)/ros2_control/open_manipulator_y_leader_system.ros2_control.xacro" />
+  <!-- World -->
+  <link name="world"/>
+  <!-- Used for fixing OpenManipulator-Y -->
+  <joint name="$(arg prefix)world_fixed" type="fixed">
+    <parent link="world"/>
+    <child link="$(arg prefix)link0"/>
+    <origin xyz="0.0 0.0 0.0" rpy="0 0 0"/>
+  </joint>
+  <xacro:open_manipulator_y_leader prefix="$(arg prefix)" />
+  <xacro:open_manipulator_y_leader_system
+    name="OpenManipulatorYLeaderSystem" prefix="$(arg prefix)" use_sim="$(arg use_sim)"
+    use_fake_hardware="$(arg use_fake_hardware)"
+    fake_sensor_commands="$(arg fake_sensor_commands)"/>
 </robot>

File: open_manipulator_description/urdf/om_y_leader/open_manipulator_y_leader_arm.urdf (robot description, URDF)
Before this commit: robot open_manipulator_y_leader, 8 links, 7 joints
Links:
- removed link base_link
- removed link link1
- removed link link2
- removed link link3
- removed link link4
- removed link link5
- removed link link6
- removed link link7
Joints:
- removed joint joint1
- removed joint joint2
- removed joint joint3
- removed joint joint4
- removed joint joint5
- removed joint joint6
- removed joint rh_r1_joint

Commit message: Modified omy leader for gazebo
Signed-off-by: Wonho Yun <ywh@robotis.com>

File: open_manipulator_description/urdf/om_y_leader/open_manipulator_y_leader.urdf.xacro (robot description, xacro)
@@ -5,7 +5,8 @@
   <xacro:arg name="use_fake_hardware" default="false" />
   <xacro:arg name="fake_sensor_commands" default="false" />
-  <xacro:property name="robot_model" value="$(env ROBOT_MODEL)" />
   <!-- Include OpenManipulator-Y_leader urdf macro -->
   <xacro:include filename="$(find open_manipulator_description)/urdf/om_y_leader/open_manipulator_y_leader_arm.urdf" />
+  <!-- Include OpenManipulator-Y_leader gazebo macro -->
+  <xacro:include filename="$(find open_manipulator_description)/gazebo/open_manipulator_y_leader.gazebo.xacro" />
   <!-- Include OpenManipulator-Y Leader ros2 control macro -->
   <xacro:include filename="$(find open_manipulator_description)/ros2_control/open_manipulator_y_leader_system.ros2_control.xacro" />
@@ -19,7 +20,13 @@
   </joint>
   <xacro:open_manipulator_y_leader prefix="$(arg prefix)" />
+  <xacro:open_manipulator_y_gazebo prefix="$(arg prefix)" />
   <xacro:open_manipulator_y_leader_system
     name="OpenManipulatorYLeaderSystem" prefix="$(arg prefix)" use_sim="$(arg use_sim)"
     use_fake_hardware="$(arg use_fake_hardware)"
     fake_sensor_commands="$(arg fake_sensor_commands)"/>
+  <gazebo>
+    <plugin filename="gz_ros2_control-system" name="gz_ros2_control::GazeboSimROS2ControlPlugin">
+      <parameters>$(find open_manipulator_bringup)/config/om_y_leader/gazebo_controller_manager.yaml</parameters>
+    </plugin>
+  </gazebo>
 </robot>
