Commit message: Refactor urdf files

File: open_manipulator_description/urdf/omx/omx.urdf.xacro (robot description, xacro)
@@ -1,4 +1,3 @@
 <?xml version="1.0"?>
-<!-- OpenManipulator Chain -->
 <robot name="omx" xmlns:xacro="http://ros.org/wiki/xacro">
   <xacro:arg name="prefix" default="" />
@@ -7,9 +6,13 @@
   <xacro:arg name="fake_sensor_commands" default="false" />
   <xacro:arg name="port_name" default="/dev/ttyUSB0" />
-  <!-- Import all Gazebo-customization elements, including Gazebo colors -->
   <xacro:include filename="$(find open_manipulator_description)/gazebo/omx.gazebo.xacro" />
-  <!-- Import URDF -->
   <xacro:include filename="$(find open_manipulator_description)/urdf/omx/omx_arm.urdf.xacro" />
   <xacro:include filename="$(find open_manipulator_description)/ros2_control/omx.ros2_control.xacro" />
+  <link name="world"/>
+  <joint name="$(arg prefix)world_fixed" type="fixed">
+    <origin xyz="0 0 0" rpy="0 0 0"/>
+    <parent link="world"/>
+    <child link="$(arg prefix)link1"/>
+  </joint>
   <xacro:omx prefix="$(arg prefix)" />
   <xacro:omx_gazebo prefix="$(arg prefix)" />
@@ -24,11 +27,3 @@
     </plugin>
   </gazebo>
-  <!-- World -->
-  <link name="world"/>
-  <!-- World fixed joint-->
-  <joint name="$(arg prefix)world_fixed" type="fixed">
-    <origin xyz="0 0 0" rpy="0 0 0"/>
-    <parent link="world"/>
-    <child link="$(arg prefix)link1"/>
-  </joint>
 </robot>

File: open_manipulator_description/urdf/omy_3m/omy_3m.urdf.xacro (robot description, xacro)
@@ -1,4 +1,3 @@
 <?xml version="1.0"?>
-<!-- OMY_base -->
 <robot name="omy_3m" xmlns:xacro="http://www.ros.org/wiki/xacro">
   <xacro:arg name="prefix" default="" />
@@ -6,15 +5,9 @@
   <xacro:arg name="use_fake_hardware" default="false" />
   <xacro:arg name="fake_sensor_commands" default="false" />
-  <xacro:property name="robot_model" value="$(env ROBOT_MODEL)" />
-  <!-- Include OMY_base urdf macro -->
   <xacro:include filename="$(find open_manipulator_description)/urdf/omy_3m/omy_3m_arm.urdf.xacro" />
-  <!-- Include OMY_base gazebo macro -->
   <xacro:include filename="$(find open_manipulator_description)/gazebo/omy_3m.gazebo.xacro" />
-  <!-- Include OMY_base ros2 control macro -->
   <xacro:include filename="$(find open_manipulator_description)/ros2_control/omy_3m.ros2_control.xacro" />
   <xacro:include filename="$(find open_manipulator_description)/ros2_control/omy_3m_end_unit.ros2_control.xacro" />
-  <!-- World -->
   <link name="world"/>
-  <!-- Used for fixing OMY_base -->
   <joint name="$(arg prefix)world_fixed" type="fixed">
     <parent link="world"/>
@@ -25,9 +18,9 @@
   <xacro:omy_3m_gazebo prefix="$(arg prefix)" />
   <xacro:omy_3m_system
-    name="Omy3mSystem" prefix="$(arg prefix)" use_sim="$(arg use_sim)"
+    name="OMY3MSystem" prefix="$(arg prefix)" use_sim="$(arg use_sim)"
     use_fake_hardware="$(arg use_fake_hardware)"
     fake_sensor_commands="$(arg fake_sensor_commands)"/>
-  <xacro:omy_3m_end_unit
-    name="Omy3mEndUnit" prefix="$(arg prefix)" use_sim="$(arg use_sim)"
+  <xacro:omy_3m_end_unit_system
+    name="OMY3MEndUnitSystem" prefix="$(arg prefix)" use_sim="$(arg use_sim)"
     use_fake_hardware="$(arg use_fake_hardware)"
     fake_sensor_commands="$(arg fake_sensor_commands)"/>

File: open_manipulator_description/urdf/omy_f3m/omy_f3m.urdf.xacro (robot description, xacro)
@@ -1,4 +1,3 @@
 <?xml version="1.0"?>
-<!-- OpenManipulator-Y -->
 <robot name="omy_f3m" xmlns:xacro="http://www.ros.org/wiki/xacro">
   <xacro:arg name="prefix" default="" />
@@ -7,19 +6,11 @@
   <xacro:arg name="fake_sensor_commands" default="false" />
   <xacro:arg name="config_type" default="omy_f3m" />
-  <xacro:property name="robot_model" value="$(env ROBOT_MODEL)" />
-  <!-- Include OpenManipulator-Y urdf macro -->
   <xacro:include filename="$(find open_manipulator_description)/urdf/omy_f3m/omy_f3m_arm.urdf.xacro" />
-  <!-- Include OpenManipulator-Y gazebo macro -->
   <xacro:include filename="$(find open_manipulator_description)/gazebo/omy_f3m.gazebo.xacro" />
-  <!-- Include Gripper urdf macro -->
   <xacro:include filename="$(find open_manipulator_description)/urdf/omy_f3m/rh_p12_rn_a.urdf.xacro" />
-  <!-- Include Gripper gazebo macro -->
   <xacro:include filename="$(find open_manipulator_description)/gazebo/rh_p12_rn_a.gazebo.xacro" />
-  <!-- Include OpenManipulator-Y ros2 control macro -->
   <xacro:include filename="$(find open_manipulator_description)/ros2_control/omy_f3m.ros2_control.xacro" />
   <xacro:include filename="$(find open_manipulator_description)/ros2_control/omy_f3m_end_unit.ros2_control.xacro" />
-  <!-- World -->
   <link name="world"/>
-  <!-- Used for fixing OpenManipulator-Y -->
   <joint name="$(arg prefix)world_fixed" type="fixed">
     <parent link="world"/>
@@ -38,9 +29,9 @@
   <xacro:rh_p12_rn_a_gazebo prefix="$(arg prefix)" />
   <xacro:omy_f3m_system
-    name="OmyF3mSystem" prefix="$(arg prefix)" use_sim="$(arg use_sim)"
+    name="OMYF3MSystem" prefix="$(arg prefix)" use_sim="$(arg use_sim)"
     use_fake_hardware="$(arg use_fake_hardware)"
     fake_sensor_commands="$(arg fake_sensor_commands)"/>
-  <xacro:omy_f3m_end_unit
-    name="OmyF3mEndUnit" prefix="$(arg prefix)" use_sim="$(arg use_sim)"
+  <xacro:omy_f3m_end_unit_system
+    name="OMYF3MEndUnitSystem" prefix="$(arg prefix)" use_sim="$(arg use_sim)"
     use_fake_hardware="$(arg use_fake_hardware)"
     fake_sensor_commands="$(arg fake_sensor_commands)"/>

File: open_manipulator_description/urdf/omy_l100/omy_l100.urdf.xacro (robot description, xacro)
@@ -5,13 +5,9 @@
   <xacro:arg name="use_fake_hardware" default="false" />
   <xacro:arg name="fake_sensor_commands" default="false" />
-  <!-- Include OpenManipulator-Y_leader urdf macro -->
+  <xacro:arg name="port_name" default="/dev/ttyUSB0" />
   <xacro:include filename="$(find open_manipulator_description)/urdf/omy_l100/omy_l100_arm.urdf" />
-  <!-- Include OpenManipulator-Y_leader gazebo macro -->
   <xacro:include filename="$(find open_manipulator_description)/gazebo/omy_l100.gazebo.xacro" />
-  <!-- Include OpenManipulator-Y Leader ros2 control macro -->
-  <xacro:include filename="$(find open_manipulator_description)/ros2_control/omy_l100_system.ros2_control.xacro" />
-  <!-- World -->
+  <xacro:include filename="$(find open_manipulator_description)/ros2_control/omy_l100.ros2_control.xacro" />
   <link name="world"/>
-  <!-- Used for fixing OpenManipulator-Y -->
   <joint name="$(arg prefix)world_fixed" type="fixed">
     <parent link="world"/>
@@ -22,7 +18,8 @@
   <xacro:omy_l100_gazebo prefix="$(arg prefix)" />
   <xacro:omy_l100_system
-    name="OpenManipulatorYLeaderSystem" prefix="$(arg prefix)" use_sim="$(arg use_sim)"
+    name="OMYL100System" prefix="$(arg prefix)" use_sim="$(arg use_sim)"
     use_fake_hardware="$(arg use_fake_hardware)"
-    fake_sensor_commands="$(arg fake_sensor_commands)"/>
+    fake_sensor_commands="$(arg fake_sensor_commands)"
+    port_name="$(arg port_name)"/>
   <gazebo>
     <plugin filename="gz_ros2_control-system" name="gz_ros2_control::GazeboSimROS2ControlPlugin">
