Commit message: Add end effector joint and link to omy_3m URDF, Change launch file to disable simulation time by default.

File: open_manipulator_description/urdf/omy_3m/omy_3m.urdf.xacro (robot description, xacro)
@@ -15,4 +15,20 @@
     <origin xyz="0.0 0.0 0.0" rpy="0 0 0"/>
   </joint>
+  <joint name="$(arg prefix)end_effector_joint" type="fixed">
+      <parent link="$(arg prefix)link6" />
+      <child link="$(arg prefix)end_effector_link" />
+      <origin xyz="0 -0.103 0" rpy="0 0 0" />
+  </joint>
+  <link name="$(arg prefix)end_effector_link">
+      <visual>
+        <origin xyz="0 0 0" rpy="0 0 0"/>
+        <geometry>
+        <box size="0.01 0.01 0.01" />
+        </geometry>
+        <material name="red">
+        <color rgba="1.0 0.0 0.0 1"/>
+        </material>
+      </visual>
+  </link>
   <xacro:omy_3m prefix="$(arg prefix)" />
   <xacro:omy_3m_gazebo prefix="$(arg prefix)" />
