Commit message: fix: remove trailing slashes from mesh file paths in URDF models for omx_f, omx_l, omy_3m, omy_f3m, and omy_l100

File: open_manipulator_description/urdf/omy_3m/omy_3m.urdf (robot description, URDF)
Before this commit: robot omy_3m, 9 links, 8 joints
Links:
- link link0: geometry collision cylinder length=0.05 radius=0.08; visual mesh filename=package://open_manipulator_description/meshes/omy_3m/base_u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 scale=0.001 0.001 0.001
- link link1: geometry collision cylinder length=0.1 radius=0.055; visual mesh filename=package://open_manipulator_description/meshes/omy_3m/link1.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 scale=0.001 0.001 0.001
- link link2: geometry collision cylinder length=0.28 radius=0.046; visual mesh filename=package://open_manipulator_description/meshes/omy_3m/link2.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 scale=0.001 0.001 0.001
- link link3: geometry collision cylinder length=0.19 radius=0.042; visual mesh filename=package://open_manipulator_description/meshes/omy_3m/link3.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 scale=0.001 0.001 0.001
- link link4: geometry collision cylinder length=0.10 radius=0.045; visual mesh filename=package://open_manipulator_description/meshes/omy_3m/link4.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 scale=0.001 0.001 0.001
- link link5: geometry collision cylinder length=0.05 radius=0.043; visual mesh filename=package://open_manipulator_description/meshes/omy_3m/link5.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 scale=0.001 0.001 0.001
- link link6: geometry collision cylinder length=0.22 radius=0.09; visual mesh filename=package://open_manipulator_description/meshes/omy_3m/link6.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 scale=0.001 0.001 0.001

File: open_manipulator_description/urdf/omy_f3m/omy_f3m.urdf (robot description, URDF)
Before this commit: robot omy_f3m, 15 links, 14 joints
Links:
- link end_effector_flange_link: geometry collision cylinder length=0.12 radius=0.035; visual mesh filename=package://open_manipulator_description/meshes/omy_f3m/flang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 scale=0.001 0.001 0.001
- link link0: geometry collision cylinder length=0.05 radius=0.08; visual mesh filename=package://open_manipulator_description/meshes/omy_f3m/base_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 scale=0.001 0.001 0.001
- link link1: geometry collision cylinder length=0.1 radius=0.055; visual mesh filename=package://open_manipulator_description/meshes/omy_f3m/link1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 scale=0.001 0.001 0.001
- link link2: geometry collision cylinder length=0.28 radius=0.046; visual mesh filename=package://open_manipulator_description/meshes/omy_f3m/link2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 scale=0.001 0.001 0.001
- link link3: geometry collision cylinder length=0.17 radius=0.042; visual mesh filename=package://open_manipulator_description/meshes/omy_f3m/link3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 scale=0.001 0.001 0.001
- link link4: geometry collision cylinder length=0.10 radius=0.045; visual mesh filename=package://open_manipulator_description/meshes/omy_f3m/link4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 scale=0.001 0.001 0.001
- link link5: geometry collision cylinder length=0.05 radius=0.043; visual mesh filename=package://open_manipulator_description/meshes/omy_f3m/link5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 scale=0.001 0.001 0.001
- link link6: geometry collision cylinder length=0.22 radius=0.08; visual mesh filename=package://open_manipulator_description/meshes/omy_f3m/link6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 scale=0.001 0.001 0.001

File: open_manipulator_description/urdf/omy_l100/omy_l100.urdf (robot description, URDF)
Before this commit: robot omy_l100, 9 links, 8 joints
Links:
- link link0: geometry collision mesh filename=package://open_manipulator_description/meshes/omy_l100/base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 scale=0.001 0.001 0.001; visual mesh filename=package://open_manipulator_description/meshes/omy_l100/base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 scale=0.001 0.001 0.001
- link link1: geometry collision mesh filename=package://open_manipulator_description/meshes/omy_l100/link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 scale=0.001 0.001 0.001; visual mesh filename=package://open_manipulator_description/meshes/omy_l100/link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 scale=0.001 0.001 0.001
- link link2: geometry collision mesh filename=package://open_manipulator_description/meshes/omy_l100/link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 scale=0.001 0.001 0.001; visual mesh filename=package://open_manipulator_description/meshes/omy_l100/link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 scale=0.001 0.001 0.001
- link link3: geometry collision mesh filename=package://open_manipulator_description/meshes/omy_l100/link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 scale=0.001 0.001 0.001; visual mesh filename=package://open_manipulator_description/meshes/omy_l100/link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 scale=0.001 0.001 0.001
- link link4: geometry collision mesh filename=package://open_manipulator_description/meshes/omy_l100/link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 scale=0.001 0.001 0.001; visual mesh filename=package://open_manipulator_description/meshes/omy_l100/link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 scale=0.001 0.001 0.001
- link link5: geometry collision mesh filename=package://open_manipulator_description/meshes/omy_l100/link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 scale=0.001 0.001 0.001; visual mesh filename=package://open_manipulator_description/meshes/omy_l100/link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 scale=0.001 0.001 0.001
- link link6: geometry collision mesh filename=package://open_manipulator_description/meshes/omy_l100/link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 scale=0.001 0.001 0.001; visual mesh filename=package://open_manipulator_description/meshes/omy_l100/link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 scale=0.001 0.001 0.001
- link link7: geometry collision mesh filename=package://open_manipulator_description/meshes/omy_l100/link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 scale=0.001 0.001 0.001; visual mesh filename=package://open_manipulator_description/meshes/omy_l100/link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 scale=0.001 0.001 0.001
