Commit message: Update omy_f3m URDF and MoveIt configuration: add end effector joint and link, adjust joint limits, and modify launch file to disable simulation time by default.

File: open_manipulator_description/urdf/omy_f3m/omy_f3m.urdf.xacro (robot description, xacro)
@@ -16,5 +16,5 @@
     <parent link="world"/>
     <child link="$(arg prefix)link0"/>
-    <origin xyz="0.0 0.0 0.0" rpy="0 0 0"/>
+    <origin xyz="0 0 0" rpy="0 0 0"/>
   </joint>
   <joint name="$(arg prefix)gripper_fixed" type="fixed">
@@ -24,4 +24,20 @@
     <child link="$(arg prefix)rh_p12_rn_base"/>
   </joint>
+  <joint name="$(arg prefix)end_effector_joint" type="fixed">
+    <parent link="$(arg prefix)end_effector_flange_link"/>
+    <child link="$(arg prefix)end_effector_link"/>
+    <origin xyz="0 -0.141 0" rpy="0 0 0"/>
+  </joint>
+  <link name="$(arg prefix)end_effector_link">
+    <visual>
+      <origin xyz="0 0 0" rpy="0 0 0"/>
+      <geometry>
+        <box size="0.01 0.01 0.01" />
+      </geometry>
+      <material name="red">
+        <color rgba="1.0 0.0 0.0 1"/>
+      </material>
+    </visual>
+  </link>
   <xacro:omy_f3m prefix="$(arg prefix)" />
   <xacro:omy_f3m_gazebo prefix="$(arg prefix)" />

Commit message: fix: Correct orientation of gripper_fixed joint in OMY F3M URDF

File: open_manipulator_description/urdf/omy_f3m/omy_f3m.urdf.xacro (robot description, xacro)
@@ -19,5 +19,5 @@
   </joint>
   <joint name="$(arg prefix)gripper_fixed" type="fixed">
-    <origin xyz="0 -0.006 0" rpy="1.57 1.57 0"/>
+    <origin xyz="0 -0.006 0" rpy="1.57 -1.57 0"/>
     <parent link="$(arg prefix)end_effector_flange_link"/>
     <axis xyz="0 0 0"/>
