Commit message: Remerged feature
Signed-off-by: Sungho Woo <wsh@robotis.com>

File: open_manipulator_description/urdf/omy_f3m/omy_f3m_arm.urdf.xacro (robot description, xacro)
@@ -223,5 +223,5 @@
             <origin xyz="0 0.03 0.04" rpy="0 0 0" />
             <geometry>
-               <cylinder radius="0.04" length="0.12"/>
+               <cylinder radius="0.035" length="0.12"/>
             </geometry>
          </collision>

Commit message: Calibrated collision
Signed-off-by: Sungho Woo <wsh@robotis.com>

File: open_manipulator_description/urdf/omy_f3m/omy_f3m_arm.urdf.xacro (robot description, xacro)
@@ -223,5 +223,5 @@
             <origin xyz="0 0.03 0.04" rpy="0 0 0" />
             <geometry>
-               <cylinder radius="0.035" length="0.12"/>
+               <cylinder radius="0.03" length="0.12"/>
             </geometry>
          </collision>

Commit message: Calibrated collision
Signed-off-by: Sungho Woo <wsh@robotis.com>

File: open_manipulator_description/urdf/omy_f3m/omy_f3m_arm.urdf.xacro (robot description, xacro)
@@ -223,5 +223,5 @@
             <origin xyz="0 0.03 0.04" rpy="0 0 0" />
             <geometry>
-               <cylinder radius="0.03" length="0.12"/>
+               <cylinder radius="0.025" length="0.12"/>
             </geometry>
          </collision>

Commit message: Calibarated collision
Signed-off-by: Sungho Woo <wsh@robotis.com>

File: open_manipulator_description/urdf/omy_f3m/omy_f3m_arm.urdf.xacro (robot description, xacro)
@@ -196,5 +196,5 @@
             <origin xyz="0 -0.1 0" rpy="1.57 0 0" />
             <geometry>
-               <cylinder radius="0.09" length="0.22"/>
+               <cylinder radius="0.08" length="0.22"/>
             </geometry>
          </collision>
@@ -223,5 +223,5 @@
             <origin xyz="0 0.03 0.04" rpy="0 0 0" />
             <geometry>
-               <cylinder radius="0.025" length="0.12"/>
+               <cylinder radius="0.035" length="0.12"/>
             </geometry>
          </collision>

Commit message: Modified rt buffer
Signed-off-by: Sungho Woo <wsh@robotis.com>

File: open_manipulator_description/urdf/omy_f3m/omy_f3m_arm.urdf.xacro (robot description, xacro)
@@ -106,5 +106,5 @@
             <origin xyz="0 0.125 0.08" rpy="0 0 0" />
             <geometry>
-               <cylinder radius="0.042" length="0.19"/>
+               <cylinder radius="0.042" length="0.17"/>
             </geometry>
          </collision>
