Commit message: Update URDF files for omx_f and omx_l arms to adjust joint origins and axes for improved configuration

File: open_manipulator_description/urdf/omx_f/omx_f_arm.urdf.xacro (robot description, xacro)
@@ -15,5 +15,5 @@
          <parent link="${prefix}link1" />
          <child link="${prefix}link2" />
-         <origin xyz="0 0 0" rpy="0 0 0" />
+         <origin xyz="0 0 0.05" rpy="0 0 0" />
          <axis xyz="0 1 0" />
          <limit velocity="4.8" effort="1000" lower="${-pi*2.0}" upper="${pi*2.0}" />
@@ -24,5 +24,5 @@
          <parent link="${prefix}link2" />
          <child link="${prefix}link3" />
-          <origin xyz="0 0 0" rpy="0 0 0" />
+          <origin xyz="0 0 0.05" rpy="0 0 0" />
          <axis xyz="0 1 0" />
          <limit velocity="4.8" effort="1000" lower="${-pi*2.0}" upper="${pi*2.0}" />
@@ -33,5 +33,5 @@
          <parent link="${prefix}link3" />
          <child link="${prefix}link4" />
-         <origin xyz="0 0 0" rpy="0 0 0" />
+         <origin xyz="0.05 0 0" rpy="0 0 0" />
          <axis xyz="0 1 0" />
          <limit velocity="4.8" effort="1000" lower="${-pi*2.0}" upper="${pi*2.0}" />
@@ -42,6 +42,6 @@
          <parent link="${prefix}link4" />
          <child link="${prefix}link5" />
-         <origin xyz="0 0 0" rpy="0 0 0" />
-         <axis xyz="0 0 1" />
+         <origin xyz="0.05 0 0" rpy="0 0 0" />
+         <axis xyz="1 0 0" />
          <limit velocity="4.8" effort="1000" lower="${-pi*2.0}" upper="${pi*2.0}" />
          <dynamics damping="0.1" />
@@ -51,16 +51,10 @@
          <parent link="${prefix}link5" />
          <child link="${prefix}link6" />
-         <origin xyz="0 0 0" rpy="0 0 0" />
-         <axis xyz="0 1 0" />
+         <origin xyz="0.05 0 0" rpy="0 0 0" />
+         <axis xyz="0 0 1" />
          <limit velocity="4.8" effort="1000" lower="${-pi*2.0}" upper="${pi*2.0}" />
          <dynamics damping="0.1" />
       </joint>
       <link name="${prefix}link6" />
-      <joint name="${prefix}end_effector_flange_joint" type="fixed">
-         <parent link="${prefix}link6" />
-         <child link="${prefix}link7" />
-         <origin xyz="0 0 0" rpy="0 0 0" />
-      </joint>
-      <link name="${prefix}link7" />
    </xacro:macro>
 </robot>
